Commit message: conversion in progress.
git-svn-id: https://svn.code.sf.net/p/personalrobots/code/pkg/trunk@20414 f5854215-dd47-0410-b2c4-cdd35faa7885

Former-commit-id: 6df599fe0298c84ab4914ffd8a2b77f2e80e6007

File: stacks/pr2/pr2_defs/defs/body_defs.urdf.xacro (robot description, xacro)
@@ -4,62 +4,60 @@
        xmlns:interface="http://playerstage.sourceforge.net/gazebo/xmlschema/#interface">
   <macro name="pr2_torso" params="name parent *origin">
-    <joint name="${name}_joint" type="prismatic">
-      <!-- KWatts: Max should be 0.31, changed to 0.20 to prevent jamming -->
-      <!-- HW ticket 481, will examine spine to determine failures -->
-      <limit min="0.0" max="0.20" effort="10000"
-             velocity="0.015" k_velocity="400000"
-             safety_length_min="0.005" safety_length_max="0.005" k_position="1000" />
-      <calibration reference_position="0.00536" values="0 0" />
-      <axis xyz="0 0 1" />
-      <joint_properties damping="10.0" />
-    </joint>
+    <link name="${name}_link">
+      <joint name="${name}_joint" type="prismatic">
+        <origin xyz="0 0 0" rpy="0 0 0" />
+        <axis xyz="0 0 1" />
+        <!-- KWatts: Max should be 0.31, changed to 0.20 to prevent jamming -->
+        <!-- HW ticket 481, will examine spine to determine failures -->
+        <limit min="0.0" max="0.20" effort="10000" velocity="0.015"/>
+        <safety_controller  k_velocity="400000" lower="${0.0+0.005}" upper="${0.20-0.005}" k_position="1000" />
+        <joint_properties damping="10.0" />
+        <parent name="${parent}">
+          <insert_block name="origin" />
+        </parent>
+      </joint>
+      <inertial>
+        <mass value="36.248046" />
+        <origin xyz="-0.1 0 -0.0885" />
+        <inertia ixx="2.771653750257" ixy="0.004284522609" ixz="-0.160418504506"
+                 iyy="2.510019507959" iyz="0.029664468704" izz="0.526432355569" />
+      </inertial>
+      <visual name="${name}_visual">
+        <origin xyz="0 0 0" rpy="0 0 0" />
+        <geometry name="${name}_visual_geom">
+          <mesh filename="torso.stlb" />
+        </geometry>
+      </visual>
+      <collision name="${name}_collision">
+        <origin xyz="-0.1 0 -0.0885" rpy="0 0 0" />
+        <geometry name="${name}_collision_geom">
+          <box size="0.30 0.620 0.823" />
+        </geometry>
+      </collision>
+    </link>
+    <gazebo name="${name}_sensor" reference="${name}_link">
+      <sensor:contact name="${name}_contact_sensor">
+        <geom>${name}_collision</geom>
+        <updateRate>100.0</updateRate>
+        <controller:ros_bumper name="${name}_ros_bumper_controller" plugin="libros_bumper.so">
+          <alwaysOn>true</alwaysOn>
+          <updateRate>100.0</updateRate>
+          <bumperTopicName>${name}_bumper</bumperTopicName>
+          <interface:bumper name="${name}_ros_bumper_iface" />
+        </controller:ros_bumper>
+      </sensor:contact>
+    </gazebo>
+    <gazebo name="gazebo_material" reference="${name}_visual">
+      <material value="PR2/Grey2" />
+    </gazebo>
+    <ogre name="${name}_visual_mesh" reference="${name}_visual">
+      <mesh value="torso.mesh" />
+    </ogre>
     <transmission type="SimpleTransmission" name="${name}_trans">
       <actuator name="${name}_motor" />
       <joint name="${name}_joint" />
       <mechanicalReduction>-52143.33</mechanicalReduction>
+      <calibration reference_position="0.00536" values="0 0" />
     </transmission>
-    <link name="${name}_link">
-      <parent name="${parent}" />
-      <insert_block name="origin" />
-      <joint name="${name}_joint" />
-      <inertial>
-        <mass value="36.248046" />
-        <com xyz="-0.1 0 -0.0885" />
-        <inertia ixx="2.771653750257" ixy="0.004284522609" ixz="-0.160418504506"
-                 iyy="2.510019507959" iyz="0.029664468704" izz="0.526432355569" />
-      </inertial>
-      <visual>
-        <origin xyz="0 0 0" rpy="0 0 0" />
-        <map name="gazebo_material" flag="gazebo">
-	  <elem key="material" value="PR2/Grey2" />
-        </map>
-        <geometry name="${name}_visual">
-          <mesh filename="torso.stlb" />
-        </geometry>
-        <map name="${name}_visual_mesh" flag="ogre">
-          <elem key="mesh" value="torso.mesh" />
-        </map>
-      </visual>
-      <collision>
-        <origin xyz="-0.1 0 -0.0885" rpy="0 0 0" />
-        <geometry name="${name}_collision">
-          <box size="0.30 0.620 0.823" />
-        </geometry>
-      </collision>
-      <map name="${name}_sensor" flag="gazebo">
-        <verbatim key="${name}_bumper_sensor">
-          <sensor:contact name="${name}_contact_sensor">
-            <geom>${name}_collision</geom>
-            <updateRate>100.0</updateRate>
-            <controller:ros_bumper name="${name}_ros_bumper_controller" plugin="libros_bumper.so">
-              <alwaysOn>true</alwaysOn>
-              <updateRate>100.0</updateRate>
-              <bumperTopicName>${name}_bumper</bumperTopicName>
-              <interface:bumper name="${name}_ros_bumper_iface" />
-            </controller:ros_bumper>
-          </sensor:contact>
-        </verbatim>
-      </map>
-    </link>
   </macro>
   <!--                    Calibration                            -->

File: stacks/pr2/pr2_defs/defs/mono_cam_defs.urdf.xacro (robot description, xacro)
@@ -2,61 +2,64 @@
 <root>
 <macro name="mono_cam" params="name parent *origin">
-  <joint name="${name}_fixed_joint" type="fixed" />
   <link name="${name}_frame">
-    <insert_block name="origin" />
-    <parent name="${parent}" />
-    <joint name="${name}_fixed_joint" />
+    <joint name="${name}_fixed_joint" type="fixed">
+      <origin xyz="0 0 0" />
+      <parent name="${parent}">
+        <insert_block name="origin" />
+      </parent>
+    </joint>
     <inertial>
       <mass value="0.01" />
-      <com xyz="0 0 0" />
+      <origin xyz="0 0 0" />
       <inertia ixx="0.001"  ixy="0.0"  ixz="0.0"
                iyy="0.001"  iyz="0.0"
                izz="0.001" />
     </inertial>
-    <visual>
+    <visual name="${name}_visual">
       <origin xyz="0 0 0" rpy="0 0 0" />
-      <map name="gazebo_material" flag="gazebo">
-        <elem key="material" value="PR2/Blue" />
-      </map>
-      <geometry name="${name}_visual">
+      <geometry name="${name}_visual_geom">
         <box size="0.01 0.01 0.01" />
       </geometry>
     </visual>
-    <collision>
+    <collision name="${name}_collision">
       <origin xyz="0 0 0" rpy="0 0 0"/>
-      <geometry name="${name}_collision">
+      <geometry name="${name}_collision_geom">
         <box size="0.01 0.01 0.01" />
       </geometry>
     </collision>
   </link>
-  <joint name="${name}_optical_fixed_joint" type="fixed" />
   <link name="${name}_optical_frame">
-    <parent name="${name}_frame" />
-    <joint name="${name}_optical_fixed_joint" />
-    <origin xyz="0 0 0"
-            rpy="${-M_PI/2} 0.0 ${-M_PI/2}" />
+    <joint name="${name}_optical_fixed_joint" type="fixed" />
+      <origin xyz="0 0 0" rpy="0 0 0" />
+      <parent name="${name}_frame" />
+        <origin xyz="0 0 0" rpy="${-M_PI/2} 0.0 ${-M_PI/2}" />
+      </parent>
+    </joint>
     <inertial>
       <mass value="0.01" />
-      <com xyz="0 0 0" />
+      <origin xyz="0 0 0" />
       <inertia ixx="0.001"  ixy="0.0"  ixz="0.0"
                iyy="0.001"  iyz="0.0"
                izz="0.001" />
     </inertial>
-    <visual>
+    <visual name="${name}_optical_visual">
       <origin xyz="0 0 0" rpy="0 0 0"/>
-      <map name="gazebo_material" flag="gazebo">
-        <elem key="material" value="PR2/Blue" />
-      </map>
-      <geometry name="${name}_optical_visual">
+      <geometry name="${name}_optical_visual_geom">
         <box size="0.01 0.01 0.01" />
       </geometry>
     </visual>
-    <collision>
+    <collision name="${name}_optical_collision">
       <origin xyz="0 0 0" rpy="0 0 0"/>
-      <geometry name="${name}_optical_collision">
+      <geometry name="${name}_optical_collision_geom">
         <box size="0.01 0.01 0.01" />
       </geometry>
     </collision>
   </link>
+  <ogre name="gazebo_material" reference="${name}_visual">
+    <material value="PR2/Blue" />
+  </ogre>
+  <ogre name="gazebo_material" reference="${name}_optical_visual">
+    <material value="PR2/Blue" />
+  </ogre>
 </macro>
 </root>

File: stacks/pr2/pr2_defs/defs/prosilica_defs.urdf.xacro (robot description, xacro)
@@ -4,93 +4,95 @@
       xmlns:interface="http://playerstage.sourceforge.net/gazebo/xmlschema/#interface">
 <macro name="prosilica_cam" params="name parent *origin">
-  <joint name="${name}_fixed_joint" type="fixed" />
   <link name="${name}_frame">
-    <insert_block name="origin" />
-    <parent name="${parent}" />
-    <joint name="${name}_fixed_joint" />
+    <joint name="${name}_fixed_joint" type="fixed">
+      <origin xyz="0 0 0" rpy="0 0 0"/>
+      <parent name="${parent}">
+        <insert_block name="origin" />
+      </parent>
+    </joint>
     <inertial>
       <mass value="0.01" />
-      <com xyz="0 0 0" />
+      <origin xyz="0 0 0" rpy="0 0 0"/>
       <inertia ixx="0.001"  ixy="0.0"  ixz="0.0"
                iyy="0.001"  iyz="0.0"
                izz="0.001" />
     </inertial>
-    <visual>
+    <visual name="${name}_visual">
       <origin xyz="0 0 0" rpy="0 0 0" />
-      <map name="gazebo_material" flag="gazebo">
-        <elem key="material" value="PR2/Blue" />
-      </map>
-      <geometry name="${name}_visual">
+      <geometry name="${name}_visual_geom">
         <box size="0.01 0.01 0.01" />
       </geometry>
     </visual>
-    <collision>
+    <collision name="${name}_collision">
       <origin xyz="0 0 0" rpy="0 0 0"/>
-      <geometry name="${name}_collision">
+      <geometry name="${name}_collision_geom">
         <box size="0.01 0.01 0.01" />
       </geometry>
     </collision>
-    <map name="sensor" flag="gazebo">
-      <verbatim key="sensor_${name}_camera">
-        <sensor:camera name="${name}_sensor">
-          <imageFormat>B8G8R8</imageFormat>
-          <imageSize>2448 2050</imageSize>
-          <hfov>45</hfov>
-          <nearClip>0.1</nearClip>
-          <farClip>100</farClip>
-          <updateRate>20.0</updateRate>
-          <controller:ros_prosilica name="${name}_controller" plugin="libros_prosilica.so">
-            <alwaysOn>true</alwaysOn>
-            <updateRate>20.0</updateRate>
-            <camInfoTopicName>/prosilica/cam_info</camInfoTopicName>
-            <imageTopicName>/prosilica/image</imageTopicName>
-            <imageRectTopicName>/prosilica/image_rect</imageRectTopicName>
-            <camInfoServiceName>/prosilica/cam_info_service</camInfoServiceName>
-            <pollServiceName>/prosilica/poll</pollServiceName>
-            <frameName>hight_def_optical_frame</frameName>
-            <CxPrime>1224.5</CxPrime>
-            <Cx>1224.5</Cx>
-            <Cy>1025.5</Cy>
-            <focal_length>2955</focal_length> <!-- image_width / (2*tan(hfov_radian /2)) -->
-            <distortion_k1>0</distortion_k1>
-            <distortion_k2>0</distortion_k2>
-            <distortion_k3>0</distortion_k3>
-            <distortion_t1>0</distortion_t1>
-            <distortion_t2>0</distortion_t2>
-            <interface:camera name="${name}_iface" />
-          </controller:ros_prosilica>
-        </sensor:camera>
-      </verbatim>
-    </map>
   </link>
-  <joint name="${name}_optical_fixed_joint" type="fixed" />
+  <gazebo name="sensor" reference="${name}_rame">
+    <sensor:camera name="${name}_sensor">
+      <imageFormat>B8G8R8</imageFormat>
+      <imageSize>2448 2050</imageSize>
+      <hfov>45</hfov>
+      <nearClip>0.1</nearClip>
+      <farClip>100</farClip>
+      <updateRate>20.0</updateRate>
+      <controller:ros_prosilica name="${name}_controller" plugin="libros_prosilica.so">
+        <alwaysOn>true</alwaysOn>
+        <updateRate>20.0</updateRate>
+        <camInfoTopicName>/prosilica/cam_info</camInfoTopicName>
+        <imageTopicName>/prosilica/image</imageTopicName>
+        <imageRectTopicName>/prosilica/image_rect</imageRectTopicName>
+        <camInfoServiceName>/prosilica/cam_info_service</camInfoServiceName>
+        <pollServiceName>/prosilica/poll</pollServiceName>
+        <frameName>hight_def_optical_frame</frameName>
+        <CxPrime>1224.5</CxPrime>
+        <Cx>1224.5</Cx>
+        <Cy>1025.5</Cy>
+        <focal_length>2955</focal_length> <!-- image_width / (2*tan(hfov_radian /2)) -->
+        <distortion_k1>0</distortion_k1>
+        <distortion_k2>0</distortion_k2>
+        <distortion_k3>0</distortion_k3>
+        <distortion_t1>0</distortion_t1>
+        <distortion_t2>0</distortion_t2>
+        <interface:camera name="${name}_iface" />
+      </controller:ros_prosilica>
+    </sensor:camera>
+  </gazebo>
+  <gazebo name="gazebo_material" reference="${name}_visual">
+    <material value="PR2/Blue" />
+  </gazebo>
   <link name="${name}_optical_frame">
-    <parent name="${name}_frame" />
-    <joint name="${name}_optical_fixed_joint" />
-    <origin xyz="${cal_high_def_x}            ${cal_high_def_y}         ${cal_high_def_z}"
-            rpy="${-M_PI/2+cal_high_def_roll} ${0.0+cal_high_def_pitch} ${-M_PI/2+cal_high_def_yaw}" />
+    <joint name="${name}_optical_fixed_joint" type="fixed">
+      <origin xyz="0 0 0" rpy="0 0 0"/>
+      <parent name="${name}_frame">
+        <origin xyz="${cal_high_def_x}            ${cal_high_def_y}         ${cal_high_def_z}"
+                rpy="${-M_PI/2+cal_high_def_roll} ${0.0+cal_high_def_pitch} ${-M_PI/2+cal_high_def_yaw}" />
+      </parent>
+    </joint>
     <inertial>
       <mass value="0.01" />
-      <com xyz="0 0 0" />
+      <origin xyz="0 0 0" rpy="0 0 0"/>
       <inertia ixx="0.001"  ixy="0.0"  ixz="0.0"
                iyy="0.001"  iyz="0.0"
                izz="0.001" />
     </inertial>
-    <visual>
+    <visual name="${name}_optical_visual">
       <origin xyz="0 0 0" rpy="0 0 0"/>
-      <map name="gazebo_material" flag="gazebo">
-        <elem key="material" value="PR2/Blue" />
-      </map>
-      <geometry name="${name}_optical_visual">
+      <geometry name="${name}_optical_visual_geom">
         <box size="0.01 0.01 0.01" />
       </geometry>
     </visual>
-    <collision>
+    <collision name="${name}_optical_collision">
       <origin xyz="0 0 0" rpy="0 0 0"/>
-      <geometry name="${name}_optical_collision">
+      <geometry name="${name}_optical_collision_geom">
         <box size="0.01 0.01 0.01" />
       </geometry>
     </collision>
   </link>
+  <gazebo name="gazebo_material" reference="${name}_optical_visual">
+    <material value="PR2/Blue" />
+  </gazebo>
 </macro>
 </root>
