Commit message: conversion in progress.
git-svn-id: https://svn.code.sf.net/p/personalrobots/code/pkg/trunk@20436 f5854215-dd47-0410-b2c4-cdd35faa7885

Former-commit-id: 353e65ce82e3b35f4f103577fb292d953ff20473

File: stacks/pr2/pr2_defs/defs/gripper_defs.urdf.xacro (robot description, xacro)
@@ -23,33 +23,32 @@
   <macro name="pr2_finger_limits" params="reflect">
     <limit effort="${finger_joint_effort_limit}" velocity="0.5"
-           min="${gripper_min_angle}" max="${gripper_max_angle}"
-           k_velocity="100.0" k_position="100.0"
-           safety_length_min="0.0" safety_length_max="0.0" />
+           min="${gripper_min_angle}" max="${gripper_max_angle}" />
+    <safety_controller k_velocity="100.0" k_position="100.0"
+                       lower="${gripper_min_angle+0.0}" upper="${gripper_max_angle-0.0}" />
   </macro>
   <macro name="pr2_finger" params="prefix parent">
     <!-- Finger proximal digit -->
-    <joint name="${prefix}_l_finger_joint" type="revolute">
-      <axis xyz="0 0 1" />
-      <anchor xyz="0 0 0" />
-      <calibration reference_position="0" values="1.0 -1.0" />
-      <pr2_finger_limits reflect="1" />
-      <joint_properties damping="${finger_damping}" />
-      <map name="${prefix}_l_finger_joint_feedback" flag="gazebo">
-        <elem key="provideFeedback" value="true"/>
-        <elem key="initialAngle" value="${gripper_min_angle}"/>
-      </map>
-      <map name="${prefix}_l_finger_joint_ode" flag="gazebo">
-        <elem key="stopKd" value="${finger_stop_kd}" />
-        <elem key="stopKp" value="${finger_stop_kp}" />
-        <elem key="fudgeFactor" value="${finger_fudge_factor}" />
-      </map>
-    </joint>
     <link name="${prefix}_l_finger_link">
-      <parent name="${parent}" />
-      <origin xyz="0.07691 0.01 0" rpy="0 0 0" />
-      <joint name="${prefix}_l_finger_joint" />
+      <joint name="${prefix}_l_finger_joint" type="revolute">
+        <origin xyz="0 0 0" rpy="0 0 0" />
+        <axis xyz="0 0 1" />
+        <pr2_finger_limits reflect="1" />
+        <joint_properties damping="${finger_damping}" />
+        <parent name="${parent}">
+          <origin xyz="0.07691 0.01 0" rpy="0 0 0" />
+        </parent>
+        <map name="${prefix}_l_finger_joint_feedback" reference="${prefix}_l_finger_joint">
+          <provideFeedback value="true"/>
+          <initialAngle value="${gripper_min_angle}"/>
+        </map>
+        <map name="${prefix}_l_finger_joint_ode" reference="${prefix}_l_finger_joint">
+          <stopKd value="${finger_stop_kd}" />
+          <stopKp value="${finger_stop_kp}" />
+          <fudgeFactor value="${finger_fudge_factor}" />
+        </map>
+      </joint>
       <inertial>
         <mass value="0.17126" />
-        <com xyz="${0.03598} 0.01730 -0.00164" />
+        <origin xyz="${0.03598} 0.01730 -0.00164" rpy="0 0 0" />
         <inertia  ixx= "0.00007756198"
                   ixy= "0.00000149095"
@@ -59,36 +58,36 @@
                   izz= "0.00018105446" />
       </inertial>
-      <visual>
-        <origin xyz="0 0 0" rpy="0 0 0" />
-        <map name="gazebo_material" flag="gazebo">
-          <elem key="material" value="PR2/Grey" />
-        </map>
-        <geometry name="${prefix}_l_finger_visual">
+      <visual name="${prefix}_l_finger_visual">
+        <origin xyz="0 0 0" rpy="0 0 0" />
+        <map name="gazebo_material" reference="${prefix}_l_finger_visual">
+          <material value="PR2/Grey" />
+        </map>
+        <map name="${prefix}_l_finger_visual_mesh" reference="${prefix}_l_finger_visual">
+          <mesh value="upper_finger_l.mesh" />
+        </map>
+        <geometry name="${prefix}_l_finger_visual_geom">
           <mesh filename="upper_finger_l.stlb" />
         </geometry>
-        <map name="${prefix}_l_finger_visual_mesh" flag="ogre">
-          <elem key="mesh" value="upper_finger_l.mesh" />
-        </map>
-      </visual>
-      <collision>
-        <origin xyz="0 0 0" rpy="0 0 0" />
-        <geometry name="${prefix}_l_finger_collision">
+      </visual>
+      <collision name="${prefix}_l_finger_collision">
+        <origin xyz="0 0 0" rpy="0 0 0" />
+        <geometry name="${prefix}_l_finger_collision_geom">
           <mesh filename="convex/upper_finger_l_convex.stlb" />
         </geometry>
-        <map name="${prefix}_l_finger_collision_mesh" flag="ogre">
-          <elem key="mesh" value="convex/upper_finger_l_convex.mesh" />
+        <map name="${prefix}_l_finger_collision_mesh" reference="${prefix}_l_finger_collision">
+          <mesh value="convex/upper_finger_l_convex.mesh" />
         </map>
         <verbose value="Yes" />
-        <map flag="collision" name="mesh">
-          <elem key="type" value="visual"/>
-        </map>
-        <map name="${prefix}_l_finger_contact" flag="gazebo">
-          <elem key="mu1" value="${finger_mu}" />
-          <elem key="mu2" value="${finger_mu}" />
-          <elem key="kp" value="1000000.0" />
-          <elem key="kd" value="1.0" />
-        </map>
-      </collision>
-      <map name="${prefix}_l_finger_sensor" flag="gazebo">
+        <map reference="${prefix}_l_finger_collision" name="mesh">
+          <type value="visual"/>
+        </map>
+        <map name="${prefix}_l_finger_contact" reference="${prefix}_l_finger_collision">
+          <mu1 value="${finger_mu}" />
+          <mu2 value="${finger_mu}" />
+          <kp value="1000000.0" />
+          <kd value="1.0" />
+        </map>
+      </collision>
+      <map name="${prefix}_l_finger_sensor" reference="${prefix}_l_finger_link">
         <verbatim key="${prefix}_l_finger_bumper_sensor">
           <sensor:contact name="${prefix}_l_finger_contact_sensor">
@@ -104,38 +103,37 @@
         </verbatim>
       </map>
-      <map name="${prefix}_l_finger_gravity" flag="gazebo">
-        <elem key="turnGravityOff">true</elem>
+      <map name="${prefix}_l_finger_gravity" reference="${prefix}_l_finger_link">
+        <turnGravityOff>true</turnGravityOff>
       </map>
     </link>
     <!-- Finger proximal digit -->
-    <joint name="${prefix}_r_finger_joint" type="revolute">
-      <axis xyz="0 0 -1" />
-      <anchor xyz="0 0 0" />
-      <calibration reference_position="0" values="1.0 -1.0" />
-      <pr2_finger_limits reflect="1" />
-      <joint_properties damping="${finger_damping}" />
-      <mimic name="${prefix}_l_finger_joint" mult="1" offset="0"/>
-      <map name="${prefix}_r_finger_mimic" flag="gazebo">
-        <elem key="mimicKp"   value="${finger_kp}" />
-        <elem key="mimicKd"   value="${finger_kd}" />
-        <elem key="mimicFMax" value="${finger_fm}" />
-      </map>
-      <map name="${prefix}_r_finger_options" flag="gazebo">
-        <elem key="provideFeedback" value="true"/>
-        <elem key="initialAngle" value="${-gripper_min_angle}"/>
-      </map>
-      <map name="${prefix}_r_finger_joint_ode" flag="gazebo">
-        <elem key="stopKd" value="${finger_stop_kd}" />
-        <elem key="stopKp" value="${finger_stop_kp}" />
-        <elem key="fudgeFactor" value="${finger_fudge_factor}" />
-      </map>
-    </joint>
     <link name="${prefix}_r_finger_link">
-      <parent name="${parent}" />
-      <origin xyz="0.07691 -0.01 0" rpy="0 0 0" />
-      <joint name="${prefix}_r_finger_joint" />
+      <joint name="${prefix}_r_finger_joint" type="revolute">
+        <axis xyz="0 0 -1" />
+        <anchor xyz="0 0 0" />
+        <pr2_finger_limits reflect="1" />
+        <joint_properties damping="${finger_damping}" />
+        <mimic name="${prefix}_l_finger_joint" mult="1" offset="0"/>
+        <map name="${prefix}_r_finger_mimic" reference="${prefix}_r_finger_joint">
+          <mimicKp   value="${finger_kp}" />
+          <mimicKd   value="${finger_kd}" />
+          <mimicFMax value="${finger_fm}" />
+        </map>
+        <map name="${prefix}_r_finger_options" reference="${prefix}_r_finger_joint">
+          <provideFeedback value="true"/>
+          <initialAngle value="${-gripper_min_angle}"/>
+        </map>
+        <map name="${prefix}_r_finger_joint_ode" reference="${prefix}_r_finger_joint">
+          <stopKd value="${finger_stop_kd}" />
+          <stopKp value="${finger_stop_kp}" />
+          <fudgeFactor value="${finger_fudge_factor}" />
+        </map>
+        <parent name="${parent}">
+          <origin xyz="0.07691 -0.01 0" rpy="0 0 0" />
+        </parent>
+      </joint>
       <inertial>
         <mass value="0.17389" />
-        <com xyz="${0.03576} -0.01736 -0.00095" />
+        <origin xyz="${0.03576} -0.01736 -0.00095" rpy="0 0 0" />
         <inertia  ixx= "0.00007738410"
                   ixy="-0.00000209309"
@@ -145,36 +143,36 @@
                   izz= "0.00018106988" />
       </inertial>
-      <visual>
-        <origin xyz="0 0 0" rpy="0 0 0" />
-        <map name="gazebo_material" flag="gazebo">
-          <elem key="material" value="PR2/Grey" />
-        </map>
-        <geometry name="${prefix}_r_finger_visual">
+      <visual name="${prefix}_r_finger_visual">
+        <origin xyz="0 0 0" rpy="0 0 0" />
+        <map name="gazebo_material" reference="${prefix}_r_finger_visual">
+          <material value="PR2/Grey" />
+        </map>
+        <map name="${prefix}_r_finger_visual_mesh" reference="${prefix}_r_finger_visual">
+          <mesh value="upper_finger_r.mesh" />
+        </map>
+        <geometry name="${prefix}_r_finger_visual_geom">
           <mesh filename="upper_finger_r.stlb" />
         </geometry>
-        <map name="${prefix}_r_finger_visual_mesh" flag="ogre">
-          <elem key="mesh" value="upper_finger_r.mesh" />
-        </map>
-      </visual>
-      <collision>
-        <origin xyz="0 0 0" rpy="0 0 0" />
-        <geometry name="${prefix}_r_finger_collision">
+      </visual>
+      <collision name="${prefix}_r_finger_collision">
+        <origin xyz="0 0 0" rpy="0 0 0" />
+        <geometry name="${prefix}_r_finger_collision_geom">
           <mesh filename="convex/upper_finger_r_convex.stlb" />
         </geometry>
-        <map name="${prefix}_r_finger_collision_mesh" flag="ogre">
-          <elem key="mesh" value="convex/upper_finger_r_convex.mesh" />
-        </map>
         <verbose value="Yes" />
-        <map flag="collision" name="mesh">
-          <elem key="type" value="visual"/>
-        </map>
-        <map name="${prefix}_r_finger_contact" flag="gazebo">
-          <elem key="mu1" value="${finger_mu}" />
-          <elem key="mu2" value="${finger_mu}" />
-          <elem key="kp" value="1000000.0" />
-          <elem key="kd" value="1.0" />
-        </map>
-      </collision>
-      <map name="${prefix}_r_finger_sensor" flag="gazebo">
+        <map name="${prefix}_r_finger_collision_mesh" reference="${prefix}_r_finger_collision">
+          <mesh value="convex/upper_finger_r_convex.mesh" />
+        </map>
+        <map name="mesh" reference="${prefix}_r_finger_collision">
+          <type value="visual"/>
+        </map>
+        <map name="${prefix}_r_finger_contact" reference="${prefix}_r_finger_collision">
+          <mu1 value="${finger_mu}" />
+          <mu2 value="${finger_mu}" />
+          <kp value="1000000.0" />
+          <kd value="1.0" />
+        </map>
+      </collision>
+      <map name="${prefix}_r_finger_sensor" reference="${prefix}_r_finger_link">
         <verbatim key="${prefix}_r_finger_bumper_sensor">
           <sensor:contact name="${prefix}_r_finger_contact_sensor">
@@ -190,74 +188,73 @@
         </verbatim>
       </map>
-      <map name="${prefix}_r_finger_gravity" flag="gazebo">
-        <elem key="turnGravityOff">true</elem>
+      <map name="${prefix}_r_finger_gravity" reference="${prefix}_r_finger_link">
+        <turnGravityOff>true</turnGravityOff>
       </map>
     </link>
     <!-- Finger tip -->
-    <joint name="${prefix}_l_finger_tip_joint" type="revolute">
-      <axis xyz="0 0 -1" />
-      <anchor xyz="0 0 0" />
-      <calibration reference_position="0" values="1.0 -1.0" />
-      <pr2_finger_limits reflect="1" />
-      <joint_properties damping="${finger_tip_damping}" />
-      <mimic name="${prefix}_l_finger_joint" mult="1" offset="0"/>
-      <map name="${prefix}_l_finger_tip_mimic" flag="gazebo">
-        <elem key="mimicKp"   value="${finger_tip_kp}" />
-        <elem key="mimicKd"   value="${finger_tip_kd}" />
-        <elem key="mimicFMax" value="${finger_tip_fm}" />
-      </map>
-      <map name="${prefix}_l_finger_tip_options" flag="gazebo">
-        <elem key="provideFeedback" value="true"/>
-        <elem key="initialAngle" value="${-gripper_min_angle}"/>
-      </map>
-      <map name="${prefix}_l_finger_tip_joint_ode" flag="gazebo">
-        <elem key="stopKd" value="${finger_stop_kd}" />
-        <elem key="stopKp" value="${finger_stop_kp}" />
-        <elem key="fudgeFactor" value="${finger_fudge_factor}" />
-      </map>
-    </joint>
     <link name="${prefix}_l_finger_tip_link">
-      <parent name="${prefix}_l_finger_link" />
-      <origin xyz="0.09137 0.00495 0" rpy="0 0 0" />
-      <joint name="${prefix}_l_finger_tip_joint" />
+      <joint name="${prefix}_l_finger_tip_joint" type="revolute">
+        <axis xyz="0 0 -1" />
+        <anchor xyz="0 0 0" />
+        <pr2_finger_limits reflect="1" />
+        <joint_properties damping="${finger_tip_damping}" />
+        <mimic name="${prefix}_l_finger_joint" mult="1" offset="0"/>
+        <map name="${prefix}_l_finger_tip_mimic" reference="${prefix}_l_finger_tip_link">
+          <mimicKp   value="${finger_tip_kp}" />
+          <mimicKd   value="${finger_tip_kd}" />
+          <mimicFMax value="${finger_tip_fm}" />
+        </map>
+        <map name="${prefix}_l_finger_tip_options" reference="${prefix}_l_finger_tip_link">
+          <provideFeedback value="true"/>
+          <initialAngle value="${-gripper_min_angle}"/>
+        </map>
+        <map name="${prefix}_l_finger_tip_joint_ode" reference="${prefix}_l_finger_tip_link">
+          <stopKd value="${finger_stop_kd}" />
+          <stopKp value="${finger_stop_kp}" />
+          <fudgeFactor value="${finger_fudge_factor}" />
+        </map>
+        <parent name="${prefix}_l_finger_link">
+          <origin xyz="0.09137 0.00495 0" rpy="0 0 0" />
+        </parent>
+      </joint>
       <inertial>
         <mass value="0.04419" />
-        <com xyz="0.00423 0.00284 0.0" />
+        <origin xyz="0.00423 0.00284 0.0" rpy="0 0 0" />
         <inertia  ixx="0.00000837047" ixy="0.00000583632" ixz="0.0"
                   iyy="0.00000987067" iyz="0.0"
                   izz="0.00001541768" />
       </inertial>
-      <visual>
-        <origin xyz="0 0 0" rpy="0 0 0" />
-        <map name="gazebo_material" flag="gazebo">
-          <elem key="material" value="PR2/Green" />
-        </map>
-        <geometry name="${prefix}_l_finger_tip_visual">
+      <visual name="${prefix}_l_finger_tip_visual">
+        <origin xyz="0 0 0" rpy="0 0 0" />
+        <map name="gazebo_material" reference="${prefix}_l_finger_tip_visual">
+          <material value="PR2/Green" />
+        </map>
+        <geometry name="${prefix}_l_finger_tip_visual_geom">
           <mesh filename="finger_tip_l.stlb" />
         </geometry>
-        <map name="${prefix}_l_finger_tip_visual_mesh" flag="ogre">
-          <elem key="mesh" value="finger_tip_l.mesh" />
-        </map>
-      </visual>
-      <collision>
-        <origin xyz="0 0 0" rpy="0 0 0" />
-        <geometry name="${prefix}_l_finger_tip_collision">
+        <map name="${prefix}_l_finger_tip_visual_mesh" reference="${prefix}_l_finger_tip_visual">
+          <mesh value="finger_tip_l.mesh" />
+        </map>
+      </visual>
+      <collision name="${prefix}_l_finger_tip_collision">
+        <origin xyz="0 0 0" rpy="0 0 0" />
+        <geometry name="${prefix}_l_finger_tip_collision_geom">
           <mesh filename="convex/finger_tip_l_convex.stlb" />
         </geometry>
-        <map name="${prefix}_l_finger_tip_collision_mesh" flag="ogre">
-          <elem key="mesh" value="convex/finger_tip_l_convex.mesh" />
+        <map name="${prefix}_l_finger_tip_collision_mesh" reference="${prefix}_l_finger_tip_collision">
+          <mesh value="convex/finger_tip_l_convex.mesh" />
         </map>
         <verbose value="Yes" />
-        <map flag="collision" name="mesh">
-          <elem key="type" value="visual"/>
-        </map>
-        <map name="${prefix}_l_finger_tip_contact" flag="gazebo">
-          <elem key="mu1" value="${finger_tip_mu}" />
-          <elem key="mu2" value="${finger_tip_mu}" />
-          <elem key="kp"  value="10000000.0" />
-          <elem key="kd"  value="1.0" />
-        </map>
-      </collision>
-      <map name="${prefix}_l_finger_tip_sensor" flag="gazebo">
+        <map reference="${prefix}_l_finger_tip_collision" name="mesh">
+          <type value="visual"/>
+        </map>
+        <map name="${prefix}_l_finger_tip_contact" reference="${prefix}_l_finger_tip_collision">
+          <mu1 value="${finger_tip_mu}" />
+          <mu2 value="${finger_tip_mu}" />
+          <kp  value="10000000.0" />
+          <kd  value="1.0" />
+        </map>
+      </collision>
+      <map name="${prefix}_l_finger_tip_sensor" reference="${prefix}_l_finger_tip_link">
         <verbatim key="${prefix}_l_finger_tip_bumper_sensor">
           <sensor:contact name="${prefix}_l_finger_tip_contact_sensor">
@@ -273,75 +270,74 @@
         </verbatim>
       </map>
-      <map name="${prefix}_l_finger_tip_gravity" flag="gazebo">
-        <elem key="turnGravityOff">true</elem>
-        <elem key="selfCollide" value="false" />
+      <map name="${prefix}_l_finger_tip_gravity" reference="${prefix}_l_finger_tip_link">
+        <turnGravityOff>true</mimicKp>
+        <selfCollide value="false" />
       </map>
     </link>
     <!-- Finger tip -->
-    <joint name="${prefix}_r_finger_tip_joint" type="revolute">
-      <axis xyz="0 0 1" />
-      <anchor xyz="0 0 0" />
-      <calibration reference_position="0" values="1.0 -1.0" />
-      <pr2_finger_limits reflect="1" />
-      <joint_properties damping="${finger_tip_damping}" />
-      <mimic name="${prefix}_l_finger_joint" mult="1" offset="0"/>
-      <map name="${prefix}_r_finger_tip_mimic" flag="gazebo">
-        <elem key="mimicKp"   value="${finger_tip_kp}" />
-        <elem key="mimicKd"   value="${finger_tip_kd}" />
-        <elem key="mimicFMax" value="${finger_tip_fm}" />
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