Commit message: conversion in progress.
git-svn-id: https://svn.code.sf.net/p/personalrobots/code/pkg/trunk@20436 f5854215-dd47-0410-b2c4-cdd35faa7885

Former-commit-id: 353e65ce82e3b35f4f103577fb292d953ff20473

File: stacks/pr2/pr2_defs/defs/head_defs.urdf.xacro (robot description, xacro)
@@ -5,39 +5,37 @@
   <property name="M_PI" value="3.1415926535897931" />
   <macro name="pr2_tilting_laser" params="name parent *origin">
-    <joint name="${name}_mount_joint" type="revolute">
-      <axis xyz="0 1 0" />
-      <anchor xyz="0 0 0" />
-      <limit min="-0.785" max="1.57" effort="0.5292" velocity="100"
-             k_position="100" k_velocity="0.05"
-             safety_length_min="0.0" safety_length_max="0.0" />
-      <calibration reference_position="-0.35" values="0 0" />
-      <joint_properties damping="0.008" />
-    </joint>
     <link name="${name}_mount_link">
-      <parent name="${parent}" />
-      <insert_block name="origin" />
-      <joint name="${name}_mount_joint" />
+      <joint name="${name}_mount_joint" type="revolute">
+        <axis xyz="0 1 0" />
+        <anchor xyz="0 0 0" />
+        <limit min="-0.785" max="1.57" effort="0.5292" velocity="100" />
+        <safety_controller k_position="100" k_velocity="0.05" lower="${-0.785+0.0}" upper="${1.57-0.0}" />
+        <joint_properties damping="0.008" />
+        <parent name="${parent}">
+          <insert_block name="origin" />
+        </parent>
+      </joint>
       <inertial>
         <mass value="0.05" />
-        <com xyz="-0.03 0 -0.03" />
+        <origin xyz="-0.03 0 -0.03" rpy="0 0 0" />
         <inertia ixx="0.0001" ixy="0" ixz="0"
-		 iyy="0.00001" iyz="0"
-		 izz="0.0001" />
-      </inertial>
-      <visual>
-        <origin xyz="0 0 0" rpy="0 0 0" />
-        <map name="gazebo_material" flag="gazebo">
-          <elem key="material" value="PR2/Red" />
-        </map>
-        <geometry name="${name}_mount_visual">
+                 iyy="0.00001" iyz="0"
+                 izz="0.0001" />
+      </inertial>
+      <visual name="${name}_mount_visual">
+        <origin xyz="0 0 0" rpy="0 0 0" />
+        <map name="gazebo_material" reference="${name}_mount_visual">
+          <material value="PR2/Red" />
+        </map>
+        <geometry name="${name}_mount_visual_geom">
           <mesh filename="hok_tilt.stlb" />
         </geometry>
-        <map name="${name}_mount_visual_mesh" flag="ogre">
-          <elem key="mesh" value="hok_tilt.mesh" />
-        </map>
-      </visual>
-      <collision>
-        <origin xyz="0 0 0" rpy="0 0 0" />
-        <geometry name="${name}_mount_collision" >
+        <map name="${name}_mount_visual_mesh" reference="${name}_mount_visual">
+          <mesh value="hok_tilt.mesh" />
+        </map>
+      </visual>
+      <collision name="${name}_mount_collision">
+        <origin xyz="0 0 0" rpy="0 0 0" />
+        <geometry name="${name}_mount_collision_geom" >
           <box size=".001 .001 .001" />
         </geometry>
@@ -48,31 +46,32 @@
       <joint name="${name}_mount_joint" />
       <mechanicalReduction>6.0</mechanicalReduction>
+      <calibration reference_position="-0.35" values="0 0" />
     </transmission>
-    <joint name="${name}_joint" type="fixed">
-      <axis xyz="0 1 0" />
-      <anchor xyz="0 0 0" />
-    </joint>
     <link name="${name}_link" type="laser">
-      <parent name="${name}_mount_link" />
-      <origin xyz="0 0 0.03" rpy="0 0 0" />
-      <joint name="${name}_joint" />
+      <joint name="${name}_joint" type="fixed">
+        <axis xyz="0 1 0" />
+        <anchor xyz="0 0 0" />
+        <parent name="${name}_mount_link">
+          <origin xyz="0 0 0.03" rpy="0 0 0" />
+        </parent>
+      </joint>
       <inertial>
         <mass value="0.001" />
-        <com xyz="0 0 0" />
+        <origin xyz="0 0 0" rpy="0 0 0" />
         <inertia ixx="0.0001" ixy="0" ixz="0" iyy="0.000001" iyz="0" izz="0.0001" />
       </inertial>
-      <visual>
-        <origin xyz="0 0 0" rpy="0 0 0" />
-        <geometry name="${name}_visual">
+      <visual name="${name}_visual">
+        <origin xyz="0 0 0" rpy="0 0 0" />
+        <geometry name="${name}_visual_geom">
           <box size="0.001 0.001 0.001" />
         </geometry>
       </visual>
-      <collision>
-        <origin xyz="0 0 0" rpy="0 0 0" />
-        <geometry name="${name}_collision" >
+      <collision name="${name}_collision">
+        <origin xyz="0 0 0" rpy="0 0 0" />
+        <geometry name="${name}_collision_geom" >
           <box size=".001 .001 .001" />
         </geometry>
       </collision>
-      <map name="sensor" flag="gazebo">
+      <map name="sensor" reference="${name}_link">
         <verbatim key="sensor_${name}_ray">
           <sensor:ray name="${name}">
@@ -116,29 +115,30 @@
   <!-- When mounted properly, should have same origin as head plate frame -->
   <macro name="pr2_head_sensor_package" params="name hd_name stereo_name parent *origin">
-    <joint name="${name}_fixed_joint" type="fixed" />
     <link name="${name}_link" >
-      <parent name="${parent}" />
-      <insert_block name="origin" />
-      <joint name="${name}_fixed_joint" />
-      <inertial>
-	<!-- Needs verification with CAD -->
-	<mass value="0.05" />
-	<com xyz="0 0 0" />
-	<inertia ixx="0.001" ixy="0.0" ixz="0.0"
-		 iyy="0.001" iyz="0.0" izz="0.01" />
+      <joint name="${name}_fixed_joint" type="fixed">
+        <parent name="${parent}">
+          <insert_block name="origin" />
+        </parent>
+      </joint>
+      <inertial>
+        <!-- Needs verification with CAD -->
+        <mass value="0.05" />
+        <origin xyz="0 0 0" rpy="0 0 0" />
+        <inertia ixx="0.001" ixy="0.0" ixz="0.0"
+                 iyy="0.001" iyz="0.0" izz="0.01" />
       </inertial>
       <!-- Should probably get real visuals here at some point -->
-      <visual>
-        <origin xyz="0 0 0" rpy="0 0 0" />
-        <map name="gazebo_material" flag="gazebo">
-          <elem key="material" value="PR2/Blue" />
-        </map>
-        <geometry name="${name}_sensor_visual">
-          <box size="0.01 0.01 0.01" />
-        </geometry>
-      </visual>
-      <collision>
-        <origin xyz="0 0 0" rpy="0 0 0" />
-        <geometry name="${name}_sensor_collision">
+      <visual name="${name}_sensor_visual">
+        <origin xyz="0 0 0" rpy="0 0 0" />
+        <map name="gazebo_material" reference="${name}_sensor_visual">
+          <material value="PR2/Blue" />
+        </map>
+        <geometry name="${name}_sensor_visual_geom">
+          <box size="0.01 0.01 0.01" />
+        </geometry>
+      </visual>
+      <collision name="${name}_sensor_collision">
+        <origin xyz="0 0 0" rpy="0 0 0" />
+        <geometry name="${name}_sensor_collision_geom">
           <box size="0.01 0.01 0.01" />
         </geometry>
@@ -147,6 +147,6 @@
     <!-- Prosilica Camera -->
     <prosilica_cam name="${hd_name}" parent="${name}_link" >
-    <!-- Center of camera is 109mm right of center screw, 35mm up -->
-    <!-- Camera is slightly recessed from front, where is camera origin? Lens? -->
+      <!-- Center of camera is 109mm right of center screw, 35mm up -->
+      <!-- Camera is slightly recessed from front, where is camera origin? Lens? -->
       <origin xyz="0 -0.109 0.035" rpy="0 0 0" />
     </prosilica_cam>
@@ -160,29 +160,30 @@
   <macro name="double_stereo_camera" params="name parent *origin">
     <!-- Define link to stereo cameras, set origin relative to that -->
-    <joint name="${name}_fixed_joint" type="fixed" />
     <link name="${name}_link">
-      <parent name="${parent}" />
-      <insert_block name="origin" />
-      <joint name="${name}_fixed_joint" />
-      <inertial>
-	<!-- Needs verification with CAD -->
-	<mass value="0.1" />
-	<com xyz="0 0 0" />
-	<inertia ixx="0.001" ixy="0.0" ixz="0.0"
-		 iyy="0.001" iyz="0.0" izz="0.01" />
+      <joint name="${name}_fixed_joint" type="fixed">
+        <parent name="${parent}">
+          <insert_block name="origin" />
+        </parent>
+      </joint>
+      <inertial>
+        <!-- Needs verification with CAD -->
+        <mass value="0.1" />
+        <origin xyz="0 0 0" rpy="0 0 0" />
+        <inertia ixx="0.001" ixy="0.0" ixz="0.0"
+                 iyy="0.001" iyz="0.0" izz="0.01" />
       </inertial>
       <!-- Should probably get real visuals here at some point -->
-      <visual>
-        <origin xyz="0 0 0" rpy="0 0 0" />
-        <map name="gazebo_material" flag="gazebo">
-          <elem key="material" value="PR2/Blue" />
-        </map>
-        <geometry name="${name}_double_stereo_visual">
-          <box size="0.01 0.01 0.01" />
-        </geometry>
-      </visual>
-      <collision>
-        <origin xyz="0 0 0" rpy="0 0 0" />
-        <geometry name="${name}_double_stereo_collision">
+      <visual name="${name}_double_stereo_visual">
+        <origin xyz="0 0 0" rpy="0 0 0" />
+        <map name="gazebo_material" reference="${name}_double_stereo_visual">
+          <material value="PR2/Blue" />
+        </map>
+        <geometry name="${name}_double_stereo_visual_geom">
+          <box size="0.01 0.01 0.01" />
+        </geometry>
+      </visual>
+      <collision name="${name}_double_stereo_collision">
+        <origin xyz="0 0 0" rpy="0 0 0" />
+        <geometry name="${name}_double_stereo_collision_geom">
           <box size="0.01 0.01 0.01" />
         </geometry>
@@ -199,88 +200,91 @@
   </macro>
   <macro name="stereo_camera" params="name parent *origin">
-    <joint name="${name}_fixed_joint" type="fixed" />
     <link name="${name}_link">
-      <parent name="${parent}" />
-      <insert_block name="origin" />
-      <joint name="${name}_fixed_joint" />
+      <joint name="${name}_fixed_joint" type="fixed">
+        <parent name="${parent}">
+          <insert_block name="origin" />
+        </parent>
+      </joint>
       <inertial>
         <mass value="0.1" />
-        <com xyz="0 0 0" />
+        <origin xyz="0 0 0" rpy="0 0 0" />
         <inertia ixx="0.00482611007"  ixy="-0.000144683999"  ixz="0.000110076136"
                  iyy="0.005218991412"  iyz="-0.000314239509"  izz="0.008618784925" />
       </inertial>
-      <visual>
+      <visual name="${name}_visual">
         <origin xyz="${stereo_center_box_center_offset_x} 0 ${stereo_center_box_center_offset_z}" rpy="0 0 0" />
-        <map name="gazebo_material" flag="gazebo">
-          <elem key="material" value="PR2/Blue" />
-        </map>
-        <geometry name="${name}_visual">
+        <map name="gazebo_material" reference="${name}_visual">
+          <material value="PR2/Blue" />
+        </map>
+        <geometry name="${name}_visual_geom">
           <box size="${stereo_size_x} ${stereo_size_y} ${stereo_size_z}" />
         </geometry>
       </visual>
-      <collision>
+      <collision name="${name}_collision">
         <origin xyz="${stereo_center_box_center_offset_x} 0 ${stereo_center_box_center_offset_z}" rpy="0 0 0" />
-        <geometry name="${name}_collision">
+        <geometry name="${name}_collision_geom">
           <box size="${stereo_size_x} ${stereo_size_y} ${stereo_size_z}" />
         </geometry>
       </collision>
     </link>
-    <joint name="${name}_optical_fixed_joint" type="fixed" />
     <link name="${name}_optical_frame" type="camera">
-      <parent name="${name}_link" />
-      <origin xyz="${cal_stereo_x}            ${0.045+cal_stereo_y}   ${.0305+cal_stereo_z}"
-              rpy="${-M_PI/2+cal_stereo_roll} ${0.0+cal_stereo_pitch} ${-M_PI/2+cal_stereo_yaw}" />
-      <joint name="${name}_optical_fixed_joint" />
+      <joint name="${name}_optical_fixed_joint" type="fixed">
+        <parent name="${name}_link">
+          <origin xyz="${cal_stereo_x}            ${0.045+cal_stereo_y}   ${.0305+cal_stereo_z}"
+                  rpy="${-M_PI/2+cal_stereo_roll} ${0.0+cal_stereo_pitch} ${-M_PI/2+cal_stereo_yaw}" />
+        </parent>
+      </joint>
       <inertial>
         <mass value="0.01" />
-        <com xyz="0 0 0" />
+        <origin xyz="0 0 0" rpy="0 0 0" />
         <inertia ixx="0.001"  ixy="0.0"  ixz="0.0"
                  iyy="0.001"  iyz="0.0"
                  izz="0.001" />
       </inertial>
-      <visual>
-        <origin xyz="0 0 0" rpy="0 0 0" />
-        <map name="gazebo_material" flag="gazebo">
-          <elem key="material" value="PR2/Blue" />
-        </map>
-        <geometry name="${name}_optical_fixed_visual">
-          <box size="0.01 0.01 0.01" />
-        </geometry>
-      </visual>
-      <collision>
-        <origin xyz="0 0 0" rpy="0 0 0" />
-        <geometry name="${name}_optical_fixed_collision">
-          <box size="0.01 0.01 0.01" />
-        </geometry>
-      </collision>
-    </link>
-    <joint name="${name}_l_stereo_camera_fixed_joint" type="fixed" />
+      <visual name="${name}_optical_fixed_visual">
+        <origin xyz="0 0 0" rpy="0 0 0" />
+        <map name="gazebo_material" reference="${name}_optical_fixed_visual">
+          <material value="PR2/Blue" />
+        </map>
+        <geometry name="${name}_optical_fixed_visual_geom">
+          <box size="0.01 0.01 0.01" />
+        </geometry>
+      </visual>
+      <collision name="${name}_optical_fixed_collision">
+        <origin xyz="0 0 0" rpy="0 0 0" />
+        <geometry name="${name}_optical_fixed_collision_geom">
+          <box size="0.01 0.01 0.01" />
+        </geometry>
+      </collision>
+    </link>
     <link name="${name}_l_stereo_camera_frame">
-      <parent name="${name}_optical_frame" />
-      <origin xyz="0 0 0" rpy="0 ${-M_PI/2} ${M_PI/2}" />
-      <joint name="${name}_l_stereo_camera_fixed_joint" />
+      <joint name="${name}_l_stereo_camera_fixed_joint" type="fixed">
+        <parent name="${name}_optical_frame">
+          <origin xyz="0 0 0" rpy="0 ${-M_PI/2} ${M_PI/2}" />
+        </parent>
+      </joint>
       <inertial>
         <mass value="0.01" />
-        <com xyz="0 0 0" />
+        <origin xyz="0 0 0" rpy="0 0 0" />
         <inertia ixx="0.001" ixy="0.000"  ixz="0.000"
                  iyy="0.001" iyz="0.000"
                  izz="0.001" />
       </inertial>
-      <visual>
-        <origin xyz="0 0 0" rpy="0 0 0" />
-        <map name="gazebo_material" flag="gazebo">
-          <elem key="material" value="PR2/Blue" />
-        </map>
-        <geometry name="${name}_l_stereo_camera_visual">
-          <box size="0.01 0.01 0.01" />
-        </geometry>
-      </visual>
-      <collision>
-        <origin xyz="0 0 0" rpy="0 0 0" />
-        <geometry name="${name}_l_stereo_camera_collision">
-          <box size="0.01 0.01 0.01" />
-        </geometry>
-      </collision>
-      <map name="sensor" flag="gazebo">
+      <visual name="${name}_l_stereo_camera_visual">
+        <origin xyz="0 0 0" rpy="0 0 0" />
+        <map name="gazebo_material" reference="${name}_l_stereo_camera_visual">
+          <material value="PR2/Blue" />
+        </map>
+        <geometry name="${name}_l_stereo_camera_visual_geom">
+          <box size="0.01 0.01 0.01" />
+        </geometry>
+      </visual>
+      <collision name="${name}_l_stereo_camera_collision">
+        <origin xyz="0 0 0" rpy="0 0 0" />
+        <geometry name="${name}_l_stereo_camera_collision_geom">
+          <box size="0.01 0.01 0.01" />
+        </geometry>
+      </collision>
+      <map name="sensor" reference="${name}_l_stereo_camera_frame">
         <verbatim key="sensor_${name}_l_camera">
           <sensor:camera name="${name}_l_sensor">
@@ -299,36 +303,37 @@
             </controller:ros_camera>
           </sensor:camera>
-       	</verbatim>
+        </verbatim>
       </map>
     </link>
-    <joint name="${name}_r_stereo_camera_fixed_joint" type="fixed" />
     <link name="${name}_r_stereo_camera_frame">
-      <parent name="${name}_l_stereo_camera_frame" />
-      <origin xyz="${stereo_dx} ${stereo_dy} ${stereo_dz}"
-              rpy="${stereo_rx} ${stereo_ry} ${stereo_rz}" />
-      <joint name="${name}_r_stereo_camera_fixed_joint" />
+      <joint name="${name}_r_stereo_camera_fixed_joint" type="fixed">
+        <parent name="${name}_l_stereo_camera_frame">
+          <origin xyz="${stereo_dx} ${stereo_dy} ${stereo_dz}"
+                  rpy="${stereo_rx} ${stereo_ry} ${stereo_rz}" />
+        </parent>
+      </joint>
       <inertial>
         <mass value="0.01" />
-        <com xyz="0 0 0" />
+        <origin xyz="0 0 0" rpy="0 0 0" />
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