Commit message: converting urdf.
git-svn-id: https://svn.code.sf.net/p/personalrobots/code/pkg/trunk@20437 f5854215-dd47-0410-b2c4-cdd35faa7885

Former-commit-id: a4873532359b68515d694d29f9b2b1a5fb2de4b3

File: stacks/pr2/pr2_defs/defs/gripper_defs.urdf.xacro (robot description, xacro)
@@ -38,13 +38,4 @@
           <origin xyz="0.07691 0.01 0" rpy="0 0 0" />
         </parent>
-        <map name="${prefix}_l_finger_joint_feedback" reference="${prefix}_l_finger_joint">
-          <provideFeedback value="true"/>
-          <initialAngle value="${gripper_min_angle}"/>
-        </map>
-        <map name="${prefix}_l_finger_joint_ode" reference="${prefix}_l_finger_joint">
-          <stopKd value="${finger_stop_kd}" />
-          <stopKp value="${finger_stop_kp}" />
-          <fudgeFactor value="${finger_fudge_factor}" />
-        </map>
       </joint>
       <inertial>
@@ -60,10 +51,4 @@
       <visual name="${prefix}_l_finger_visual">
         <origin xyz="0 0 0" rpy="0 0 0" />
-        <map name="gazebo_material" reference="${prefix}_l_finger_visual">
-          <material value="PR2/Grey" />
-        </map>
-        <map name="${prefix}_l_finger_visual_mesh" reference="${prefix}_l_finger_visual">
-          <mesh value="upper_finger_l.mesh" />
-        </map>
         <geometry name="${prefix}_l_finger_visual_geom">
           <mesh filename="upper_finger_l.stlb" />
@@ -75,36 +60,49 @@
           <mesh filename="convex/upper_finger_l_convex.stlb" />
         </geometry>
-        <map name="${prefix}_l_finger_collision_mesh" reference="${prefix}_l_finger_collision">
-          <mesh value="convex/upper_finger_l_convex.mesh" />
-        </map>
         <verbose value="Yes" />
-        <map reference="${prefix}_l_finger_collision" name="mesh">
-          <type value="visual"/>
-        </map>
-        <map name="${prefix}_l_finger_contact" reference="${prefix}_l_finger_collision">
-          <mu1 value="${finger_mu}" />
-          <mu2 value="${finger_mu}" />
-          <kp value="1000000.0" />
-          <kd value="1.0" />
-        </map>
-      </collision>
-      <map name="${prefix}_l_finger_sensor" reference="${prefix}_l_finger_link">
-        <verbatim key="${prefix}_l_finger_bumper_sensor">
-          <sensor:contact name="${prefix}_l_finger_contact_sensor">
-            <geom>${prefix}_l_finger_collision</geom>
-            <updateRate>100.0</updateRate>
-            <controller:ros_bumper name="${prefix}_l_finger_ros_bumper_controller" plugin="libros_bumper.so">
-              <alwaysOn>true</alwaysOn>
-              <updateRate>100.0</updateRate>
-              <bumperTopicName>${prefix}_l_finger_bumper</bumperTopicName>
-              <interface:bumper name="${prefix}_l_finger_ros_bumper_iface" />
-            </controller:ros_bumper>
-          </sensor:contact>
-        </verbatim>
-      </map>
-      <map name="${prefix}_l_finger_gravity" reference="${prefix}_l_finger_link">
-        <turnGravityOff>true</turnGravityOff>
-      </map>
-    </link>
+      </collision>
+    </link>
+    <gazebo name="${prefix}_l_finger_gravity" reference="${prefix}_l_finger_link">
+      <turnGravityOff>true</turnGravityOff>
+    </gazebo>
+    <gazebo name="${prefix}_l_finger_sensor" reference="${prefix}_l_finger_link">
+      <sensor:contact name="${prefix}_l_finger_contact_sensor">
+        <geom>${prefix}_l_finger_collision</geom>
+        <updateRate>100.0</updateRate>
+        <controller:ros_bumper name="${prefix}_l_finger_ros_bumper_controller" plugin="libros_bumper.so">
+          <alwaysOn>true</alwaysOn>
+          <updateRate>100.0</updateRate>
+          <bumperTopicName>${prefix}_l_finger_bumper</bumperTopicName>
+          <interface:bumper name="${prefix}_l_finger_ros_bumper_iface" />
+        </controller:ros_bumper>
+      </sensor:contact>
+    </gazebo>
+    <gazebo name="${prefix}_l_finger_contact" reference="${prefix}_l_finger_collision">
+      <mu1 value="${finger_mu}" />
+      <mu2 value="${finger_mu}" />
+      <kp value="1000000.0" />
+      <kd value="1.0" />
+    </gazebo>
+    <gazebo name="gazebo_material" reference="${prefix}_l_finger_visual">
+      <material value="PR2/Grey" />
+    </gazebo>
+    <gazebo name="${prefix}_l_finger_joint_ode" reference="${prefix}_l_finger_joint">
+      <stopKd value="${finger_stop_kd}" />
+      <stopKp value="${finger_stop_kp}" />
+      <fudgeFactor value="${finger_fudge_factor}" />
+    </gazebo>
+    <gazebo name="${prefix}_l_finger_joint_feedback" reference="${prefix}_l_finger_joint">
+      <provideFeedback value="true"/>
+      <initialAngle value="${gripper_min_angle}"/>
+    </gazebo>
+    <ogre reference="${prefix}_l_finger_collision" name="mesh" reference="${prefix}_l_finger_collision">
+      <type value="visual"/>
+    </ogre>
+    <ogre name="${prefix}_l_finger_collision_mesh" reference="${prefix}_l_finger_collision">
+      <mesh value="convex/upper_finger_l_convex.mesh" />
+    </ogre>
+    <ogre name="${prefix}_l_finger_visual_mesh" reference="${prefix}_l_finger_visual">
+      <mesh value="upper_finger_l.mesh" />
+    </ogre>
     <!-- Finger proximal digit -->
     <link name="${prefix}_r_finger_link">
@@ -115,18 +113,4 @@
         <joint_properties damping="${finger_damping}" />
         <mimic name="${prefix}_l_finger_joint" mult="1" offset="0"/>
-        <map name="${prefix}_r_finger_mimic" reference="${prefix}_r_finger_joint">
-          <mimicKp   value="${finger_kp}" />
-          <mimicKd   value="${finger_kd}" />
-          <mimicFMax value="${finger_fm}" />
-        </map>
-        <map name="${prefix}_r_finger_options" reference="${prefix}_r_finger_joint">
-          <provideFeedback value="true"/>
-          <initialAngle value="${-gripper_min_angle}"/>
-        </map>
-        <map name="${prefix}_r_finger_joint_ode" reference="${prefix}_r_finger_joint">
-          <stopKd value="${finger_stop_kd}" />
-          <stopKp value="${finger_stop_kp}" />
-          <fudgeFactor value="${finger_fudge_factor}" />
-        </map>
         <parent name="${parent}">
           <origin xyz="0.07691 -0.01 0" rpy="0 0 0" />
@@ -145,10 +129,4 @@
       <visual name="${prefix}_r_finger_visual">
         <origin xyz="0 0 0" rpy="0 0 0" />
-        <map name="gazebo_material" reference="${prefix}_r_finger_visual">
-          <material value="PR2/Grey" />
-        </map>
-        <map name="${prefix}_r_finger_visual_mesh" reference="${prefix}_r_finger_visual">
-          <mesh value="upper_finger_r.mesh" />
-        </map>
         <geometry name="${prefix}_r_finger_visual_geom">
           <mesh filename="upper_finger_r.stlb" />
@@ -161,35 +139,53 @@
         </geometry>
         <verbose value="Yes" />
-        <map name="${prefix}_r_finger_collision_mesh" reference="${prefix}_r_finger_collision">
-          <mesh value="convex/upper_finger_r_convex.mesh" />
-        </map>
-        <map name="mesh" reference="${prefix}_r_finger_collision">
-          <type value="visual"/>
-        </map>
-        <map name="${prefix}_r_finger_contact" reference="${prefix}_r_finger_collision">
-          <mu1 value="${finger_mu}" />
-          <mu2 value="${finger_mu}" />
-          <kp value="1000000.0" />
-          <kd value="1.0" />
-        </map>
-      </collision>
-      <map name="${prefix}_r_finger_sensor" reference="${prefix}_r_finger_link">
-        <verbatim key="${prefix}_r_finger_bumper_sensor">
-          <sensor:contact name="${prefix}_r_finger_contact_sensor">
-            <geom>${prefix}_r_finger_collision</geom>
-            <updateRate>100.0</updateRate>
-            <controller:ros_bumper name="${prefix}_r_finger_ros_bumper_controller" plugin="libros_bumper.so">
-              <alwaysOn>true</alwaysOn>
-              <updateRate>100.0</updateRate>
-              <bumperTopicName>${prefix}_r_finger_bumper</bumperTopicName>
-              <interface:bumper name="${prefix}_r_finger_ros_bumper_iface" />
-            </controller:ros_bumper>
-          </sensor:contact>
-        </verbatim>
-      </map>
-      <map name="${prefix}_r_finger_gravity" reference="${prefix}_r_finger_link">
-        <turnGravityOff>true</turnGravityOff>
-      </map>
-    </link>
+      </collision>
+    </link>
+    <gazebo name="${prefix}_r_finger_gravity" reference="${prefix}_r_finger_link">
+      <turnGravityOff>true</turnGravityOff>
+    </gazebo>
+    <gazebo name="${prefix}_r_finger_sensor" reference="${prefix}_r_finger_link">
+      <sensor:contact name="${prefix}_r_finger_contact_sensor">
+        <geom>${prefix}_r_finger_collision</geom>
+        <updateRate>100.0</updateRate>
+        <controller:ros_bumper name="${prefix}_r_finger_ros_bumper_controller" plugin="libros_bumper.so">
+          <alwaysOn>true</alwaysOn>
+          <updateRate>100.0</updateRate>
+          <bumperTopicName>${prefix}_r_finger_bumper</bumperTopicName>
+          <interface:bumper name="${prefix}_r_finger_ros_bumper_iface" />
+        </controller:ros_bumper>
+      </sensor:contact>
+    </gazebo>
+    <gazebo name="${prefix}_r_finger_contact" reference="${prefix}_r_finger_collision">
+      <mu1 value="${finger_mu}" />
+      <mu2 value="${finger_mu}" />
+      <kp value="1000000.0" />
+      <kd value="1.0" />
+    </gazebo>
+    <gazebo name="gazebo_material" reference="${prefix}_r_finger_visual">
+      <material value="PR2/Grey" />
+    </gazebo>
+    <gazebo name="${prefix}_r_finger_joint_ode" reference="${prefix}_r_finger_joint">
+      <stopKd value="${finger_stop_kd}" />
+      <stopKp value="${finger_stop_kp}" />
+      <fudgeFactor value="${finger_fudge_factor}" />
+    </gazebo>
+    <gazebo name="${prefix}_r_finger_options" reference="${prefix}_r_finger_joint">
+      <provideFeedback value="true"/>
+      <initialAngle value="${-gripper_min_angle}"/>
+    </gazebo>
+    <gazebo name="${prefix}_r_finger_mimic" reference="${prefix}_r_finger_joint">
+      <mimicKp   value="${finger_kp}" />
+      <mimicKd   value="${finger_kd}" />
+      <mimicFMax value="${finger_fm}" />
+    </gazebo>
+    <ogre name="mesh" reference="${prefix}_r_finger_collision">
+      <type value="visual"/>
+    </ogre>
+    <ogre name="${prefix}_r_finger_collision_mesh" reference="${prefix}_r_finger_collision">
+      <mesh value="convex/upper_finger_r_convex.mesh" />
+    </ogre>
+    <ogre name="${prefix}_r_finger_visual_mesh" reference="${prefix}_r_finger_visual">
+      <mesh value="upper_finger_r.mesh" />
+    </ogre>
     <!-- Finger tip -->
     <link name="${prefix}_l_finger_tip_link">
@@ -200,18 +196,4 @@
         <joint_properties damping="${finger_tip_damping}" />
         <mimic name="${prefix}_l_finger_joint" mult="1" offset="0"/>
-        <map name="${prefix}_l_finger_tip_mimic" reference="${prefix}_l_finger_tip_link">
-          <mimicKp   value="${finger_tip_kp}" />
-          <mimicKd   value="${finger_tip_kd}" />
-          <mimicFMax value="${finger_tip_fm}" />
-        </map>
-        <map name="${prefix}_l_finger_tip_options" reference="${prefix}_l_finger_tip_link">
-          <provideFeedback value="true"/>
-          <initialAngle value="${-gripper_min_angle}"/>
-        </map>
-        <map name="${prefix}_l_finger_tip_joint_ode" reference="${prefix}_l_finger_tip_link">
-          <stopKd value="${finger_stop_kd}" />
-          <stopKp value="${finger_stop_kp}" />
-          <fudgeFactor value="${finger_fudge_factor}" />
-        </map>
         <parent name="${prefix}_l_finger_link">
           <origin xyz="0.09137 0.00495 0" rpy="0 0 0" />
@@ -227,13 +209,7 @@
       <visual name="${prefix}_l_finger_tip_visual">
         <origin xyz="0 0 0" rpy="0 0 0" />
-        <map name="gazebo_material" reference="${prefix}_l_finger_tip_visual">
-          <material value="PR2/Green" />
-        </map>
         <geometry name="${prefix}_l_finger_tip_visual_geom">
           <mesh filename="finger_tip_l.stlb" />
         </geometry>
-        <map name="${prefix}_l_finger_tip_visual_mesh" reference="${prefix}_l_finger_tip_visual">
-          <mesh value="finger_tip_l.mesh" />
-        </map>
       </visual>
       <collision name="${prefix}_l_finger_tip_collision">
@@ -242,37 +218,55 @@
           <mesh filename="convex/finger_tip_l_convex.stlb" />
         </geometry>
-        <map name="${prefix}_l_finger_tip_collision_mesh" reference="${prefix}_l_finger_tip_collision">
-          <mesh value="convex/finger_tip_l_convex.mesh" />
-        </map>
         <verbose value="Yes" />
-        <map reference="${prefix}_l_finger_tip_collision" name="mesh">
-          <type value="visual"/>
-        </map>
-        <map name="${prefix}_l_finger_tip_contact" reference="${prefix}_l_finger_tip_collision">
-          <mu1 value="${finger_tip_mu}" />
-          <mu2 value="${finger_tip_mu}" />
-          <kp  value="10000000.0" />
-          <kd  value="1.0" />
-        </map>
-      </collision>
-      <map name="${prefix}_l_finger_tip_sensor" reference="${prefix}_l_finger_tip_link">
-        <verbatim key="${prefix}_l_finger_tip_bumper_sensor">
-          <sensor:contact name="${prefix}_l_finger_tip_contact_sensor">
-            <geom>${prefix}_l_finger_tip_collision</geom>
-            <updateRate>100.0</updateRate>
-            <controller:ros_bumper name="${prefix}_l_finger_tip_ros_bumper_controller" plugin="libros_bumper.so">
-              <alwaysOn>true</alwaysOn>
-              <updateRate>100.0</updateRate>
-              <bumperTopicName>${prefix}_l_finger_tip_bumper</bumperTopicName>
-              <interface:bumper name="${prefix}_l_finger_tip_ros_bumper_iface" />
-            </controller:ros_bumper>
-          </sensor:contact>
-        </verbatim>
-      </map>
-      <map name="${prefix}_l_finger_tip_gravity" reference="${prefix}_l_finger_tip_link">
-        <turnGravityOff>true</mimicKp>
-        <selfCollide value="false" />
-      </map>
-    </link>
+      </collision>
+    </link>
+    <gazebo name="${prefix}_l_finger_tip_gravity" reference="${prefix}_l_finger_tip_link">
+      <turnGravityOff>true</mimicKp>
+      <selfCollide value="false" />
+    </gazebo>
+    <gazebo name="${prefix}_l_finger_tip_sensor" reference="${prefix}_l_finger_tip_link">
+      <sensor:contact name="${prefix}_l_finger_tip_contact_sensor">
+        <geom>${prefix}_l_finger_tip_collision</geom>
+        <updateRate>100.0</updateRate>
+        <controller:ros_bumper name="${prefix}_l_finger_tip_ros_bumper_controller" plugin="libros_bumper.so">
+          <alwaysOn>true</alwaysOn>
+          <updateRate>100.0</updateRate>
+          <bumperTopicName>${prefix}_l_finger_tip_bumper</bumperTopicName>
+          <interface:bumper name="${prefix}_l_finger_tip_ros_bumper_iface" />
+        </controller:ros_bumper>
+      </sensor:contact>
+    </gazebo>
+    <gazebo name="${prefix}_l_finger_tip_contact" reference="${prefix}_l_finger_tip_collision">
+      <mu1 value="${finger_tip_mu}" />
+      <mu2 value="${finger_tip_mu}" />
+      <kp  value="10000000.0" />
+      <kd  value="1.0" />
+    </gazebo>
+    <gazebo name="gazebo_material" reference="${prefix}_l_finger_tip_visual">
+      <material value="PR2/Green" />
+    </gazebo>
+    <gazebo name="${prefix}_l_finger_tip_joint_ode" reference="${prefix}_l_finger_tip_link">
+      <stopKd value="${finger_stop_kd}" />
+      <stopKp value="${finger_stop_kp}" />
+      <fudgeFactor value="${finger_fudge_factor}" />
+    </gazebo>
+    <gazebo name="${prefix}_l_finger_tip_options" reference="${prefix}_l_finger_tip_link">
+      <provideFeedback value="true"/>
+      <initialAngle value="${-gripper_min_angle}"/>
+    </gazebo>
+    <gazebo name="${prefix}_l_finger_tip_mimic" reference="${prefix}_l_finger_tip_link">
+      <mimicKp   value="${finger_tip_kp}" />
+      <mimicKd   value="${finger_tip_kd}" />
+      <mimicFMax value="${finger_tip_fm}" />
+    </gazebo>
+    <ogre reference="${prefix}_l_finger_tip_collision" name="mesh">
+      <type value="visual"/>
+    </ogre>
+    <ogre name="${prefix}_l_finger_tip_collision_mesh" reference="${prefix}_l_finger_tip_collision">
+      <mesh value="convex/finger_tip_l_convex.mesh" />
+    </ogre>
+    <ogre name="${prefix}_l_finger_tip_visual_mesh" reference="${prefix}_l_finger_tip_visual">
+      <mesh value="finger_tip_l.mesh" />
+    </ogre>
     <!-- Finger tip -->
     <link name="${prefix}_r_finger_tip_link">
@@ -283,18 +277,4 @@
         <joint_properties damping="${finger_tip_damping}" />
         <mimic name="${prefix}_l_finger_joint" mult="1" offset="0"/>
-        <map name="${prefix}_r_finger_tip_mimic" reference="${prefix}_r_finger_tip_joint">
-          <mimicKp   value="${finger_tip_kp}" />
-          <mimicKd   value="${finger_tip_kd}" />
-          <mimicFMax value="${finger_tip_fm}" />
-        </map>
-        <map name="${prefix}_r_finger_tip_options" reference="${prefix}_r_finger_tip_joint">
-          <provideFeedback value="true"/>
-          <initialAngle value="${gripper_min_angle}"/>
-        </map>
-        <map name="${prefix}_r_finger_tip_joint_ode" reference="${prefix}_r_finger_tip_joint">
-          <stopKd value="${finger_stop_kd}" />
-          <stopKp value="${finger_stop_kp}" />
-          <fudgeFactor value="${finger_fudge_factor}" />
-        </map>
         <parent name="${prefix}_r_finger_link">
           <origin xyz="${0.09137} ${-0.00495} 0" rpy="0 0 0" />
@@ -310,13 +290,7 @@
       <visual name="${prefix}_r_finger_tip_visual">
         <origin xyz="0 0 0" rpy="0 0 0" />
-        <map name="gazebo_material" reference="${prefix}_r_finger_tip_visual">
-          <material value="PR2/Green" />
-        </map>
         <geometry name="${prefix}_r_finger_tip_visual_geom">
           <mesh filename="finger_tip_r.stlb" />
         </geometry>
-        <map name="${prefix}_r_finger_tip_visual_mesh" reference="${prefix}_r_finger_tip_visual">
-          <mesh value="finger_tip_r.mesh" />
-        </map>
       </visual>
       <collision name="${prefix}_r_finger_tip_collision">
@@ -325,58 +299,74 @@
           <mesh filename="convex/finger_tip_r_convex.stlb" />
         </geometry>
-        <map name="${prefix}_r_finger_tip_collision_mesh" reference="${prefix}_r_finger_tip_collision">
-          <mesh value="convex/finger_tip_r_convex.mesh" />
-        </map>
         <verbose value="Yes" />
-        <map reference="${prefix}_r_finger_tip_collision" name="mesh">
-          <type value="visual"/>
-        </map>
-        <map name="${prefix}_r_finger_tip_contact" reference="${prefix}_r_finger_tip_collision">
-          <mu1 value="${finger_tip_mu}" />
-          <mu2 value="${finger_tip_mu}" />
-          <kp  value="10000000.0" />
-          <kd  value="1.0" />
-        </map>
-      </collision>
-      <map name="${prefix}_r_finger_tip_sensor" reference="${prefix}_r_finger_tip_link">
-        <verbatim key="${prefix}_r_finger_tip_bumper_sensor">
-          <sensor:contact name="${prefix}_r_finger_tip_contact_sensor">
-            <geom>${prefix}_r_finger_tip_collision</geom>
-            <updateRate>100.0</updateRate>
-            <controller:ros_bumper name="${prefix}_r_finger_tip_ros_bumper_controller" plugin="libros_bumper.so">
-              <alwaysOn>true</alwaysOn>
-              <updateRate>100.0</updateRate>
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