Commit message: converting urdf.
git-svn-id: https://svn.code.sf.net/p/personalrobots/code/pkg/trunk@20437 f5854215-dd47-0410-b2c4-cdd35faa7885

Former-commit-id: a4873532359b68515d694d29f9b2b1a5fb2de4b3

File: stacks/pr2/pr2_defs/defs/head_defs.urdf.xacro (robot description, xacro)
@@ -25,13 +25,7 @@
       <visual name="${name}_mount_visual">
         <origin xyz="0 0 0" rpy="0 0 0" />
-        <map name="gazebo_material" reference="${name}_mount_visual">
-          <material value="PR2/Red" />
-        </map>
         <geometry name="${name}_mount_visual_geom">
           <mesh filename="hok_tilt.stlb" />
         </geometry>
-        <map name="${name}_mount_visual_mesh" reference="${name}_mount_visual">
-          <mesh value="hok_tilt.mesh" />
-        </map>
       </visual>
       <collision name="${name}_mount_collision">
@@ -42,4 +36,10 @@
       </collision>
     </link>
+    <gazebo name="gazebo_material" reference="${name}_mount_visual">
+      <material value="PR2/Red" />
+    </gazebo>
+    <ogre name="${name}_mount_visual_mesh" reference="${name}_mount_visual">
+      <mesh value="hok_tilt.mesh" />
+    </ogre>
     <transmission type="SimpleTransmission" name="${name}_mount_trans">
       <actuator name="${name}_mount_motor" />
@@ -73,30 +73,28 @@
         </geometry>
       </collision>
-      <map name="sensor" reference="${name}_link">
-        <verbatim key="sensor_${name}_ray">
-          <sensor:ray name="${name}">
-            <rayCount>640</rayCount>
-            <rangeCount>640</rangeCount>
-            <laserCount>1</laserCount>
-            <origin>0.0 0.0 0.0</origin>
-            <displayRays>false</displayRays>
-            <minAngle>-80</minAngle>
-            <maxAngle> 80</maxAngle>
-            <minRange>0.05</minRange>
-            <maxRange>10.0</maxRange>
-            <resRange>0.01</resRange>
-            <updateRate>20.0</updateRate>
-            <controller:ros_laser name="ros_${name}_controller" plugin="libros_laser.so">
-              <gaussianNoise>0.005</gaussianNoise>
-              <alwaysOn>true</alwaysOn>
-              <updateRate>20.0</updateRate>
-              <topicName>tilt_scan</topicName>
-              <frameName>${name}_link</frameName>
-              <interface:laser name="ros_${name}_iface" />
-            </controller:ros_laser>
-          </sensor:ray>
-        </verbatim>
-      </map>
-    </link>
+    </link>
+    <gazebo name="sensor" reference="${name}_link">
+      <sensor:ray name="${name}">
+        <rayCount>640</rayCount>
+        <rangeCount>640</rangeCount>
+        <laserCount>1</laserCount>
+        <origin>0.0 0.0 0.0</origin>
+        <displayRays>false</displayRays>
+        <minAngle>-80</minAngle>
+        <maxAngle> 80</maxAngle>
+        <minRange>0.05</minRange>
+        <maxRange>10.0</maxRange>
+        <resRange>0.01</resRange>
+        <updateRate>20.0</updateRate>
+        <controller:ros_laser name="ros_${name}_controller" plugin="libros_laser.so">
+          <gaussianNoise>0.005</gaussianNoise>
+          <alwaysOn>true</alwaysOn>
+          <updateRate>20.0</updateRate>
+          <topicName>tilt_scan</topicName>
+          <frameName>${name}_link</frameName>
+          <interface:laser name="ros_${name}_iface" />
+        </controller:ros_laser>
+      </sensor:ray>
+    </gazebo>
   </macro>
   <property name="stereo_size_x" value="0.005" />
@@ -131,7 +129,4 @@
       <visual name="${name}_sensor_visual">
         <origin xyz="0 0 0" rpy="0 0 0" />
-        <map name="gazebo_material" reference="${name}_sensor_visual">
-          <material value="PR2/Blue" />
-        </map>
         <geometry name="${name}_sensor_visual_geom">
           <box size="0.01 0.01 0.01" />
@@ -145,4 +140,7 @@
       </collision>
     </link>
+    <gazebo name="gazebo_material" reference="${name}_sensor_visual">
+      <material value="PR2/Blue" />
+    </gazebo>
     <!-- Prosilica Camera -->
     <prosilica_cam name="${hd_name}" parent="${name}_link" >
@@ -176,7 +174,4 @@
       <visual name="${name}_double_stereo_visual">
         <origin xyz="0 0 0" rpy="0 0 0" />
-        <map name="gazebo_material" reference="${name}_double_stereo_visual">
-          <material value="PR2/Blue" />
-        </map>
         <geometry name="${name}_double_stereo_visual_geom">
           <box size="0.01 0.01 0.01" />
@@ -190,4 +185,7 @@
       </collision>
     </link>
+    <gazebo name="gazebo_material" reference="${name}_double_stereo_visual">
+      <material value="PR2/Blue" />
+    </gazebo>
     <!-- Wide camera is on robot right (hca1), narrow on left (hca2)? -->
     <!-- 15mm offset from center needs check with CAD -->
@@ -214,7 +212,4 @@
       <visual name="${name}_visual">
         <origin xyz="${stereo_center_box_center_offset_x} 0 ${stereo_center_box_center_offset_z}" rpy="0 0 0" />
-        <map name="gazebo_material" reference="${name}_visual">
-          <material value="PR2/Blue" />
-        </map>
         <geometry name="${name}_visual_geom">
           <box size="${stereo_size_x} ${stereo_size_y} ${stereo_size_z}" />
@@ -228,4 +223,7 @@
       </collision>
     </link>
+    <gazebo name="gazebo_material" reference="${name}_visual">
+      <material value="PR2/Blue" />
+    </gazebo>
     <link name="${name}_optical_frame" type="camera">
       <joint name="${name}_optical_fixed_joint" type="fixed">
@@ -244,7 +242,4 @@
       <visual name="${name}_optical_fixed_visual">
         <origin xyz="0 0 0" rpy="0 0 0" />
-        <map name="gazebo_material" reference="${name}_optical_fixed_visual">
-          <material value="PR2/Blue" />
-        </map>
         <geometry name="${name}_optical_fixed_visual_geom">
           <box size="0.01 0.01 0.01" />
@@ -258,4 +253,7 @@
       </collision>
     </link>
+    <gazebo name="gazebo_material" reference="${name}_optical_fixed_visual">
+      <material value="PR2/Blue" />
+    </gazebo>
     <link name="${name}_l_stereo_camera_frame">
       <joint name="${name}_l_stereo_camera_fixed_joint" type="fixed">
@@ -273,7 +271,4 @@
       <visual name="${name}_l_stereo_camera_visual">
         <origin xyz="0 0 0" rpy="0 0 0" />
-        <map name="gazebo_material" reference="${name}_l_stereo_camera_visual">
-          <material value="PR2/Blue" />
-        </map>
         <geometry name="${name}_l_stereo_camera_visual_geom">
           <box size="0.01 0.01 0.01" />
@@ -286,24 +281,25 @@
         </geometry>
       </collision>
-      <map name="sensor" reference="${name}_l_stereo_camera_frame">
-        <verbatim key="sensor_${name}_l_camera">
-          <sensor:camera name="${name}_l_sensor">
-            <imageSize>640 480</imageSize>
-            <imageFormat>L8</imageFormat>
-            <hfov>90</hfov>
-            <nearClip>0.1</nearClip>
-            <farClip>100</farClip>
-            <updateRate>20.0</updateRate>
-            <controller:ros_camera name="${name}_l_controller" plugin="libros_camera.so">
-              <alwaysOn>true</alwaysOn>
-              <updateRate>20.0</updateRate>
-              <topicName>${name}/left_image</topicName>
-              <frameName>${name}_l_stereo_camera_frame</frameName>
-              <interface:camera name="${name}_l_iface" />
-            </controller:ros_camera>
-          </sensor:camera>
-        </verbatim>
-      </map>
-    </link>
+    </link>
+    <gazebo name="sensor" reference="${name}_l_stereo_camera_frame">
+      <sensor:camera name="${name}_l_sensor">
+        <imageSize>640 480</imageSize>
+        <imageFormat>L8</imageFormat>
+        <hfov>90</hfov>
+        <nearClip>0.1</nearClip>
+        <farClip>100</farClip>
+        <updateRate>20.0</updateRate>
+        <controller:ros_camera name="${name}_l_controller" plugin="libros_camera.so">
+          <alwaysOn>true</alwaysOn>
+          <updateRate>20.0</updateRate>
+          <topicName>${name}/left_image</topicName>
+          <frameName>${name}_l_stereo_camera_frame</frameName>
+          <interface:camera name="${name}_l_iface" />
+        </controller:ros_camera>
+      </sensor:camera>
+    </gazebo>
+    <gazebo name="gazebo_material" reference="${name}_l_stereo_camera_visual">
+      <material value="PR2/Blue" />
+    </gazebo>
     <link name="${name}_r_stereo_camera_frame">
       <joint name="${name}_r_stereo_camera_fixed_joint" type="fixed">
@@ -322,7 +318,4 @@
       <visual name="${name}_r_stereo_camera_visual">
         <origin xyz="0 0 0" rpy="0 0 0" />
-        <map name="gazebo_material" reference="${name}_r_stereo_camera_visual">
-          <material value="PR2/Blue" />
-        </map>
         <geometry name="${name}_r_stereo_camera_visual_geom">
           <box size="0.01 0.01 0.01" />
@@ -335,49 +328,48 @@
         </geometry>
       </collision>
-      <map name="sensor" reference="${name}_r_stereo_camera_frame">
-        <verbatim key="sensor_${name}_r_camera">
-          <sensor:camera name="${name}_r_sensor">
-            <imageSize>640 480</imageSize>
-            <imageFormat>L8</imageFormat>
-            <hfov>90</hfov>
-            <nearClip>0.1</nearClip>
-            <farClip>100</farClip>
-            <updateRate>20.0</updateRate>
-            <controller:ros_camera name="${name}_r_controller" plugin="libros_camera.so">
-              <alwaysOn>true</alwaysOn>
-              <updateRate>20.0</updateRate>
-              <topicName>${name}/right_image</topicName>
-              <frameName>${name}_r_stereo_camera_frame</frameName>
-              <interface:camera name="${name}_r_iface" />
-            </controller:ros_camera>
-          </sensor:camera>
-        </verbatim>
-      </map>
-    </link>
+    </link>
+    <gazebo name="sensor" reference="${name}_r_stereo_camera_frame">
+      <sensor:camera name="${name}_r_sensor">
+        <imageSize>640 480</imageSize>
+        <imageFormat>L8</imageFormat>
+        <hfov>90</hfov>
+        <nearClip>0.1</nearClip>
+        <farClip>100</farClip>
+        <updateRate>20.0</updateRate>
+        <controller:ros_camera name="${name}_r_controller" plugin="libros_camera.so">
+          <alwaysOn>true</alwaysOn>
+          <updateRate>20.0</updateRate>
+          <topicName>${name}/right_image</topicName>
+          <frameName>${name}_r_stereo_camera_frame</frameName>
+          <interface:camera name="${name}_r_iface" />
+        </controller:ros_camera>
+      </sensor:camera>
+    </gazebo>
+    <gazebo name="gazebo_material" reference="${name}_r_stereo_camera_visual">
+      <material value="PR2/Blue" />
+    </gazebo>
     <!-- stereo plugin that produces a raw_stereo message
     -->
-    <map name="sensor">
-      <verbatim key="controller_${name}_camera">
-        <controller:ros_stereo_camera name="${name}_controller" plugin="libros_stereo_camera.so">
-          <alwaysOn>true</alwaysOn>
-          <updateRate>20.0</updateRate>
-          <leftCamera>${name}_l_sensor</leftCamera>
-          <rightCamera>${name}_r_sensor</rightCamera>
-          <topicName>${name}/raw_stereo</topicName>
-          <frameName>${name}_optical_frame</frameName>
-          <CxPrime>320</CxPrime>
-          <Cx>320</Cx>
-          <Cy>240</Cy>
-          <focal_length>320</focal_length> <!-- image_width / (2*tan(hfov_radian /2)) -->
-          <distortion_k1>0</distortion_k1>
-          <distortion_k2>0</distortion_k2>
-          <distortion_k3>0</distortion_k3>
-          <distortion_t1>0</distortion_t1>
-          <distortion_t2>0</distortion_t2>
-          <baseline>${stereo_dy}</baseline> <!-- home pos. of robot has +x forward, +y left -->
-          <interface:stereocamera name="${name}_iface" />
-        </controller:ros_stereo_camera>
-      </verbatim>
-    </map>
+    <gazebo name="sensor">
+      <controller:ros_stereo_camera name="${name}_controller" plugin="libros_stereo_camera.so">
+        <alwaysOn>true</alwaysOn>
+        <updateRate>20.0</updateRate>
+        <leftCamera>${name}_l_sensor</leftCamera>
+        <rightCamera>${name}_r_sensor</rightCamera>
+        <topicName>${name}/raw_stereo</topicName>
+        <frameName>${name}_optical_frame</frameName>
+        <CxPrime>320</CxPrime>
+        <Cx>320</Cx>
+        <Cy>240</Cy>
+        <focal_length>320</focal_length> <!-- image_width / (2*tan(hfov_radian /2)) -->
+        <distortion_k1>0</distortion_k1>
+        <distortion_k2>0</distortion_k2>
+        <distortion_k3>0</distortion_k3>
+        <distortion_t1>0</distortion_t1>
+        <distortion_t2>0</distortion_t2>
+        <baseline>${stereo_dy}</baseline> <!-- home pos. of robot has +x forward, +y left -->
+        <interface:stereocamera name="${name}_iface" />
+      </controller:ros_stereo_camera>
+    </gazebo>
   </macro>
   <macro name="pr2_head_pan" params="name parent *origin">
@@ -400,13 +392,7 @@
       <visual name="${name}_visual">
         <origin xyz="0 0 0.0" rpy="0 0 0 " />
-        <map name="gazebo_material" reference="${name}_visual">
-          <material value="PR2/Blue" />
-        </map>
         <geometry name="${name}_visual_geom">
           <mesh filename="head_pan.stlb" />
         </geometry>
-        <map name="${name}_visual_mesh" reference="${name}_visual">
-          <mesh value="head_pan.mesh" />
-        </map>
       </visual>
       <collision name="${name}_collision">
@@ -417,4 +403,10 @@
       </collision>
     </link>
+    <gazebo name="gazebo_material" reference="${name}_visual">
+      <material value="PR2/Blue" />
+    </gazebo>
+    <ogre name="${name}_visual_mesh" reference="${name}_visual">
+      <mesh value="head_pan.mesh" />
+    </ogre>
     <transmission type="SimpleTransmission" name="${name}_trans">
       <actuator name="${name}_motor" />
@@ -444,13 +436,7 @@
       <visual name="${name}_visual">
         <origin xyz="0 0 0" rpy="0.0 0.0 0.0 " />
-        <map name="gazebo_material" reference="${name}_visual">
-          <material value="PR2/Green" />
-        </map>
         <geometry name="${name}_visual_geom">
           <mesh filename="head_tilt.stlb" />
         </geometry>
-        <map name="${name}_visual_mesh" reference="${name}_visual">
-          <mesh value="head_tilt.mesh" />
-        </map>
       </visual>
       <collision name="${name}_collision">
@@ -461,4 +447,10 @@
       </collision>
     </link>
+    <gazebo name="gazebo_material" reference="${name}_visual">
+      <material value="PR2/Green" />
+    </gazebo>
+    <ogre name="${name}_visual_mesh" reference="${name}_visual">
+      <mesh value="head_tilt.mesh" />
+    </ogre>
     <transmission type="SimpleTransmission" name="${name}_trans">
       <actuator name="${name}_motor" />
@@ -491,7 +483,4 @@
       <visual name="${name}_plate_frame_visual">
         <origin xyz="0 0 0" rpy="0 0 0" />
-        <map name="gazebo_material" reference="${name}_plate_frame_visual">
-          <material value="PR2/Blue" />
-        </map>
         <geometry name="${name}_plate_frame_visual_geom">
           <box size="0.01 0.01 0.01" />
@@ -505,4 +494,7 @@
       </collision>
     </link>
+    <gazebo name="gazebo_material" reference="${name}_plate_frame_visual">
+      <material value="PR2/Blue" />
+    </gazebo>
   </macro>
   <!-- Alpha 2.0 head -->
@@ -530,13 +522,7 @@
       <visual name="${name}_mount_visual">
         <origin xyz="0 0 0" rpy="0 0 0" />
-        <map name="gazebo_material" reference="${name}_mount_visual">
-          <material value="PR2/Red" />
-        </map>
         <geometry name="${name}_mount_visual_geom">
           <mesh filename="hok_tilt.stlb" />
         </geometry>
-        <map name="${name}_mount_visual_mesh" reference="${name}_mount_visual">
-          <mesh value="hok_tilt.mesh" />
-        </map>
       </visual>
       <collision name="${name}_mount_collision">
@@ -547,4 +533,10 @@
       </collision>
     </link>
+    <gazebo name="gazebo_material" reference="${name}_mount_visual">
+      <material value="PR2/Red" />
+    </gazebo>
+    <ogre name="${name}_mount_visual_mesh" reference="${name}_mount_visual">
+      <mesh value="hok_tilt.mesh" />
+    </ogre>
     <transmission type="SimpleTransmission" name="${name}_mount_trans">
       <actuator name="${name}_mount_motor" />
@@ -578,30 +570,28 @@
         </geometry>
       </collision>
-      <map name="sensor" reference="${name}_link">
-        <verbatim key="sensor_${name}_ray">
-          <sensor:ray name="${name}">
-            <rayCount>640</rayCount>
-            <rangeCount>640</rangeCount>
-            <laserCount>1</laserCount>
-            <origin>0.0 0.0 0.0</origin>
-            <displayRays>false</displayRays>
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