Commit message: work in progress.
git-svn-id: https://svn.code.sf.net/p/personalrobots/code/pkg/trunk@20406 f5854215-dd47-0410-b2c4-cdd35faa7885

Former-commit-id: fd2151d20ddf378e542fba5b15372d56bec5912f

File: stacks/pr2/pr2_defs/defs/arm_defs.urdf.xacro (robot description, xacro)
@@ -487,16 +487,14 @@
     </gazebo>
     <gazebo name="${side}_wrist_flex_sensor" reference="${side}_wrist_flex_link">
-      <verbatim key="${side}_wrist_flex_bumper_sensor">
-        <sensor:contact name="${side}_wrist_flex_contact_sensor">
-          <geom>${side}_wrist_flex_collision</geom>
+      <sensor:contact name="${side}_wrist_flex_contact_sensor">
+        <geom>${side}_wrist_flex_collision</geom>
+        <updateRate>100.0</updateRate>
+        <controller:ros_bumper name="${side}_wrist_flex_ros_bumper_controller" plugin="libros_bumper.so">
+          <alwaysOn>true</alwaysOn>
           <updateRate>100.0</updateRate>
-          <controller:ros_bumper name="${side}_wrist_flex_ros_bumper_controller" plugin="libros_bumper.so">
-            <alwaysOn>true</alwaysOn>
-            <updateRate>100.0</updateRate>
-            <bumperTopicName>${side}_wrist_flex_bumper</bumperTopicName>
-            <interface:bumper name="${side}_wrist_flex_ros_bumper_iface" />
-          </controller:ros_bumper>
-        </sensor:contact>
-      </verbatim>
+          <bumperTopicName>${side}_wrist_flex_bumper</bumperTopicName>
+          <interface:bumper name="${side}_wrist_flex_ros_bumper_iface" />
+        </controller:ros_bumper>
+      </sensor:contact>
     </gazebo>
     <gazebo name="gazebo_material" reference="${side}_wrist_flex_visual">

File: stacks/pr2/pr2_defs/defs/base_defs.urdf.xacro (robot description, xacro)
@@ -27,109 +27,110 @@
   <property name="base_laser_collision_offset_z" value="0.03" />
   <macro name="pr2_wheel" params="suffix parent reflect">
-    <joint name="${parent}_${suffix}_wheel_joint" type="revolute">
-      <axis xyz="0 1 0" />
-      <anchor xyz="0 0 0" />
-      <limit effort="100" velocity="100" k_velocity="10" />
-      <calibration values="1.5 -1" />
-      <joint_properties damping="0.0" friction="0.0" />
-    </joint>
     <link name="${parent}_${suffix}_wheel_link">
-      <parent name="${parent}_rotation_link" />
-      <joint name="${parent}_${suffix}_wheel_joint" />
+      <joint name="0 0 0" type="0 0 0">
+        <axis xyz="0 1 0" />
+        <limit effort="100" velocity="100"/>
+        <safety_controller k_velocity="10" />
+        <joint_properties damping="0.0" friction="0.0" />
+        <parent name="${parent}_rotation_link">
+          <joint name="${parent}_${suffix}_wheel_joint" type="revolute">
+        </parent>
+      </joint>
       <origin xyz="0 ${reflect*caster_wheel_offset_y} 0" rpy="0 0 0" />
       <inertial>
         <mass value="0.44036" /> <!-- check jmh 20081205 -->
-        <com xyz=" 0 0 0 " />
+        <origin xyz=" 0 0 0 " />
         <inertia  ixx="0.012411765597" ixy="-0.000711733678" ixz="0.00050272983"
                   iyy="0.015218160428" iyz="-0.000004273467" izz="0.011763977943" />
       </inertial>
-      <visual>
-        <origin xyz="0 0 0" rpy="0 0 0" />
-        <map name="gazebo_material" flag="gazebo">
-          <!-- TODO should be different for left and right wheel-->
-          <elem key="material" value="PR2/${parent}_${suffix}_wheel_link" />
-        </map>
-        <geometry name="${parent}_${suffix}_wheel_visual">
+      <visual name="${parent}_${suffix}_wheel_visual">
+        <origin xyz="0 0 0" rpy="0 0 0" />
+        <geometry name="${parent}_${suffix}_wheel_visual_geom">
           <mesh filename="pr2_wheel.stlb" />
         </geometry>
-        <map name="${parent}_${suffix}_wheel_visual_mesh" flag="ogre">
-          <elem key="mesh" value="pr2_wheel.mesh" />
-        </map>
-      </visual>
-      <collision>
+      </visual>
+      <collision name="${parent}_${suffix}_wheel_collision">
         <origin xyz="0 0 0" rpy="${M_PI/2} 0 0" />
-        <geometry name="${parent}_${suffix}_wheel_collision">
+        <geometry name="${parent}_${suffix}_wheel_collision_geom">
           <cylinder radius="${wheel_radius}" length="${wheel_length}" />
         </geometry>
-        <map name="friction_coefficients" flag="gazebo">
-          <elem key="mu1" value="100.0" />
-          <elem key="mu2" value="100.0" />
-          <elem key="kp"  value="1000000.0" />
-          <elem key="kd"  value="1.0" />
-        </map>
-      </collision>
-      <map name="${parent}_${suffix}_wheel_sensor" flag="gazebo">
-        <verbatim key="${parent}_${suffix}_wheel_bumper_sensor">
-          <sensor:contact name="${parent}_${suffix}_wheel_contact_sensor">
-            <geom>${parent}_${suffix}_wheel_collision</geom>
-            <updateRate>100.0</updateRate>
-            <controller:ros_bumper name="${parent}_${suffix}_wheel_ros_bumper_controller" plugin="libros_bumper.so">
-              <alwaysOn>true</alwaysOn>
-              <updateRate>100.0</updateRate>
-              <bumperTopicName>${parent}_${suffix}_wheel_bumper</bumperTopicName>
-              <interface:bumper name="${parent}_${suffix}_wheel_ros_bumper_iface" />
-            </controller:ros_bumper>
-          </sensor:contact>
-        </verbatim>
-      </map>
-    </link>
+      </collision>
+    </link>
+    <gazebo name="${parent}_${suffix}_wheel_sensor" reference="${parent}_${suffix}_wheel_link">
+      <sensor:contact name="${parent}_${suffix}_wheel_contact_sensor">
+        <geom>${parent}_${suffix}_wheel_collision</geom>
+        <updateRate>100.0</updateRate>
+        <controller:ros_bumper name="${parent}_${suffix}_wheel_ros_bumper_controller" plugin="libros_bumper.so">
+          <alwaysOn>true</alwaysOn>
+          <updateRate>100.0</updateRate>
+          <bumperTopicName>${parent}_${suffix}_wheel_bumper</bumperTopicName>
+          <interface:bumper name="${parent}_${suffix}_wheel_ros_bumper_iface" />
+        </controller:ros_bumper>
+      </sensor:contact>
+    </gazebo>
+    <gazebo name="friction_coefficients" reference="${parent}_${suffix}_wheel_collision">
+      <mu1 value="100.0" />
+      <mu2 value="100.0" />
+      <kp  value="1000000.0" />
+      <kd  value="1.0" />
+    </gazebo>
+    <ogre name="${parent}_${suffix}_wheel_visual_mesh" reference="${parent}_${suffix}_wheel_visual">
+      <mesh value="pr2_wheel.mesh" />
+    </ogre>
+    <ogre name="gazebo_material" reference="${parent}_${suffix}_wheel_visual">
+      <!-- TODO should be different for left and right wheel-->
+      <material value="PR2/${parent}_${suffix}_wheel_link" />
+    </ogre>
     <transmission type="SimpleTransmission" name="${parent}_${suffix}_wheel_trans">
       <actuator name="${parent}_${suffix}_wheel_motor" />
       <joint name="${parent}_${suffix}_wheel_joint" />
       <mechanicalReduction>${reflect*75.05}</mechanicalReduction>
+      <calibration values="1.5 -1" />
     </transmission>
   </macro>
   <macro name="pr2_caster" params="suffix parent *origin">
-    <joint name="${suffix}_caster_rotation_joint" type="revolute">
-      <axis xyz="0 0 1" />
-      <anchor xyz="0 0 0" />
-      <limit effort="100" velocity="100" k_velocity="10" />
-      <calibration reference_position="0.0" values="1.5 -1" />
-      <joint_properties damping="0.0" friction="0.0" />
-    </joint>
     <link name="${suffix}_caster_rotation_link">
-      <parent name="${parent}" />
-      <insert_block name="origin" />
-      <joint name="${suffix}_caster_rotation_joint" />
+      <joint name="${suffix}_caster_rotation_joint" type="revolute">
+        <origin xyz="0 0 0" rpy="0 0 0" />
+        <axis xyz="0 0 1" />
+        <limit effort="100" velocity="100"/>
+        <safety_controller k_velocity="10" />
+        <joint_properties damping="0.0" friction="0.0" />
+        <parent name="${parent}">
+          <insert_block name="origin">
+        </parent>
+      </joint>
       <inertial>
         <mass value="3.473082" />
-        <com xyz="0 0 0.07" />
+        <origin xyz="0 0 0.07" />
         <inertia  ixx="0.012411765597" ixy="-0.000711733678" ixz="0.00050272983"
                   iyy="0.015218160428" iyz="-0.000004273467" izz="0.011763977943" />
       </inertial>
-      <visual>
-        <origin xyz="0 0 0" rpy="0 0 0" />
-        <map name="gazebo_material" flag="gazebo">
-          <elem key="material" value="PR2/Green" />
-        </map>
-        <geometry name="${suffix}_caster_rotation_visual">
+      <visual name="${suffix}_caster_rotation_visual">
+        <origin xyz="0 0 0" rpy="0 0 0" />
+        <geometry name="${suffix}_caster_rotation_visual_geom">
           <mesh filename="caster.stlb" />
         </geometry>
-        <map name="${suffix}_caster_rotation_visual_mesh" flag="ogre">
-          <elem key="mesh" value="caster.mesh" />
-        </map>
-      </visual>
-      <collision>
+      </visual>
+      <collision name="${suffix}_caster_rotation_collision">
         <origin xyz="0 0 0.07" rpy="0.0 0.0 0.0" />
-        <geometry name="${suffix}_caster_rotation_collision">
+        <geometry name="${suffix}_caster_rotation_collision_geom">
           <box size="0.192 0.164 0.013" />
         </geometry>
       </collision>
     </link>
+    <ogre name="${suffix}_caster_rotation_visual_mesh" reference="${suffix}_caster_rotation_visual">
+      <elem key="mesh" value="caster.mesh" />
+    </ogre>
+    <ogre name="gazebo_material" reference="${suffix}_caster_rotation_visual">
+      <elem key="material" value="PR2/Green" />
+    </ogre>
     <transmission type="SimpleTransmission" name="${suffix}_caster_rotation_trans">
       <actuator name="${suffix}_caster_rotation_motor" />
       <joint name="${suffix}_caster_rotation_joint" />
       <mechanicalReduction>-75.05</mechanicalReduction>
+      <calibration reference_position="0.0" values="1.5 -1" />
     </transmission>
+    <!-- wheel macros -->
     <pr2_wheel parent="${suffix}_caster" suffix="l" reflect="1" />
     <pr2_wheel parent="${suffix}_caster" suffix="r" reflect="-1" />
@@ -139,108 +140,108 @@
   <!--                                                      -->
   <macro name="pr2_wheel_alpha2" params="suffix parent reflect">
-    <joint name="${parent}_${suffix}_wheel_joint" type="revolute">
-      <axis xyz="0 1 0" />
-      <anchor xyz="0 0 0" />
-      <limit effort="100" velocity="100" k_velocity="10" />
-      <calibration values="1.5 -1" />
-      <joint_properties damping="0.0" friction="0.0" />
-    </joint>
     <link name="${parent}_${suffix}_wheel_link">
-      <parent name="${parent}_rotation_link" />
-      <joint name="${parent}_${suffix}_wheel_joint" />
-      <origin xyz="0 ${reflect*caster_wheel_offset_y} 0" rpy="0 0 0" />
+      <joint name="${parent}_${suffix}_wheel_joint" type="revolute">
+        <origin xyz="0 0 0" rpy="0 0 0" />
+        <axis xyz="0 1 0" />
+        <limit effort="100" velocity="100"/>
+        <safety_controller  k_velocity="10" />
+        <joint_properties damping="0.0" friction="0.0" />
+        <parent name="${parent}_rotation_link">
+          <origin xyz="0 ${reflect*caster_wheel_offset_y} 0" rpy="0 0 0" />
+        </parent>
+      </joint>
       <inertial>
         <mass value="0.44036" /> <!-- check jmh 20081205 -->
-        <com xyz=" 0 0 0 " />
+        <origin xyz="0 0 0" />
         <inertia  ixx="0.012411765597" ixy="-0.000711733678" ixz="0.00050272983"
                   iyy="0.015218160428" iyz="-0.000004273467" izz="0.011763977943" />
       </inertial>
-      <visual>
-        <origin xyz="0 0 0" rpy="0 0 0" />
-        <map name="gazebo_material" flag="gazebo">
-          <!-- TODO should be different for left and right wheel-->
-          <elem key="material" value="PR2/${parent}_${suffix}_wheel_link" />
-        </map>
-        <geometry name="${parent}_${suffix}_wheel_visual">
+      <visual name="${parent}_${suffix}_wheel_visual">
+        <origin xyz="0 0 0" rpy="0 0 0" />
+        <geometry name="${parent}_${suffix}_wheel_visual_geom">
           <mesh filename="pr2_wheel.stlb" />
         </geometry>
-        <map name="${parent}_${suffix}_wheel_visual_mesh" flag="ogre">
-          <elem key="mesh" value="pr2_wheel.mesh" />
-        </map>
-      </visual>
-      <collision>
+      </visual>
+      <collision name="${parent}_${suffix}_wheel_collision">
         <origin xyz="0 0 0" rpy="${M_PI/2} 0 0" />
-        <geometry name="${parent}_${suffix}_wheel_collision">
+        <geometry name="${parent}_${suffix}_wheel_collision_geom">
           <cylinder radius="${wheel_radius}" length="${wheel_length}" />
         </geometry>
-        <map name="friction_coefficients" flag="gazebo">
-          <elem key="mu1" value="100.0" />
-          <elem key="mu2" value="100.0" />
-          <elem key="kp"  value="1000000.0" />
-          <elem key="kd"  value="1.0" />
-        </map>
-      </collision>
-      <map name="${parent}_${suffix}_wheel_sensor" flag="gazebo">
-        <verbatim key="${parent}_${suffix}_wheel_bumper_sensor">
-          <sensor:contact name="${parent}_${suffix}_wheel_contact_sensor">
-            <geom>${parent}_${suffix}_wheel_collision</geom>
-            <updateRate>100.0</updateRate>
-            <controller:ros_bumper name="${parent}_${suffix}_wheel_ros_bumper_controller" plugin="libros_bumper.so">
-              <alwaysOn>true</alwaysOn>
-              <updateRate>100.0</updateRate>
-              <bumperTopicName>${parent}_${suffix}_wheel_bumper</bumperTopicName>
-              <interface:bumper name="${parent}_${suffix}_wheel_ros_bumper_iface" />
-            </controller:ros_bumper>
-          </sensor:contact>
-        </verbatim>
-      </map>
-    </link>
+      </collision>
+    </link>
+    <gazebo name="${parent}_${suffix}_wheel_sensor" reference="${parent}_${suffix}_wheel_link">
+      <sensor:contact name="${parent}_${suffix}_wheel_contact_sensor">
+        <geom>${parent}_${suffix}_wheel_collision</geom>
+        <updateRate>100.0</updateRate>
+        <controller:ros_bumper name="${parent}_${suffix}_wheel_ros_bumper_controller" plugin="libros_bumper.so">
+          <alwaysOn>true</alwaysOn>
+          <updateRate>100.0</updateRate>
+          <bumperTopicName>${parent}_${suffix}_wheel_bumper</bumperTopicName>
+          <interface:bumper name="${parent}_${suffix}_wheel_ros_bumper_iface" />
+        </controller:ros_bumper>
+      </sensor:contact>
+    </gazebo>
+    <gazebo name="friction_coefficients" reference="${parent}_${suffix}_wheel_collision">
+      <mu1 value="100.0" />
+      <mu2 value="100.0" />
+      <kp  value="1000000.0" />
+      <kd  value="1.0" />
+    </gazebo>
+    <ogre name="${parent}_${suffix}_wheel_visual_mesh" reference="${parent}_${suffix}_wheel_visual">
+      <mesh value="pr2_wheel.mesh" />
+    </ogre>
+    <ogre name="gazebo_material" reference="${parent}_${suffix}_wheel_visual">
+      <!-- TODO should be different for left and right wheel-->
+      <material value="PR2/${parent}_${suffix}_wheel_link" />
+    </ogre>
     <transmission type="SimpleTransmission" name="${parent}_${suffix}_wheel_trans">
       <actuator name="${parent}_${suffix}_wheel_motor_alpha2" />
       <joint name="${parent}_${suffix}_wheel_joint" />
       <mechanicalReduction>${-1 * reflect * 79.226}</mechanicalReduction>
+      <calibration values="1.5 -1" />
     </transmission>
   </macro>
   <macro name="pr2_caster_alpha2" params="suffix parent *origin ref_position">
-    <joint name="${suffix}_caster_rotation_joint" type="revolute">
-      <axis xyz="0 0 1" />
-      <anchor xyz="0 0 0" />
-      <limit effort="100" velocity="100" k_velocity="10" />
-      <calibration reference_position="${ref_position}" values="1.5 -1" />
-      <joint_properties damping="0.0" friction="0.0" />
-    </joint>
     <link name="${suffix}_caster_rotation_link">
-      <parent name="${parent}" />
-      <insert_block name="origin" />
-      <joint name="${suffix}_caster_rotation_joint" />
-      <inertial>
-        <mass value="3.473082" />
-        <com xyz="0 0 0.07" />
+      <joint name="${suffix}_caster_rotation_joint" type="revolute">
+        <origin xyz="0 0 0" rpy="0 0 0 0"/>
+        <axis xyz="0 0 1" />
+        <limit effort="100" velocity="100"/>
+        <safety_controller  k_velocity="10" />
+        <joint_properties damping="0.0" friction="0.0" />
+        <parent name="${parent}">
+          <insert_block name="origin" />
+        </parent>
+      </joint>
+      <inertial>
+        <mass value="3.473082"/>
+        <origin xyz="0 0 0.07" />
         <inertia  ixx="0.012411765597" ixy="-0.000711733678" ixz="0.00050272983"
                   iyy="0.015218160428" iyz="-0.000004273467" izz="0.011763977943" />
       </inertial>
-      <visual>
-        <origin xyz="0 0 0" rpy="0 0 0" />
-        <map name="gazebo_material" flag="gazebo">
-          <elem key="material" value="PR2/Green" />
-        </map>
-        <geometry name="${suffix}_caster_rotation_visual">
+      <visual name="${suffix}_caster_rotation_visual">
+        <origin xyz="0 0 0" rpy="0 0 0" />
+        <geometry name="${suffix}_caster_rotation_visual_geom">
           <mesh filename="caster.stlb" />
         </geometry>
-        <map name="${suffix}_caster_rotation_visual_mesh" flag="ogre">
-          <elem key="mesh" value="caster.mesh" />
-        </map>
-      </visual>
-      <collision>
+      </visual>
+      <collision name="${suffix}_caster_rotation_collision">
         <origin xyz="0 0 0.07" rpy="0.0 0.0 0.0" />
-        <geometry name="${suffix}_caster_rotation_collision">
+        <geometry name="${suffix}_caster_rotation_collision_geom">
           <box size="0.192 0.164 0.013" />
         </geometry>
       </collision>
     </link>
+    <ogre name="${suffix}_caster_rotation_visual_mesh" reference="${suffix}_caster_rotation_visual">
+      <elem key="mesh" value="caster.mesh" />
+    </ogre>
+    <ogre name="gazebo_material" reference="${suffix}_caster_rotation_visual">
+      <elem key="material" value="PR2/Green" />
+    </ogre>
     <transmission type="SimpleTransmission" name="${suffix}_caster_rotation_trans">
       <actuator name="${suffix}_caster_rotation_motor_alpha2" />
       <joint name="${suffix}_caster_rotation_joint" />
       <mechanicalReduction>79.226</mechanicalReduction>
+      <calibration reference_position="${ref_position}" values="1.5 -1" />
     </transmission>
     <!-- Double check these are right for the Alpha 2.0's -->
@@ -249,102 +250,115 @@
   </macro>
   <macro name="pr2_base_alpha2" params="name *origin">
-    <joint name="${name}_joint" type="planar" />
     <link name="${name}_link">
-      <parent name="world" />
-      <insert_block name="origin" />
-      <joint name="${name}_joint" />
+      <joint name="${name}_joint" type="planar">
+        <origin xyz="0 0 0" rpy="0 0 0" />
+        <parent name="world">
+          <insert_block name="origin" />
+        </parent>
+      </joint>
       <inertial>
         <mass value="${base_mass}" />
-        <com xyz="${base_cg_x} ${base_cg_y} ${base_cg_z}" />
+        <origin xyz="${base_cg_x} ${base_cg_y} ${base_cg_z}" />
         <inertia ixx="5.652232699207" ixy="-0.009719934438" ixz="1.293988226423"
                  iyy="5.669473158652" iyz="-0.007379583694" izz="3.683196351726" />
       </inertial>
-      <visual>
+      <visual name="${name}_visual">
         <origin xyz="0 0 ${base_height_offset}" rpy="0 0 0" />
-        <map name="gazebo_material" flag="gazebo">
-          <elem key="material" value="PR2/Green" />
-        </map>
-        <geometry name="${name}_visual">
+        <geometry name="${name}_visual_geom">
           <mesh filename="base.stlb" />
         </geometry>
-        <map name="${name}_visual_mesh" flag="ogre" >
-          <elem key="mesh" value="base.mesh" />
-        </map>
-      </visual>
-      <collision>
+      </visual>
+      <collision name="${name}_collision">
         <origin xyz="0 0 ${base_height_offset+base_size_z/2}" rpy="0 0 0" />
-        <geometry name="${name}_collision">
+        <geometry name="${name}_collision_geom">
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