Commit message: udpating new urdf.
git-svn-id: https://svn.code.sf.net/p/personalrobots/code/pkg/trunk@20489 f5854215-dd47-0410-b2c4-cdd35faa7885

Former-commit-id: 124cdf8a24bdb01a4308d1c42f8c91e8a202a2ac

File: stacks/pr2/pr2_defs/defs/arm_defs.urdf.xacro (robot description, xacro)
@@ -3,4 +3,6 @@
        xmlns:controller="http://playerstage.sourceforge.net/gazebo/xmlschema/#controller"
        xmlns:interface="http://playerstage.sourceforge.net/gazebo/xmlschema/#interface">
+  <include filename="$(find pr2_defs)/defs/arm_ext.xacro" />
+  <include filename="$(find pr2_defs)/defs/arm_cal.xacro" />
   <property name="M_PI" value="3.1415926535897931" />
   <property name="VELOCITY_LIMIT_SCALE" value="0.6" />
@@ -52,5 +54,5 @@
       <visual name="${side}_shoulder_pan_visual">
         <origin xyz="0 0 0" rpy="0 0 0" />
-        <geometry name="${side}_shoulder_pan_visual">
+        <geometry name="${side}_shoulder_pan_visual_geom">
           <mesh filename="shoulder_yaw.stlb" />
         </geometry>
@@ -59,44 +61,9 @@
       <collision name="${side}_shoulder_pan_collision">
         <origin xyz="0.0 0 0.0" rpy="0 0 0" />
-        <geometry name="${side}_shoulder_pan_collision">
+        <geometry name="${side}_shoulder_pan_collision_geom">
           <mesh filename="convex/shoulder_yaw_convex.stlb" />
         </geometry>
       </collision>
     </link>
-    <ogre name="${side}_shoulder_pan_collision_mesh" reference="${side}_shoulder_pan_collision">
-      <mesh value="convex/shoulder_yaw_convex.mesh" />
-    </ogre>
-    <ogre name="${side}_shoulder_pan_visual_mesh" reference="${side}_shoulder_pan_visual">
-      <mesh value="shoulder_yaw.mesh" />
-    </ogre>
-    <gazebo name="${side}_shoulder_pan_material" reference="${side}_shoulder_pan_visual">
-      <material value="PR2/Blue" />
-    </gazebo>
-    <gazebo name="${side}_shoulder_pan_sensor" reference="${side}_shoulder_pan_link">
-      <sensor:contact name="${side}_shoulder_pan_contact_sensor">
-        <geom>${side}_shoulder_pan_collision</geom>
-        <updateRate>100.0</updateRate>
-        <controller:ros_bumper name="${side}_shoulder_pan_ros_bumper_controller" plugin="libros_bumper.so">
-          <alwaysOn>true</alwaysOn>
-          <updateRate>100.0</updateRate>
-          <bumperTopicName>${side}_shoulder_pan_bumper</bumperTopicName>
-          <interface:bumper name="${side}_shoulder_pan_ros_bumper_iface" />
-        </controller:ros_bumper>
-      </sensor:contact>
-    <gazebo>
-    <gazebo name="${side}_shoulder_pan_gravity" reference="${side}_shoulder_pan_link">
-      <turnGravityOff>true</turnGravityOff>
-    </gazebo>
-    <gazebo name="${side}_shoulder_pan_joint_stop" reference="${side}_shoulder_pan_joint">
-      <stopKd value="1.0" />
-      <stopKp value="1000000.0" />
-    </gazebo>
-    <transmission type="SimpleTransmission" name="${side}_shoulder_pan_trans">
-      <actuator name="${side}_shoulder_pan_motor" />
-      <joint name="${side}_shoulder_pan_joint" />
-      <mechanicalReduction>${63.16/cal_r_shoulder_pan_gearing}</mechanicalReduction>
-      <calibration reference_position="${(reflect*M_PI/4)*cal_r_shoulder_pan_gearing+cal_r_shoulder_pan_flag}"
-                   values="1.5 -1" />
-    </transmission>
     <!-- Shoulder lift -->
     <link name="${side}_shoulder_lift_link">
@@ -123,5 +90,5 @@
       <visual name="${side}_shoulder_lift_visual">
         <origin xyz="0 0 0" rpy="0 0 0" />
-        <geometry name="${side}_shoulder_lift_visual">
+        <geometry name="${side}_shoulder_lift_visual_geom">
           <mesh filename="shoulder_lift.stlb" />
         </geometry>
@@ -130,43 +97,9 @@
       <collision name="${side}_shoulder_lift_collision">
         <origin xyz="0 0 0" rpy="0 0 0" />
-        <geometry name="${side}_shoulder_lift_collision">
+        <geometry name="${side}_shoulder_lift_collision_geom">
           <mesh filename="convex/shoulder_lift_convex.stlb" />
         </geometry>
       </collision>
     </link>
-    <ogre name="${side}_shoulder_lift_collision_mesh" reference="${side}_shoulder_lift_collision">
-      <mesh value="convex/shoulder_lift_convex.mesh" />
-    </ogre>
-    <gazebo name="${side}_shoulder_lift_sensor" reference="${side}_shoulder_lift_link">
-      <sensor:contact name="${side}_shoulder_lift_contact_sensor">
-        <geom>${side}_shoulder_lift_collision</geom>
-        <updateRate>100.0</updateRate>
-        <controller:ros_bumper name="${side}_shoulder_lift_ros_bumper_controller" plugin="libros_bumper.so">
-          <alwaysOn>true</alwaysOn>
-          <updateRate>100.0</updateRate>
-          <bumperTopicName>${side}_r_shoulder_lift_bumper</bumperTopicName>
-          <interface:bumper name="${side}_shoulder_lift_ros_bumper_iface" />
-        </controller:ros_bumper>
-      </sensor:contact>
-    </gazebo>
-    <gazebo name="${side}_shoulder_lift_gravity" reference="${side}_shoulder_lift_link">
-      <turnGravityOff>true</turnGravityOff>
-    </gazebo>
-    <ogre name="gazebo_material" reference="${side}_shoulder_lift_visual">
-      <material value="PR2/Grey" />
-    </ogre>
-    <ogre name="${side}_shoulder_lift_visual_mesh" reference="${side}_shoulder_lift_visual">
-      <mesh value="shoulder_lift.mesh" />
-    </ogre>
-    <gazebo name="${side}_shoulder_lift_joint_stop" reference="${side}_shoulder_lift_joint">
-      <stopKd value="1.0" />
-      <stopKp value="1000000.0" />
-    </gazebo>
-    <transmission type="SimpleTransmission" name="${side}_shoulder_lift_trans">
-      <actuator name="${side}_shoulder_lift_motor" />
-      <joint name="${side}_shoulder_lift_joint" />
-      <mechanicalReduction>${61.89/cal_r_shoulder_lift_gearing}</mechanicalReduction>
-      <calibration reference_position="cal_r_shoulder_lift_flag" values="1.5 -1" />
-    </transmission>
     <!-- Upperarm roll: internal fixed attchment point for upper arm -->
     <link name="${side}_upper_arm_roll_link">
@@ -189,5 +122,6 @@
                   izz="0.01" />
       </inertial>
-      <visual name="${side}_upper_arm_roll_visual"> <!-- TODO: This component doesn't actually have a mesh -->
+      <visual name="${side}_upper_arm_roll_visual">
+        <!-- TODO: This component doesn't actually have a mesh -->
         <origin xyz="0 0 0" rpy="0 0 0" />
         <geometry name="${side}_upper_arm_roll_visual_geom">
@@ -195,5 +129,6 @@
         </geometry>
       </visual>
-      <collision name="${side}_upper_arm_roll_collision"> <!-- TODO: collision tag should be optional -->
+      <collision name="${side}_upper_arm_roll_collision">
+        <!-- TODO: collision tag should be optional -->
         <origin xyz="0.0 0 0" rpy="0 0 0" />
         <geometry name="${side}_upper_arm_roll_collision_geom">
@@ -202,24 +137,4 @@
       </collision>
     </link>
-    <gazebo name="${side}_upper_arm_roll_gravity" reference="${side}_upper_arm_roll_collision">
-      <turnGravityOff>true</turnGravityOff>
-    </gazebo>
-    <gazebo name="gazebo_material" reference=name="${side}_upper_arm_roll_visual">
-      <material value="PR2/RollLinks" />
-    </gazebo>
-    <ogre name="${side}_upper_arm_roll_visual_mesh" reference=name="${side}_upper_arm_roll_visual">
-      <mesh value="upper_arm_roll.mesh" />
-    </ogre>
-    <gazebo name="${side}_upper_arm_roll_joint_ode" reference="${side}_upper_arm_roll_joint">
-      <stopKd value="1.0" />
-      <stopKp value="1000000.0" />
-      <fudgeFactor value="0.5" />
-    </gazebo>
-    <transmission type="SimpleTransmission" name="${side}_upper_arm_roll_trans">
-      <actuator name="${side}_upper_arm_roll_motor" />
-      <joint name="${side}_upper_arm_roll_joint" />
-      <mechanicalReduction>${32.65/cal_r_upper_arm_roll_gearing}</mechanicalReduction>
-      <calibration reference_position="${(reflect*M_PI/2)*cal_r_upper_arm_roll_gearing + cal_r_upper_arm_roll_flag}" values="1.5 -1" />
-    </transmission>
   </macro>
   <!-- ============================   Upper Arm   ============================ -->
@@ -256,28 +171,4 @@
       </collision>
     </link>
-    <ogre name="${side}_upper_arm_visual_mesh" reference="{side}_upper_arm_visual">
-      <mesh value="upper_arm.mesh" />
-    </ogre>
-    <ogre name="${side}_upper_arm_collision_mesh" reference="${side}_upper_arm_collision">
-      <mesh value="convex/upper_arm_convex.mesh" />
-    </ogre>
-    <gazebo name="${side}_upper_arm_sensor" reference="${side}_upper_arm_link">
-      <sensor:contact name="${side}_upper_arm_contact_sensor">
-        <geom>${side}_upper_arm_collision</geom><!-- TODO -->
-        <updateRate>100.0</updateRate>
-        <controller:ros_bumper name="${side}_upper_arm_ros_bumper_controller" plugin="libros_bumper.so">
-          <alwaysOn>true</alwaysOn>
-          <updateRate>100.0</updateRate>
-          <bumperTopicName>${side}_upper_arm_bumper</bumperTopicName>
-          <interface:bumper name="${side}_upper_arm_ros_bumper_iface" />
-        </controller:ros_bumper>
-      </sensor:contact>
-    </gazebo>
-    <gazebo name="${side}_upper_arm_gravity" reference="${side}_upper_arm_link">
-      <turnGravityOff>true</turnGravityOff>
-    </gazebo>
-    <gazebo name="gazebo_material" reference="{side}_upper_arm_visual">
-      <material value="PR2/Green" />
-    </gazebo>
     <!-- Elbow flex -->
     <link name="${side}_elbow_flex_link">
@@ -312,38 +203,4 @@
       </collision>
     </link>
-    <ogre name="${side}_elbow_flex_visual_mesh" reference="${side}_elbow_flex_visual">
-      <mesh value="elbow_flex.mesh" />
-    </ogre>
-    <ogre name="${side}_elbow_flex_collision_mesh" reference="${side}_elbow_flex_collision">
-      <mesh value="convex/elbow_flex_convex.mesh" />
-    </ogre>
-    <gazebo name="${side}_elbow_flex_joint_ode" reference="${side}_elbow_flex_joint">
-      <stopKd value="1.0" />
-      <stopKp value="1000000.0" />
-    </gazebo>
-    <gazebo name="gazebo_material" reference="${side}_elbow_flex_visual">
-      <material value="PR2/Grey" />
-    </gazebo>
-    <gazebo name="${side}_elbow_flex_sensor" reference="${side}_elbow_flex_link">
-      <sensor:contact name="${side}_elbow_flex_contact_sensor">
-        <geom>${side}_elbow_flex_collision</geom>
-        <updateRate>100.0</updateRate>
-        <controller:ros_bumper name="${side}_elbow_flex_ros_bumper_controller" plugin="libros_bumper.so">
-          <alwaysOn>true</alwaysOn>
-          <updateRate>100.0</updateRate>
-          <bumperTopicName>${side}_elbow_flex_bumper</bumperTopicName>
-          <interface:bumper name="${side}_elbow_flex_ros_bumper_iface" />
-        </controller:ros_bumper>
-      </sensor:contact>
-    </gazebo>
-    <gazebo name="${side}_elbow_flex_gravity" reference="${side}_elbow_flex_link">
-      <turnGravityOff>true</turnGravityOff>
-    </gazebo>
-    <transmission type="SimpleTransmission" name="${side}_elbow_flex_trans">
-      <actuator name="${side}_elbow_flex_motor" />
-      <joint name="${side}_elbow_flex_joint" />
-      <mechanicalReduction>-36.17</mechanicalReduction>
-      <calibration reference_position="${-1.1606 + cal_r_elbow_flex_flag}" values="1.5 -1" />
-    </transmission>
     <!-- Forearm roll -->
     <link name="${side}_forearm_roll_link">
@@ -379,22 +236,4 @@
       </collision>
     </link>
-    <ogre name="${side}_forearm_roll_visual_mesh" reference="${side}_forearm_roll_visual">
-      <mesh value="forearm_roll.mesh" />
-    </ogre>
-    <gazebo name="gazebo_material" reference="${side}_forearm_roll_visual">
-      <material value="PR2/RollLinks" />
-    </gazebo>
-    <gazebo name="${side}_forearm_roll_joint_ode" reference="${side}_forearm_roll_joint">
-      <fudgeFactor value="0.5" />
-    </gazebo>
-    <gazebo name="${side}_forearm_roll_gravity" reference="${side}_forearm_roll_link">
-      <turnGravityOff>true</turnGravityOff>
-    </gazebo>
-    <transmission type="SimpleTransmission" name="${side}_forearm_roll_trans">
-      <actuator name="${side}_forearm_roll_motor" />
-      <joint name="${side}_forearm_roll_joint" />
-      <mechanicalReduction>${576/25*55/14}</mechanicalReduction>
-      <calibration reference_position="cal_r_forearm_roll_flag" values="1.5 -1" />
-    </transmission>
   </macro>
   <!-- ============================   Forearm   ============================ -->
@@ -427,28 +266,4 @@
       </collision>
     </link>
-    <gazebo name="${side}_forearm_gravity" reference="${side}_forearm_link">
-      <turnGravityOff>true</turnGravityOff>
-    </gazebo>
-    <gazebo name="${side}_forearm_sensor" reference="${side}_forearm_link">
-      <sensor:contact name="${side}_forearm_contact_sensor">
-        <geom>${side}_forearm_collision</geom>
-        <updateRate>100.0</updateRate>
-        <controller:ros_bumper name="${side}_forearm_ros_bumper_controller" plugin="libros_bumper.so">
-          <alwaysOn>true</alwaysOn>
-          <updateRate>100.0</updateRate>
-          <bumperTopicName>${side}_forearm_bumper</bumperTopicName>
-          <interface:bumper name="${side}_forearm_ros_bumper_iface" />
-        </controller:ros_bumper>
-      </sensor:contact>
-    </gazebo>
-    <gazebo name="gazebo_material" reference="${side}_forearm_visual">
-      <material value="PR2/Blue" />
-    </gazebo>
-    <ogre name="${side}_forearm_collision_mesh" reference="${side}_forearm_collision">
-      <mesh value="convex/forearm_convex.mesh" />
-    </ogre>
-    <ogre name="${side}_forearm_visual_mesh" reference="${side}_forearm_visual">
-      <mesh value="forearm.mesh" />
-    </ogre>
     <!-- Wrist flex -->
     <link name="${side}_wrist_flex_link">
@@ -483,32 +298,4 @@
       </collision>
     </link>
-    <gazebo name="${side}_wrist_flex_gravity" reference="${side}_wrist_flex_link">
-      <turnGravityOff>true</turnGravityOff>
-    </gazebo>
-    <gazebo name="${side}_wrist_flex_sensor" reference="${side}_wrist_flex_link">
-      <sensor:contact name="${side}_wrist_flex_contact_sensor">
-        <geom>${side}_wrist_flex_collision</geom>
-        <updateRate>100.0</updateRate>
-        <controller:ros_bumper name="${side}_wrist_flex_ros_bumper_controller" plugin="libros_bumper.so">
-          <alwaysOn>true</alwaysOn>
-          <updateRate>100.0</updateRate>
-          <bumperTopicName>${side}_wrist_flex_bumper</bumperTopicName>
-          <interface:bumper name="${side}_wrist_flex_ros_bumper_iface" />
-        </controller:ros_bumper>
-      </sensor:contact>
-    </gazebo>
-    <gazebo name="gazebo_material" reference="${side}_wrist_flex_visual">
-      <material value="PR2/Grey" />
-    </gazebo>
-    <gazebo name="${side}_wrist_flex_joint_ode" reference="${side}_wrist_flex_joint">
-      <stopKd value="1.0" />
-      <stopKp value="1000000.0" />
-    </gazebo>
-    <ogre name="${side}_wrist_flex_collision_mesh" reference="${side}_wrist_flex_collision">
-      <mesh value="convex/wrist_flex_convex.mesh" />
-    </ogre>
-    <ogre name="${side}_wrist_flex_visual_mesh" reference="${side}_wrist_flex_visual">
-      <mesh value="wrist_flex.mesh" />
-    </ogre>
     <!-- Wrist roll -->
     <link name="${side}_wrist_roll_link">
@@ -544,38 +331,4 @@
       </collision>
     </link>
-    <gazebo name="${side}_wrist_roll_gravity" reference="${side}_wrist_roll_link">
-      <turnGravityOff>true</turnGravityOff>
-    </gazebo>
-    <gazebo name="${side}_wrist_roll_sensor" reference="${side}_wrist_roll_link">
-      <sensor:contact name="${side}_wrist_roll_contact_sensor">
-        <geom>${side}_wrist_roll_collision</geom>
-        <updateRate>100.0</updateRate>
-        <controller:ros_bumper name="${side}_wrist_roll_ros_bumper_controller" plugin="libros_bumper.so">
-          <alwaysOn>true</alwaysOn>
-          <updateRate>100.0</updateRate>
-          <bumperTopicName>${side}_wrist_roll_bumper</bumperTopicName>
-          <interface:bumper name="${side}_wrist_roll_ros_bumper_iface" />
-        </controller:ros_bumper>
-      </sensor:contact>
-    </gazebo>
-    <ogre name="${side}_wrist_roll_visual_mesh" reference="${side}_wrist_roll_visual">
-      <mesh value="wrist_roll.mesh" />
-    </ogre>
-    <ogre name="gazebo_material" reference="${side}_wrist_roll_visual">
-      <material value="PR2/RollLinks" />
-    </ogre>
-    <gazebo name="${side}_wrist_roll_joint_ode" reference="${side}_wrist_roll_joint">
-      <fudgeFactor value="0.5" />
-    </gazebo>
-    <transmission type="WristTransmission" name="${side}_wrist_trans">
-      <rightActuator name="${side}_wrist_r_motor" />
-      <leftActuator name="${side}_wrist_l_motor" />
-      <flexJoint name="${side}_wrist_flex_joint" mechanicalReduction="${624/35*54/16}">
-        <calibration reference_position="${0.4363+cal_r_wrist_flex_flag}" values="1.5 -1" />
-      </flexJoint>
-      <rollJoint name="${side}_wrist_roll_joint" mechanicalReduction="${624/35*54/16}" >
-      </rollJoint>
-      <calibration reference_position="${1.27+cal_r_wrist_roll_flag}" values="1.5 -1" />
-    </transmission>
   </macro>
   <macro name="pr2_arm" params="side parent reflect *origin">
@@ -585,55 +338,10 @@
     <pr2_upper_arm side="${side}" reflect="${reflect}" parent="${side}_upper_arm_roll_link" />
     <pr2_forearm side="${side}" reflect="${reflect}" parent="${side}_forearm_roll_link" />
-  </macro>
-  <!--                    Calibration                            -->
-  <macro name="upper_arm_calibrator" params="side">
-    <controller name="${side}_cal_shoulder_pan" topic="${side}_cal_shoulder_pan"
-                type="JointUDCalibrationControllerNode">
-      <calibrate joint="${side}_shoulder_pan_joint"
-                 actuator="${side}_shoulder_pan_motor"
-                 transmission="${side}_shoulder_pan_trans"
-                 velocity="1.0" />
-      <pid p="7" i="0.5" d="0" iClamp="1.0" />
-    </controller>
-    <controller name="cal_shoulder_lift_${side}" topic="cal_shoulder_lift_${side}"
-                type="JointUDCalibrationControllerNode">
-      <calibrate joint="${side}_shoulder_lift_joint"
-                 actuator="${side}_shoulder_lift_motor"
-                 transmission="${side}_shoulder_lift_trans"
-                 velocity="-1.0" />
-      <pid p="9" i="1.0" d="0" iClamp="6.0" />
-    </controller>
-    <controller name="cal_${side}_upper_arm_roll" topic="cal_${side}_upper_arm_roll"
-                type="JointUDCalibrationControllerNode">
-      <calibrate joint="${side}_upper_arm_roll_joint"
-                 actuator="${side}_upper_arm_roll_motor"
-                 transmission="${side}_upper_arm_roll_trans"
-                 velocity="1.0" />
-      <pid p="6" i="0.2" d="0" iClamp="2.0" />
-    </controller>
-    <controller name="cal_${side}_elbow_flex" topic="cal_${side}_elbow_flex"
-                type="JointUDCalibrationControllerNode">
-      <calibrate joint="${side}_elbow_flex_joint"
-                 actuator="${side}_elbow_flex_motor"
-                 transmission="${side}_elbow_flex_trans"
-                 velocity="-1.0" />
-      <pid p="6" i="0.2" d="0" iClamp="1.0" />
-    </controller>
-  </macro>
-  <macro name="forearm_calibrator" params="side">
-    <controller name="cal_${side}_forearm_roll" type="JointUDCalibrationControllerNode">
-      <calibrate joint="${side}_forearm_roll_joint"
-                 actuator="${side}_forearm_roll_motor"
-                 transmission="${side}_forearm_roll_trans"
-                 velocity="-1.2" />
-      <pid p="5.0" i="0" d="0" iClamp="0" />
-    </controller>
-    <controller type="WristCalibrationControllerNode" name="cal_${side}_wrist">
-      <calibrate transmission="${side}_wrist_trans"
-                 actuator_l="${side}_wrist_l_motor" actuator_r="${side}_wrist_r_motor"
-                 flex_joint="${side}_wrist_flex_joint" roll_joint="${side}_wrist_roll_joint"
-                 velocity="1.2" />
-      <pid p="3.0" i="0.2" d="0" iClamp="2.0" />
-    </controller>
+    <!-- gazebo / ogre / transmission extensions -->
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