Commit message: update new urdf.
git-svn-id: https://svn.code.sf.net/p/personalrobots/code/pkg/trunk@20509 f5854215-dd47-0410-b2c4-cdd35faa7885

Former-commit-id: 2d672f0b9e91dc7fdc48e462e548b754273c0e7c

File: stacks/pr2/pr2_defs/defs/base_defs.urdf.xacro (robot description, xacro)
@@ -34,5 +34,5 @@
         <joint_properties damping="0.0" friction="0.0" />
         <parent name="${parent}_rotation_link">
-          <joint name="${parent}_${suffix}_wheel_joint" type="revolute">
+          <joint name="${parent}_${suffix}_wheel_joint" type="revolute"/>
         </parent>
       </joint>
@@ -98,5 +98,5 @@
         <joint_properties damping="0.0" friction="0.0" />
         <parent name="${parent}">
-          <insert_block name="origin">
+          <insert_block name="origin"/>
         </parent>
       </joint>
@@ -433,5 +433,5 @@
         <origin xyz="0 0 0" rpy="0 0 0" />
         <axis xyz="0 1 0" />
-        <parent name="${name}_link" />
+        <parent name="${name}_link">
           <origin xyz="${base_laser_x} ${base_laser_y} ${base_height_offset+base_laser_z}" rpy="0 0 0" />
         </parent>
@@ -487,5 +487,5 @@
         <axis xyz="0 1 0" />
         <anchor xyz="0 0 0" />
-        <parent name="${name}_link" />
+        <parent name="${name}_link">
           <origin xyz="0.18 0 ${base_height_offset+0.235}" rpy="0 0 0" />
         </parent>

File: stacks/pr2/pr2_defs/defs/gripper_defs.urdf.xacro (robot description, xacro)
@@ -96,5 +96,5 @@
       <initialAngle value="${gripper_min_angle}"/>
     </gazebo>
-    <ogre reference="${prefix}_l_finger_collision" name="mesh" reference="${prefix}_l_finger_collision">
+    <ogre name="mesh" reference="${prefix}_l_finger_collision">
       <type value="visual"/>
     </ogre>
@@ -222,5 +222,5 @@
     </link>
     <gazebo name="${prefix}_l_finger_tip_gravity" reference="${prefix}_l_finger_tip_link">
-      <turnGravityOff>true</mimicKp>
+      <turnGravityOff>true</turnGravityOff>
       <selfCollide value="false" />
     </gazebo>
@@ -470,5 +470,4 @@
           <axis>0 1 0</axis>
           <anchorOffset>0 0 0</anchorOffset>
-          </anchorOffset>
       </joint:slider>
       <joint:slider name="${side}_gripper_r_finger_tip_slider_joint">
