Commit message: Add resource locations to rviz extension defs
git-svn-id: https://svn.code.sf.net/p/personalrobots/code/pkg/trunk@21755 f5854215-dd47-0410-b2c4-cdd35faa7885

Former-commit-id: 6c37f10ac8cc2198cb6ce0cf29b754c6dd4bea7b

File: stacks/pr2/pr2_defs/defs/arm_rviz.xacro (robot description, xacro)
@@ -1,4 +1,6 @@
 <?xml version="1.0"?>
 <robot>
+  <rviz_resource_location path="$(find pr2_ogre)/Media/materials/scripts"/>
+  <rviz_resource_location path="$(find pr2_ogre)/Media/materials/textures"/>
   <macro name="pr2_shoulder_rviz" params="side">
     <rviz reference="${side}_shoulder_pan_link">

File: stacks/pr2/pr2_defs/defs/base_rviz.xacro (robot description, xacro)
@@ -1,4 +1,6 @@
 <?xml version="1.0"?>
 <robot>
+  <rviz_resource_location path="$(find pr2_ogre)/Media/materials/scripts"/>
+  <rviz_resource_location path="$(find pr2_ogre)/Media/materials/textures"/>
   <macro name="pr2_wheel_rviz" params="suffix parent">
     <rviz reference="${parent}_${suffix}_wheel_link">

File: stacks/pr2/pr2_defs/defs/body_rviz.xacro (robot description, xacro)
@@ -1,4 +1,6 @@
 <?xml version="1.0"?>
 <robot>
+  <rviz_resource_location path="$(find pr2_ogre)/Media/materials/scripts"/>
+  <rviz_resource_location path="$(find pr2_ogre)/Media/materials/textures"/>
   <macro name="pr2_torso_rviz" params="name parent">
     <rviz reference="${name}_link">

File: stacks/pr2/pr2_defs/defs/gripper_rviz.xacro (robot description, xacro)
@@ -1,4 +1,6 @@
 <?xml version="1.0"?>
 <robot>
+  <rviz_resource_location path="$(find pr2_ogre)/Media/materials/scripts"/>
+  <rviz_resource_location path="$(find pr2_ogre)/Media/materials/textures"/>
   <macro name="pr2_finger_rviz" params="prefix">
     <rviz reference="${prefix}_l_finger_link">

File: stacks/pr2/pr2_defs/defs/head_rviz.xacro (robot description, xacro)
@@ -1,4 +1,6 @@
 <?xml version="1.0"?>
 <robot>
+  <rviz_resource_location path="$(find pr2_ogre)/Media/materials/scripts"/>
+  <rviz_resource_location path="$(find pr2_ogre)/Media/materials/textures"/>
   <macro name="pr2_tilting_laser_rviz" params="name parent *origin">
     <rviz reference="${name}_mount_link">

File: stacks/pr2/pr2_defs/defs/mono_cam_rviz.xacro (robot description, xacro)
@@ -1,4 +1,6 @@
 <?xml version="1.0"?>
 <root>
+  <rviz_resource_location path="$(find pr2_ogre)/Media/materials/scripts"/>
+  <rviz_resource_location path="$(find pr2_ogre)/Media/materials/textures"/>
   <macro name="mono_cam_rviz" params="name">
     <rviz reference="${name}_link">

File: stacks/pr2/pr2_defs/defs/prosilica_rviz.xacro (robot description, xacro)
@@ -1,11 +1,13 @@
 <?xml version="1.0"?>
 <root>
-<macro name="prosilica_cam_rviz" params="name">
-  <rviz reference="${name}_link">
-    <material value="PR2/Blue" />
-  </rviz>
-  <rviz reference="${name}_optical_link">
-    <material value="PR2/Blue" />
-  </rviz>
-</macro>
+  <rviz_resource_location path="$(find pr2_ogre)/Media/materials/scripts"/>
+  <rviz_resource_location path="$(find pr2_ogre)/Media/materials/textures"/>
+  <macro name="prosilica_cam_rviz" params="name">
+    <rviz reference="${name}_link">
+      <material value="PR2/Blue" />
+    </rviz>
+    <rviz reference="${name}_optical_link">
+      <material value="PR2/Blue" />
+    </rviz>
+  </macro>
 </root>
