Commit message: Fix material for X_caster_rotation_link, in new urdf
git-svn-id: https://svn.code.sf.net/p/personalrobots/code/pkg/trunk@21896 f5854215-dd47-0410-b2c4-cdd35faa7885

Former-commit-id: c5aabef7c0f81d6347258056efa0d3e3dc738e73

File: stacks/pr2/pr2_defs/defs/base/base_rviz.xacro (robot description, xacro)
@@ -11,5 +11,5 @@
   <macro name="pr2_caster_rviz" params="suffix">
     <rviz reference="${suffix}_caster_rotation_link">
-      <elem key="material" value="PR2/Green" />
+      <material value="PR2/Green" />
     </rviz>
   </macro>
