Commit message: making urdf copy of all .xacro.xml robot files.
git-svn-id: https://svn.code.sf.net/p/personalrobots/code/pkg/trunk@22213 f5854215-dd47-0410-b2c4-cdd35faa7885

Former-commit-id: 52402e222d12408dca4cd3320dcec3b4d4a219c6

File: stacks/pr2/pr2_defs/defs/arm/mono_cam_defs.urdf.xacro (robot description, xacro)
@@ -30,7 +30,7 @@
       </collision>
     </link>
-    <joint name="${name}_optical_frame_joint" type="fixed" />
+    <joint name="${name}_optical_frame_joint" type="fixed">
       <origin xyz="0 0 0" rpy="${-M_PI/2} 0.0 ${-M_PI/2}" />
-      <parent link="${name}_frame" //>
+      <parent link="${name}_frame" />
       <child link="${name}_optical_frame"/>
     </joint>

File: stacks/pr2/pr2_defs/defs/arm/mono_cam_gazebo.xacro (robot description, xacro)
@@ -1,6 +1,8 @@
 <?xml version="1.0"?>
-<root>
+<robot xmlns:sensor="http://playerstage.sourceforge.net/gazebo/xmlschema/#sensor"
+       xmlns:controller="http://playerstage.sourceforge.net/gazebo/xmlschema/#controller"
+       xmlns:interface="http://playerstage.sourceforge.net/gazebo/xmlschema/#interface">
   <macro name="mono_cam_gazebo" params="name">
-  <gazebo reference="${name}_optical_frame">
+    <gazebo reference="${name}_optical_frame">
       <sensor:camera name="${name}_sensor">
         <imageSize>640 480</imageSize>
@@ -22,3 +24,3 @@
     </gazebo>
   </macro>
-</root>
+</robot>

File: stacks/pr2/pr2_defs/defs/base/alpha2_base_defs.urdf.xacro (robot description, xacro)
@@ -3,9 +3,11 @@
        xmlns:controller="http://playerstage.sourceforge.net/gazebo/xmlschema/#controller"
        xmlns:interface="http://playerstage.sourceforge.net/gazebo/xmlschema/#interface">
-  <!--include filename="$(find pr2_defs)/defs/base_rviz.xacro" /-->
-  <include filename="$(find pr2_defs)/defs/base/alpha_base_rviz.xacro" />
-  <include filename="$(find pr2_defs)/defs/base/alpha_base_gazebo.xacro" />
-  <include filename="$(find pr2_defs)/defs/base/alpha_base_transmission.xacro" />
+  <include filename="$(find pr2_defs)/defs/base/alpha2_base_rviz.xacro" />
+  <include filename="$(find pr2_defs)/defs/base/alpha2_base_gazebo.xacro" />
+  <include filename="$(find pr2_defs)/defs/base/alpha2_base_transmission.xacro" />
   <property name="M_PI" value="3.1415926535897931" />
+  <property name="caster_offset_x" value="0.2225" />
+  <property name="caster_offset_y" value="0.2225" />
+  <property name="caster_offset_z" value="0.0282" />
   <property name="caster_wheel_offset_y" value="0.049" /> <!-- from function spreadsheet -->
   <property name="wheel_length" value="0.03" />  <!-- FIXME -->
@@ -14,5 +16,5 @@
   <property name="base_cg_x" value="-0.061" />
   <property name="base_cg_y" value="0.0" />
-  <property name="base_cg_z" value="0.293" //>
+  <property name="base_cg_z" value="0.293" />
   <property name="base_mass" value="116.0" />
   <!-- base appears "raised" from our initial geom def from function -->

File: stacks/pr2/pr2_defs/defs/head/alpha2_head_defs.urdf.xacro (robot description, xacro)
@@ -3,7 +3,7 @@
        xmlns:controller="http://playerstage.sourceforge.net/gazebo/xmlschema/#controller"
        xmlns:interface="http://playerstage.sourceforge.net/gazebo/xmlschema/#interface">
-  <include filename="$(find pr2_defs)/defs/alpha2_head_rviz.xacro" />
-  <include filename="$(find pr2_defs)/defs/alpha2_head_gazebo.xacro" />
-  <include filename="$(find pr2_defs)/defs/alpha2_head_transmission.xacro" />
+  <include filename="$(find pr2_defs)/defs/head/alpha2_head_rviz.xacro" />
+  <include filename="$(find pr2_defs)/defs/head/alpha2_head_gazebo.xacro" />
+  <include filename="$(find pr2_defs)/defs/head/alpha2_head_transmission.xacro" />
   <property name="M_PI" value="3.1415926535897931" />
   <!-- Alpha 2.0 head -->

File: stacks/pr2/pr2_defs/defs/head/alpha2_head_gazebo.xacro (robot description, xacro)
@@ -16,4 +16,5 @@
     <gazebo reference="${name}_link">
       <material value="PR2/Green" />
+    </gazebo>
   </macro>
   <macro name="pr2_head_tilt_alpha2a_gazebo" params="name">
