Commit message: update in progress per api review 2.
git-svn-id: https://svn.code.sf.net/p/personalrobots/code/pkg/trunk@22081 f5854215-dd47-0410-b2c4-cdd35faa7885

Former-commit-id: 7de6fa334d42e90f123729333438e2f6b8f89a31

File: stacks/pr2/pr2_defs/defs/arm/arm_defs.urdf.xacro (robot description, xacro)
@@ -32,11 +32,8 @@
     <!-- Shoulder pan -->
     <joint name="${side}_shoulder_pan_joint" type="revolute">
-      <!-- transform from link to joint frame -->
-      <origin xyz="0 0 0" rpy="0 0 0"/>
       <axis xyz="0 0 1" />
-      <parent name="${parent}">
-        <!-- transform from parent link to this joint frame -->
-        <insert_block name="origin" />
-      </parent>
+      <insert_block name="origin" /> <!-- transform from parent link to this joint frame -->
+      <parent link="${parent}"/>
+      <child link="${side}_shoulder_pan_link"/>
       <limit lower="${reflect*M_PI/4-1.5}"  upper="${reflect*M_PI/4+1.5}"
              effort="30" velocity="${VELOCITY_LIMIT_SCALE*3.48}" />
@@ -72,5 +69,4 @@
     <!-- Shoulder lift -->
     <joint name="${side}_shoulder_lift_joint" type="revolute">
-      <origin xyz="0 0 0" rpy="0 0 0"/>
       <axis xyz="0 1 0"/>
       <!-- Limits updated from Function's CAD values as of 2009_02_24 (link_data.xls) -->
@@ -81,7 +77,7 @@
       <calibration reference_position="${cal_r_shoulder_lift_flag}" />
       <dynamics damping="10.0" />
-      <parent name="${side}_shoulder_pan_link">
-        <origin xyz="0.1 0 0" rpy="0 0 0" />
-      </parent>
+      <origin xyz="0.1 0 0" rpy="0 0 0" />
+      <parent link="${side}_shoulder_pan_link"/>
+      <child link="${side}_shoulder_lift_link"/>
     </joint>
     <link name="${side}_shoulder_lift_link">
@@ -109,9 +105,8 @@
     <!-- Upperarm roll: internal fixed attchment point for upper arm -->
     <joint name="${side}_upper_arm_roll_joint" type="revolute">
-      <origin xyz="0 0 0" rpy="0 0 0" />
       <axis xyz="1 0 0" />
-      <parent name="${side}_shoulder_lift_link" >
-        <origin xyz="0 0 0" rpy="0 0 0" />
-      </parent>
+      <origin xyz="0 0 0" rpy="0 0 0" />
+      <parent link="${side}_shoulder_lift_link" />
+      <child link="${side}_upper_arm_roll_link"/>
       <limit lower="${reflect*1.55-2.35}" upper="${reflect*1.55+2.35}" effort="30" velocity="${VELOCITY_LIMIT_SCALE*5.45}" />
       <safety_controller k_position="100" k_velocity="2" soft_lower_limit="${reflect*1.55-2.35+0.15}" soft_upper_limit="${reflect*1.55+2.35-0.15}" />
@@ -148,7 +143,6 @@
     <joint name="${side}_upper_arm_joint" type="fixed">
       <origin xyz="0 0 0" rpy="0 0 0" />
-      <parent name="${parent}">
-        <origin xyz="0 0 0" rpy="0 0 0" />
-      </parent>
+      <parent link="${parent}"/>
+      <child link="${side}_upper_arm_link"/>
     </joint>
     <link name="${side}_upper_arm_link">
@@ -179,5 +173,4 @@
     <!-- Elbow flex -->
     <joint name="${side}_elbow_flex_joint" type="revolute">
-      <origin xyz="0 0 0" rpy="0 0 0" />
       <axis xyz="0 1 0" />
       <limit lower="-2.3" upper="0.1" effort="30" velocity="${VELOCITY_LIMIT_SCALE*5.5}" />
@@ -185,7 +178,7 @@
       <calibration reference_position="${-1.1606 + cal_r_elbow_flex_flag}"/>
       <dynamics damping="1.0" />
-      <parent name="${side}_upper_arm_link">
-        <origin xyz="0.4 0 0" rpy="0 0 0" />
-      </parent>
+      <origin xyz="0.4 0 0" rpy="0 0 0" />
+      <parent link="${side}_upper_arm_link"/>
+      <child link="${side}_elbow_flex_link"/>
     </joint>
     <link name="${side}_elbow_flex_link">
@@ -212,5 +205,4 @@
     <!-- Forearm roll -->
     <joint name="${side}_forearm_roll_joint" type="continuous">
-      <origin xyz="0 0 0" rpy="0 0 0" />
       <axis xyz="-1 0 0" />
       <limit effort="30" velocity="${VELOCITY_LIMIT_SCALE*6}" />
@@ -218,7 +210,7 @@
       <calibration reference_position="${cal_r_forearm_roll_flag}" />
       <dynamics damping="0.1" />
-      <parent name="${side}_elbow_flex_link">
-        <origin xyz="0 0 0" rpy="0 0 0" />
-      </parent>
+      <origin xyz="0 0 0" rpy="0 0 0" />
+      <parent link="${side}_elbow_flex_link"/>
+      <child link="${side}_forearm_roll_link"/>
     </joint>
     <link name="${side}_forearm_roll_link">
@@ -249,7 +241,6 @@
     <joint name="${side}_forearm_joint" type="fixed">
       <origin xyz="0 0 0" rpy="0 0 0" />
-      <parent name="${parent}">
-        <origin xyz="0 0 0" rpy="0 0 0" />
-      </parent>
+      <parent link="${parent}"/>
+      <child link="${side}_forearm_link"/>
     </joint>
     <link name="${side}_forearm_link">
@@ -276,5 +267,4 @@
     <!-- Wrist flex -->
     <joint name="${side}_wrist_flex_joint" type="revolute">
-      <origin xyz="0 0 0" rpy="0 0 0" />
       <axis xyz="0 -1 0" />
       <limit lower="-0.1" upper="2.2" effort="200" velocity="${VELOCITY_LIMIT_SCALE*5.13}" />
@@ -282,7 +272,7 @@
       <dynamics damping="0.1" />
       <calibration reference_position="${0.4363+cal_r_wrist_flex_flag}" />
-      <parent name="${side}_forearm_link">
-        <origin xyz="0.32025 0 0" rpy="0 0 0" />
-      </parent>
+      <origin xyz="0.32025 0 0" rpy="0 0 0" />
+      <parent link="${side}_forearm_link"/>
+      <child link="${side}_wrist_flex_link"/>
     </joint>
     <link name="${side}_wrist_flex_link">
@@ -309,12 +299,11 @@
     <!-- Wrist roll -->
     <joint name="${side}_wrist_roll_joint" type="continuous">
-      <origin xyz="0 0 0" rpy="0 0 0" />
       <axis xyz="1 0 0" />
       <limit effort="10" velocity="${VELOCITY_LIMIT_SCALE*6}" k_velocity="2" />
       <dynamics damping="0.1" />
       <calibration reference_position="${1.27+cal_r_wrist_roll_flag}" values="1.5 -1" />
-      <parent name="${side}_wrist_flex_link">
-        <origin xyz="0 0 0" rpy="0 0 0" />
-      </parent>
+      <origin xyz="0 0 0" rpy="0 0 0" />
+      <parent link="${side}_wrist_flex_link"/>
+      <child link="${side}_wrist_roll_link"/>
     </joint>
     <link name="${side}_wrist_roll_link">

File: stacks/pr2/pr2_defs/defs/arm/mono_cam_defs.urdf.xacro (robot description, xacro)
@@ -5,8 +5,7 @@
   <macro name="mono_cam" params="name parent *origin">
     <joint name="${name}_frame_joint" type="fixed">
-      <origin xyz="0 0 0" />
-      <parent name="${parent}">
-        <insert_block name="origin" />
-      </parent>
+      <insert_block name="origin" />
+      <parent link="${parent}"/>
+      <child link="${name}_frame"/>
     </joint>
     <link name="${name}_frame">
@@ -32,8 +31,7 @@
     </link>
     <joint name="${name}_optical_frame_joint" type="fixed" />
-      <origin xyz="0 0 0" rpy="0 0 0" />
-      <parent name="${name}_frame" />
-        <origin xyz="0 0 0" rpy="${-M_PI/2} 0.0 ${-M_PI/2}" />
-      </parent>
+      <origin xyz="0 0 0" rpy="${-M_PI/2} 0.0 ${-M_PI/2}" />
+      <parent link="${name}_frame" //>
+      <child link="${name}_optical_frame"/>
     </joint>
     <link name="${name}_optical_frame">

File: stacks/pr2/pr2_defs/defs/base/alpha2_base_defs.urdf.xacro (robot description, xacro)
@@ -35,12 +35,11 @@
   <macro name="pr2_wheel_alpha2" params="suffix parent reflect">
     <joint name="${parent}_${suffix}_wheel_joint" type="continuous">
-      <origin xyz="0 0 0" rpy="0 0 0" />
       <axis xyz="0 1 0" />
       <limit effort="100" velocity="100"/>
       <safety_controller  k_velocity="10" />
       <dynamics damping="0.0" friction="0.0" />
-      <parent name="${parent}_rotation_link">
-        <origin xyz="0 ${reflect*caster_wheel_offset_y} 0" rpy="0 0 0" />
-      </parent>
+      <origin xyz="0 ${reflect*caster_wheel_offset_y} 0" rpy="0 0 0" />
+      <parent link="${parent}_rotation_link"/>
+      <child link="${parent}_${suffix}_wheel_link"/>
     </joint>
     <link name="${parent}_${suffix}_wheel_link">
@@ -71,5 +70,4 @@
   <macro name="pr2_caster_alpha2" params="suffix parent *origin ref_position">
     <joint name="${suffix}_caster_rotation_joint" type="continuous">
-      <origin xyz="0 0 0" rpy="0 0 0 0"/>
       <axis xyz="0 0 1" />
       <limit effort="100" velocity="100"/>
@@ -77,7 +75,7 @@
       <calibration reference_position="${ref_position}" />
       <dynamics damping="0.0" friction="0.0" />
-      <parent name="${parent}">
-        <insert_block name="origin" />
-      </parent>
+      <insert_block name="origin" />
+      <parent link="${parent}"/>
+      <child link="${suffix}_caster_rotation_link" />
     </joint>
     <link name="${suffix}_caster_rotation_link">
@@ -110,8 +108,7 @@
   <macro name="pr2_base_alpha2" params="name *origin">
     <joint name="${name}_joint" type="planar">
-      <origin xyz="0 0 0" rpy="0 0 0" />
-      <parent name="world">
-        <insert_block name="origin" />
-      </parent>
+      <insert_block name="origin" />
+      <parent link="world"/>
+      <child link="${name}_link" />
     </joint>
     <link name="${name}_link">
@@ -137,9 +134,8 @@
     <!-- base laser -->
     <joint name="base_laser_joint" type="fixed">
-      <origin xyz="0 0 0" rpy="0 0 0" />
       <axis xyz="0 1 0" />
-      <parent name="${name}_link">
-        <origin xyz="${base_laser_x} ${base_laser_y} ${base_height_offset+base_laser_z}" rpy="0 0 0" />
-      </parent>
+      <origin xyz="${base_laser_x} ${base_laser_y} ${base_height_offset+base_laser_z}" rpy="0 0 0" />
+      <parent link="${name}_link"/>
+      <child link="base_laser" />
     </joint>
     <link name="base_laser" type="laser">

File: stacks/pr2/pr2_defs/defs/base/base_defs.urdf.xacro (robot description, xacro)
@@ -32,12 +32,11 @@
   <macro name="pr2_wheel" params="suffix parent reflect">
     <joint name="${parent}_${suffix}_wheel_joint" type="continuous">
-      <origin xyz="0 0 0" rpy="0 0 0" />
       <axis xyz="0 1 0" />
       <limit effort="100" velocity="100"/>
       <safety_controller k_velocity="10" />
       <dynamics damping="0.0" friction="0.0" />
-      <parent name="${parent}_rotation_link">
-        <origin xyz="0 ${reflect*caster_wheel_offset_y} 0" rpy="0 0 0" />
-      </parent>
+      <origin xyz="0 ${reflect*caster_wheel_offset_y} 0" rpy="0 0 0" />
+      <parent link="${parent}_rotation_link"/>
+      <child link="${parent}_${suffix}_wheel_link"/>
     </joint>
     <link name="${parent}_${suffix}_wheel_link">
@@ -68,5 +67,4 @@
   <macro name="pr2_caster" params="suffix parent *origin">
     <joint name="${suffix}_caster_rotation_joint" type="continuous">
-      <origin xyz="0 0 0" rpy="0 0 0" />
       <axis xyz="0 0 1" />
       <limit effort="100" velocity="100"/>
@@ -74,7 +72,7 @@
       <calibration reference_position="0.0" />
       <dynamics damping="0.0" friction="0.0" />
-      <parent name="${parent}">
-        <insert_block name="origin"/>
-      </parent>
+      <insert_block name="origin"/>
+      <parent link="${parent}"/>
+      <child link="${suffix}_caster_rotation_link"/>
     </joint>
     <link name="${suffix}_caster_rotation_link">
@@ -110,8 +108,7 @@
   <macro name="pr2_base" params="name *origin">
     <joint name="${name}_joint" type="planar">
-      <origin xyz="0 0 0" rpy="0 0 0" />
-      <parent name="world">
-        <insert_block name="origin" />
-      </parent>
+      <insert_block name="origin" />
+      <parent link="world"/>
+      <child link="${name}_link"/>
     </joint>
     <link name="${name}_link">
@@ -137,9 +134,8 @@
     <!-- base laser -->
     <joint name="base_laser_joint" type="fixed">
-      <origin xyz="0 0 0" rpy="0 0 0" />
       <axis xyz="0 1 0" />
-      <parent name="${name}_link">
-        <origin xyz="${base_laser_x} ${base_laser_y} ${base_height_offset+base_laser_z}" rpy="0 0 0" />
-      </parent>
+      <origin xyz="${base_laser_x} ${base_laser_y} ${base_height_offset+base_laser_z}" rpy="0 0 0" />
+      <parent link="${name}_link"/>
+      <child link="base_laser"/>
     </joint>
     <link name="base_laser" type="laser">
@@ -164,10 +160,9 @@
     <!-- modeling plug on base holder magnet location -->
     <joint name="plug_magnet_joint" type="fixed">
-      <origin xyz="0 0 0" rpy="0 0 0" />
       <axis xyz="0 1 0" />
       <anchor xyz="0 0 0" />
-      <parent name="${name}_link">
-        <origin xyz="0.18 0 ${base_height_offset+0.235}" rpy="0 0 0" />
-      </parent>
+      <origin xyz="0.18 0 ${base_height_offset+0.235}" rpy="0 0 0" />
+      <parent link="${name}_link"/>
+      <child link="plug_magnet"/>
     </joint>
     <link name="plug_magnet" type="laser">

File: stacks/pr2/pr2_defs/defs/body/body_defs.urdf.xacro (robot description, xacro)
@@ -8,5 +8,4 @@
   <macro name="pr2_torso" params="name parent *origin">
     <joint name="${name}_joint" type="prismatic">
-      <origin xyz="0 0 0" rpy="0 0 0" />
       <axis xyz="0 0 1" />
       <!-- KWatts: Max should be 0.31, changed to 0.20 to prevent jamming -->
@@ -16,7 +15,7 @@
       <calibration reference_position="0.00536" />
       <dynamics damping="10.0" />
-      <parent name="${parent}">
-        <insert_block name="origin" />
-      </parent>
+      <insert_block name="origin" />
+      <parent link="${parent}"/>
+      <child link="${name}_link"/>
     </joint>
     <link name="${name}_link">

File: stacks/pr2/pr2_defs/defs/gripper/gripper_defs.urdf.xacro (robot description, xacro)
@@ -22,11 +22,10 @@
     <!-- Finger proximal digit -->
     <joint name="${prefix}_l_finger_joint" type="revolute">
-      <origin xyz="0 0 0" rpy="0 0 0" />
       <axis xyz="0 0 1" />
       <pr2_finger_limits reflect="1" />
-      <joint_properties damping="${finger_damping}" />
-      <parent name="${parent}">
-        <origin xyz="0.07691 0.01 0" rpy="0 0 0" />
-      </parent>
+      <dynamics damping="${finger_damping}" />
+      <origin xyz="0.07691 0.01 0" rpy="0 0 0" />
+      <parent link="${parent}"/>
+      <child link="${prefix}_l_finger_link"/>
     </joint>
     <link name="${prefix}_l_finger_link">
@@ -60,9 +59,9 @@
       <origin xyz="0 0 0" rpy="0 0 0" />
       <pr2_finger_limits reflect="1" />
-      <joint_properties damping="${finger_damping}" />
+      <dynamics damping="${finger_damping}" />
       <mimic name="${prefix}_l_finger_joint" mult="1" offset="0"/>
-      <parent name="${parent}">
-        <origin xyz="0.07691 -0.01 0" rpy="0 0 0" />
-      </parent>
+      <origin xyz="0.07691 -0.01 0" rpy="0 0 0" />
+      <parent link="${parent}"/>
+      <child link="${prefix}_r_finger_link"/>
     </joint>
     <link name="${prefix}_r_finger_link">
@@ -96,9 +95,9 @@
       <origin xyz="0 0 0" rpy="0 0 0" />
       <pr2_finger_limits reflect="1" />
-      <joint_properties damping="${finger_tip_damping}" />
+      <dynamics damping="${finger_tip_damping}" />
       <mimic name="${prefix}_l_finger_joint" mult="1" offset="0"/>
-      <parent name="${prefix}_l_finger_link">
-        <origin xyz="0.09137 0.00495 0" rpy="0 0 0" />
-      </parent>
+      <origin xyz="0.09137 0.00495 0" rpy="0 0 0" />
+      <parent link="${prefix}_l_finger_link"/>
+      <child link="${prefix}_l_finger_tip_link"/>
     </joint>
     <link name="${prefix}_l_finger_tip_link">
@@ -129,9 +128,9 @@
       <origin xyz="0 0 0" rpy="0 0 0" />
       <pr2_finger_limits reflect="1" />
-      <joint_properties damping="${finger_tip_damping}" />
+      <dynamics damping="${finger_tip_damping}" />
       <mimic name="${prefix}_l_finger_joint" mult="1" offset="0"/>
-      <parent name="${prefix}_r_finger_link">
-        <origin xyz="${0.09137} ${-0.00495} 0" rpy="0 0 0" />
-      </parent>
+      <origin xyz="${0.09137} ${-0.00495} 0" rpy="0 0 0" />
+      <parent link="${prefix}_r_finger_link"/>
+      <child link="${prefix}_r_finger_tip_link"/>
     </joint>
     <link name="${prefix}_r_finger_tip_link">
@@ -163,8 +162,7 @@
   <macro name="pr2_gripper" params="side parent *origin gear_ratio screw_reduction">
     <joint name="${side}_gripper_palm_joint" type="fixed">
-      <origin xyz="0 0 0" rpy="0 0 0" />
-      <parent name="${parent}">
-        <insert_block name="origin"/>
-      </parent>
+      <insert_block name="origin"/>
+      <parent link="${parent}"/>
+      <child link="${side}_gripper_palm_link"/>
     </joint>
     <link name="${side}_gripper_palm_link">
@@ -192,12 +190,11 @@
     <!-- floating link for simulating gripper constraints -->
     <joint name="${side}_gripper_float_joint" type="prismatic">
-      <origin xyz="0 0 0" rpy="0 0 0" />
       <limit lower="-0.05" upper="0.001" effort="0" />
       <safety_controller soft_lower_limit="${-0.05+0.0}" soft_upper_limit="${0.001-0.0}" />
       <axis xyz="1 0 0" />
-      <joint_properties damping="10.0" />
-      <parent name="${side}_gripper_palm_link">
-        <origin xyz="0.05 0 0" rpy="0 0 0" />
-      </parent>
+      <dynamics damping="10.0" />
+      <origin xyz="0.05 0 0" rpy="0 0 0" />
+      <parent link="${side}_gripper_palm_link"/>
+      <child link="${side}_gripper_float_link"/>
     </joint>
     <link name="${side}_gripper_float_link">
@@ -224,8 +221,7 @@
     </link>
     <joint name="${side}_gripper_tool_joint" type="fixed">
-      <origin xyz="0 0 0" rpy="0 0 0" />
-      <parent name="${side}_gripper_palm_link">
-        <origin xyz="0.18 0 0" rpy="0 0 0" />
-      </parent>
+      <origin xyz="0.18 0 0" rpy="0 0 0" />
+      <parent link="${side}_gripper_palm_link"/>
+      <child link="${side}_gripper_tool_frame"/>
     </joint>
     <link name="${side}_gripper_tool_frame">

File: stacks/pr2/pr2_defs/defs/head/alpha2_head_defs.urdf.xacro (robot description, xacro)
@@ -12,5 +12,4 @@
   <macro name="pr2_head_pan_alpha2" params="name parent *origin">
     <joint name="${name}_joint" type="revolute">
-      <origin xyz="0 0 0" rpy="0 0 0" />
       <axis xyz="0 0 1" />
       <limit lower="-2.92" upper="2.92" effort="2.645" velocity="6" />
@@ -18,7 +17,7 @@
       <calibration reference_position="${0.0+cal_head_pan_flag_alpha2}" />
       <dynamics damping="1.0" />
-      <parent name="${parent}">
-        <insert_block name="origin" />
-      </parent>
+      <insert_block name="origin" />
+      <parent link="${parent}"/>
+      <child link="${name}_link"/>
     </joint>
     <link name="${name}_link">
@@ -50,5 +49,4 @@
   <macro name="pr2_head_tilt_alpha2" params="name parent *origin">
     <joint name="${name}_joint" type="revolute">
-      <origin xyz="0 0 0" rpy="0 0 0" />
       <axis xyz="0 1 0" />
       <limit lower="-0.45" upper="1.37" effort="12" velocity="5" />
@@ -56,7 +54,7 @@
       <calibration reference_position="${0.0+cal_head_tilt_flag}" />
       <dynamics damping="1.0" />
-      <parent name="${parent}">
-        <insert_block name="origin" />
-      </parent>
+      <insert_block name="origin" />
+      <parent link="${parent}"/>
+      <child link="${name}_link"/>
     </joint>
     <link name="${name}_link">
@@ -87,5 +85,4 @@
     <!-- Motor must be configured with 148877 motor -->
     <joint name="${name}_joint" type="revolute">
-      <origin xyz="0 0 0" rpy="0 0 0" />
       <axis xyz="0 1 0" />
       <limit lower="-0.45" upper="1.37" effort="12.0" velocity="5" />
@@ -93,7 +90,7 @@
       <calibration reference_position="${0.0+cal_head_tilt_flag_alpha2}" />
       <dynamics damping="1.0" />
-      <parent name="${parent}">
-        <insert_block name="origin" />
-      </parent>
+      <insert_block name="origin" />
+      <parent link="${parent}"/>
+      <child link="${name}_link"/>
     </joint>
     <link name="${name}_link">
@@ -123,5 +120,4 @@
  <macro name="pr2_head_tilt_alpha2b" params="name parent *origin">
     <joint name="${name}_joint" type="revolute">
-      <origin xyz="0 0 0" rpy="0 0 0" />
       <axis xyz="0 1 0" />
       <limit lower="-0.45" upper="1.37" effort="12.0" velocity="5" />
@@ -129,7 +125,7 @@
       <calibration reference_position="${0.0+cal_head_tilt_flag_alpha2}" />
       <dynamics damping="1.0" />
-      <parent name="${parent}">
-        <insert_block name="origin" />
-      </parent>
+      <insert_block name="origin" />
+      <parent link="${parent}"/>
+      <child link="${name}_link"/>
     </joint>
     <link name="${name}_link">
@@ -169,8 +165,7 @@
     <!-- Head plate frame -->
     <joint name="${name}_plate_frame_joint" type="fixed">
-      <origin xyz="0 0 0" rpy="0 0 0" />
-      <parent name="${name}_tilt_link">
-        <origin xyz="0.0232 0 0.0645" rpy="0 0 0" />
-      </parent>
+      <origin xyz="0.0232 0 0.0645" rpy="0 0 0" />
+      <parent link="${name}_tilt_link"/>
+      <child link="${name}_plate_frame"/>
     </joint>
     <link name="${name}_plate_frame">
@@ -210,7 +205,7 @@
     <!-- Head plate frame -->
     <joint name="${name}_plate_frame_joint" type="fixed">
-      <parent name="${name}_tilt_link">
-        <origin xyz="0.0232 0 0.0645" rpy="0 0 0" />
-      </parent>
+      <origin xyz="0.0232 0 0.0645" rpy="0 0 0" />
+      <parent link="${name}_tilt_link"/>
+      <child link="${name}_plate_frame"/>
     </joint>
     <link name="${name}_plate_frame">
@@ -250,8 +245,7 @@
     <!-- Head plate frame -->
     <joint name="${name}_plate_frame_joint" type="fixed">
-      <origin xyz="0 0 0" rpy="0 0 0" />
-      <parent name="${name}_tilt_link">
-        <origin xyz="0.0232 0 0.0645" rpy="0 0 0" />
-      </parent>
+      <origin xyz="0.0232 0 0.0645" rpy="0 0 0" />
+      <parent link="${name}_tilt_link"/>
+      <child link="${name}_plate_frame"/>
     </joint>
     <link name="${name}_plate_frame">

File: stacks/pr2/pr2_defs/defs/head/alpha2_head_sensor_package_defs.urdf.xacro (robot description, xacro)
@@ -9,5 +9,4 @@
   <macro name="pr2_tilting_laser_alpha2" params="name parent *origin">
     <joint name="${name}_mount_joint" type="revolute">
-      <origin xyz="0 0 0" rpy="0 0 0" />
       <axis xyz="0 1 0" />
       <limit lower="-0.785" upper="1.57" effort="0.5292" velocity="10.0" />
@@ -15,7 +14,7 @@
       <calibration reference_position="0.0" />
       <dynamics damping="1.0" />
-      <parent name="${parent}">
-        <insert_block name="origin" />
-      </parent>
+      <insert_block name="origin" />
+      <parent link="${parent}"/>
+      <child link="${name}_mount_link"/>
     </joint>
     <link name="${name}_mount_link">
@@ -41,9 +40,8 @@
     </link>
     <joint name="${name}_joint" type="fixed">
-      <origin xyz="0 0 0" rpy="0 0 0" />
       <axis xyz="0 1 0" />
-      <parent name="${name}_mount_link">
-        <origin xyz="0 0 0.03" rpy="0 0 0" />
-      </parent>
+      <origin xyz="0 0 0.03" rpy="0 0 0" />
+      <parent link="${name}_mount_link"/>
+      <child link="${name}_link"/>
     </joint>
     <link name="${name}_link" type="laser">
