Commit message: update in progress per api review 2.
git-svn-id: https://svn.code.sf.net/p/personalrobots/code/pkg/trunk@22081 f5854215-dd47-0410-b2c4-cdd35faa7885

Former-commit-id: 7de6fa334d42e90f123729333438e2f6b8f89a31

File: stacks/pr2/pr2_defs/defs/head/head_defs.urdf.xacro (robot description, xacro)
@@ -9,5 +9,4 @@
   <macro name="pr2_head_pan" params="name parent *origin">
     <joint name="${name}_joint" type="revolute">
-      <origin xyz="0 0 0" rpy="0 0 0" />
       <axis xyz="0 0 1" />
       <limit lower="-2.92" upper="2.92" effort="2.645" velocity="6" />
@@ -15,7 +14,7 @@
       <calibration reference_position="${-2.79+cal_head_pan_flag}" />
       <dynamics damping="1.0" />
-      <parent name="${parent}">
-        <insert_block name="origin" />
-      </parent>
+      <insert_block name="origin" />
+      <parent link="${parent}"/>
+      <child link="${name}_link"/>
     </joint>
     <link name="${name}_link">
@@ -46,5 +45,4 @@
   <macro name="pr2_head_tilt" params="name parent *origin">
     <joint name="${name}_joint" type="revolute">
-      <origin xyz="0 0 0" rpy="0 0 0" />
       <axis xyz="0 1 0" />
       <limit lower="-0.55" upper="1.047" effort="12.21" velocity="100" />
@@ -52,7 +50,7 @@
       <calibration reference_position="${-0.195+cal_head_tilt_flag}" />
       <dynamics damping="1.0" />
-      <parent name="${parent}">
-        <insert_block name="origin" />
-      </parent>
+      <insert_block name="origin" />
+      <parent link="${parent}"/>
+      <child link="${name}_link"/>
     </joint>
     <link name="${name}_link">
@@ -91,8 +89,7 @@
     <!-- Head plate frame -->
     <joint name="${name}_plate_frame_joint" type="fixed">
-      <origin xyz="0 0 0" rpy="0 0 0" />
-      <parent name="${name}_tilt_link">
-        <origin xyz="0.0232 0 0.0645" rpy="0 0 0" />
-      </parent>
+      <origin xyz="0.0232 0 0.0645" rpy="0 0 0" />
+      <parent link="${name}_tilt_link"/>
+      <child link="${name}_plate_frame"/>
     </joint>
     <link name="${name}_plate_frame">

File: stacks/pr2/pr2_defs/defs/head/head_sensor_package_defs.urdf.xacro (robot description, xacro)
@@ -19,5 +19,4 @@
   <macro name="pr2_tilting_laser" params="name parent *origin">
     <joint name="${name}_mount_joint" type="revolute">
-      <origin xyz="0 0 0" rpy="0 0 0" />
       <axis xyz="0 1 0" />
       <limit lower="-0.785" upper="1.57" effort="0.5292" velocity="100" />
@@ -25,7 +24,7 @@
       <calibration reference_position="-0.35" />
       <dynamics damping="0.008" />
-      <parent name="${parent}">
-        <insert_block name="origin" />
-      </parent>
+      <insert_block name="origin" />
+      <parent link="${parent}"/>
+      <child link="${name}_mount_link"/>
     </joint>
     <link name="${name}_mount_link">
@@ -51,9 +50,8 @@
     </link>
     <joint name="${name}_joint" type="fixed">
-      <origin xyz="0 0 0" rpy="0 0 0" />
       <axis xyz="0 1 0" />
-      <parent name="${name}_mount_link">
-        <origin xyz="0 0 0.03" rpy="0 0 0" />
-      </parent>
+      <origin xyz="0 0 0.03" rpy="0 0 0" />
+      <parent link="${name}_mount_link"/>
+      <child link="${name}_link"/>
     </joint>
     <link name="${name}_link" type="laser">
@@ -86,8 +84,7 @@
   <macro name="pr2_head_sensor_package" params="name hd_name stereo_name parent *origin">
     <joint name="${name}_frame_joint" type="fixed">
-      <origin xyz="0 0 0" rpy="0 0 0" />
-      <parent name="${parent}">
-        <insert_block name="origin" />
-      </parent>
+      <insert_block name="origin" />
+      <parent link="${parent}"/>
+      <child link="${name}_link"/>
     </joint>
     <link name="${name}_link" >
@@ -132,8 +129,7 @@
     <!-- Define link to stereo cameras, set origin relative to that -->
     <joint name="${name}_frame_joint" type="fixed">
-      <origin xyz="0 0 0" rpy="0 0 0" />
-      <parent name="${parent}">
-        <insert_block name="origin" />
-      </parent>
+      <insert_block name="origin" />
+      <parent link="${parent}"/>
+      <child link="${name}_link"/>
     </joint>
     <link name="${name}_link">
@@ -173,8 +169,7 @@
   <macro name="stereo_camera" params="name parent *origin">
     <joint name="${name}_frame_joint" type="fixed">
-      <origin xyz="0 0 0" rpy="0 0 0" />
-      <parent name="${parent}">
-        <insert_block name="origin" />
-      </parent>
+      <insert_block name="origin" />
+      <parent link="${parent}"/>
+      <child link="${name}_link"/>
     </joint>
     <link name="${name}_link">
@@ -199,9 +194,7 @@
     </link>
     <joint name="${name}_optical_frame_joint" type="fixed">
-      <origin xyz="0 0 0" rpy="0 0 0" />
-      <parent name="${name}_link">
-        <origin xyz="${cal_stereo_x}            ${0.045+cal_stereo_y}   ${.0305+cal_stereo_z}"
-                rpy="${-M_PI/2+cal_stereo_roll} ${0.0+cal_stereo_pitch} ${-M_PI/2+cal_stereo_yaw}" />
-      </parent>
+      <origin xyz="${cal_stereo_x}            ${0.045+cal_stereo_y}   ${.0305+cal_stereo_z}" rpy="${-M_PI/2+cal_stereo_roll} ${0.0+cal_stereo_pitch} ${-M_PI/2+cal_stereo_yaw}" />
+      <parent link="${name}_link"/>
+      <child link="${name}_optical_frame"/>
     </joint>
     <link name="${name}_optical_frame" type="camera">
@@ -227,8 +220,7 @@
     </link>
     <joint name="${name}_l_stereo_camera_frame_joint" type="fixed">
-      <origin xyz="0 0 0" rpy="0 0 0" />
-      <parent name="${name}_optical_frame">
-        <origin xyz="0 0 0" rpy="0 ${-M_PI/2} ${M_PI/2}" />
-      </parent>
+      <origin xyz="0 0 0" rpy="0 ${-M_PI/2} ${M_PI/2}" />
+      <parent link="${name}_optical_frame"/>
+      <child link="${name}_l_stereo_camera_frame"/>
     </joint>
     <link name="${name}_l_stereo_camera_frame">
@@ -254,9 +246,7 @@
     </link>
     <joint name="${name}_r_stereo_camera_frame_joint" type="fixed">
-      <origin xyz="0 0 0" rpy="0 0 0" />
-      <parent name="${name}_l_stereo_camera_frame">
-        <origin xyz="${stereo_dx} ${stereo_dy} ${stereo_dz}"
-                rpy="${stereo_rx} ${stereo_ry} ${stereo_rz}" />
-      </parent>
+      <origin xyz="${stereo_dx} ${stereo_dy} ${stereo_dz}" rpy="${stereo_rx} ${stereo_ry} ${stereo_rz}" />
+      <parent link="${name}_l_stereo_camera_frame"/>
+      <child link="${name}_r_stereo_camera_frame"/>
     </joint>
     <link name="${name}_r_stereo_camera_frame">

File: stacks/pr2/pr2_defs/defs/head/prosilica_defs.urdf.xacro (robot description, xacro)
@@ -7,8 +7,7 @@
   <macro name="prosilica_cam" params="name parent *origin">
     <joint name="${name}_frame_joint" type="fixed">
-      <origin xyz="0 0 0" rpy="0 0 0"/>
-      <parent name="${parent}">
-        <insert_block name="origin" />
-      </parent>
+      <insert_block name="origin" />
+      <parent link="${parent}"/>
+      <child link="${name}_frame"/>
     </joint>
     <link name="${name}_frame">
@@ -34,9 +33,8 @@
     </link>
     <joint name="${name}_optical_frame_joint" type="fixed">
-      <origin xyz="0 0 0" rpy="0 0 0"/>
-      <parent name="${name}_frame">
-        <origin xyz="${cal_high_def_x}            ${cal_high_def_y}         ${cal_high_def_z}"
+      <origin xyz="${cal_high_def_x}            ${cal_high_def_y}         ${cal_high_def_z}"
                 rpy="${-M_PI/2+cal_high_def_roll} ${0.0+cal_high_def_pitch} ${-M_PI/2+cal_high_def_yaw}" />
-      </parent>
+      <parent link="${name}_frame"/>
+      <child link="${name}_optical_frame"/>
     </joint>
     <link name="${name}_optical_frame">
