Commit message: * Remove rviz extensions * Add materials for all links
git-svn-id: https://svn.code.sf.net/p/personalrobots/code/pkg/trunk@22242 f5854215-dd47-0410-b2c4-cdd35faa7885

Former-commit-id: 17a79e2c205e12292d5ac85083c0790ff1aadb25

File: stacks/pr2/pr2_defs/defs/arm/arm_defs.urdf.xacro (robot description, xacro)
@@ -4,5 +4,4 @@
        xmlns:interface="http://playerstage.sourceforge.net/gazebo/xmlschema/#interface">
   <include filename="$(find pr2_defs)/defs/arm/arm_gazebo.xacro" />
-  <include filename="$(find pr2_defs)/defs/arm/arm_rviz.xacro" />
   <include filename="$(find pr2_defs)/defs/arm/arm_transmission.xacro" />
   <property name="M_PI" value="3.1415926535897931" />
@@ -58,5 +57,5 @@
           <mesh filename="$(find pr2_defs)/meshes/shoulder_yaw.stl" />
         </geometry>
-        <texture name="PR2/Blue" />
+        <material name="Blue" />
       </visual>
       <collision name="${side}_shoulder_pan_collision">
@@ -94,5 +93,5 @@
           <mesh filename="$(find pr2_defs)/meshes/shoulder_lift.stl" />
         </geometry>
-        <texture name="PR2/Grey" />
+        <material name="Grey" />
       </visual>
       <collision name="${side}_shoulder_lift_collision">
@@ -129,4 +128,5 @@
           <mesh filename="$(find pr2_defs)/meshes/upper_arm_roll.stl" />
         </geometry>
+        <material name="RollLinks" />
       </visual>
       <collision name="${side}_upper_arm_roll_collision">
@@ -163,4 +163,5 @@
           <mesh filename="$(find pr2_defs)/meshes/upper_arm.stl" />
         </geometry>
+        <material name="Green" />
       </visual>
       <collision name="${side}_upper_arm_collision">
@@ -195,4 +196,5 @@
           <mesh filename="$(find pr2_defs)/meshes/elbow_flex.stl" />
         </geometry>
+        <material name="Grey" />
       </visual>
       <collision name="${side}_elbow_flex_collision">
@@ -228,4 +230,5 @@
           <mesh filename="$(find pr2_defs)/meshes/forearm_roll.stl" />
         </geometry>
+        <material name="RollLinks" />
       </visual>
       <collision name="${side}_forearm_roll_collision"> <!-- TODO: collision tag should be optional -->
@@ -257,4 +260,5 @@
           <mesh filename="$(find pr2_defs)/meshes/forearm.stl" />
         </geometry>
+        <material name="Blue" />
       </visual>
       <collision name="${side}_forearm_collision">
@@ -289,4 +293,5 @@
           <mesh filename="$(find pr2_defs)/meshes/wrist_flex.stl" />
         </geometry>
+        <material name="Grey" />
       </visual>
       <collision name="${side}_wrist_flex_collision">
@@ -321,4 +326,5 @@
           <mesh filename="$(find pr2_defs)/meshes/wrist_roll.stl" />
         </geometry>
+        <material name="RollLinks" />
       </visual>
       <collision name="${side}_wrist_roll_collision">
@@ -345,8 +351,4 @@
     <pr2_upper_arm_transmission side="${side}" />
     <pr2_forearm_transmission side="${side}" />
-    <!-- rviz extensions -->
-    <pr2_shoulder_rviz side="${side}" />
-    <pr2_upper_arm_rviz side="${side}" />
-    <pr2_forearm_rviz side="${side}" />
   </macro>
 </robot>

File: stacks/pr2/pr2_defs/defs/base/alpha2_base_defs.urdf.xacro (robot description, xacro)
@@ -3,5 +3,4 @@
        xmlns:controller="http://playerstage.sourceforge.net/gazebo/xmlschema/#controller"
        xmlns:interface="http://playerstage.sourceforge.net/gazebo/xmlschema/#interface">
-  <include filename="$(find pr2_defs)/defs/base/alpha2_base_rviz.xacro" />
   <include filename="$(find pr2_defs)/defs/base/alpha2_base_gazebo.xacro" />
   <include filename="$(find pr2_defs)/defs/base/alpha2_base_transmission.xacro" />
@@ -57,4 +56,5 @@
           <mesh filename="$(find pr2_defs)/meshes/pr2_wheel.stl" />
         </geometry>
+        <material name="Caster_${suffix}" />
       </visual>
       <collision name="${parent}_${suffix}_wheel_collision">
@@ -67,5 +67,4 @@
     <!-- extensions -->
     <pr2_wheel_alpha2_gazebo parent="${parent}" suffix="${suffix}" />
-    <pr2_wheel_alpha2_rviz parent="${parent}" suffix="${suffix}" />
     <pr2_wheel_alpha2_transmission parent="${parent}" suffix="${suffix}" reflect="${reflect}" />
   </macro>
@@ -93,4 +92,5 @@
           <mesh filename="$(find pr2_defs)/meshes/caster.stl" />
         </geometry>
+        <material name="Green" />
       </visual>
       <collision name="${suffix}_caster_rotation_collision">
@@ -106,5 +106,4 @@
     <!-- extensions -->
     <pr2_caster_alpha2_transmission suffix="${suffix}" />
-    <pr2_caster_alpha2_rviz suffix="${suffix}" />
   </macro>
   <macro name="pr2_base_alpha2" params="name *origin">
@@ -126,4 +125,5 @@
           <mesh filename="$(find pr2_defs)/meshes/base.stl" />
         </geometry>
+        <material name="Green" />
       </visual>
       <collision name="${name}_collision">
@@ -152,4 +152,5 @@
           <box size="${base_laser_size_x} ${base_laser_size_y} ${base_laser_size_z}"/>
         </geometry>
+        <material name="Red" />
       </visual>
       <collision name="base_lcollision">
@@ -175,5 +176,4 @@
     <!-- gazebo extensions -->
     <pr2_base_alpha2_gazebo name="${name}" />
-    <pr2_base_alpha2_rviz name="${name}" />
   </macro>
 </robot>

File: stacks/pr2/pr2_defs/defs/base/base_defs.urdf.xacro (robot description, xacro)
@@ -3,6 +3,4 @@
        xmlns:controller="http://playerstage.sourceforge.net/gazebo/xmlschema/#controller"
        xmlns:interface="http://playerstage.sourceforge.net/gazebo/xmlschema/#interface">
-  <!--include filename="$(find pr2_defs)/defs/base_rviz.xacro" /-->
-  <include filename="$(find pr2_defs)/defs/base/base_rviz.xacro" />
   <include filename="$(find pr2_defs)/defs/base/base_gazebo.xacro" />
   <include filename="$(find pr2_defs)/defs/base/base_transmission.xacro" />
@@ -52,4 +50,5 @@
           <mesh filename="$(find pr2_defs)/meshes/pr2_wheel.stl" />
         </geometry>
+        <material name="Caster_${suffix}" />
       </visual>
       <collision name="${parent}_${suffix}_wheel_collision">
@@ -62,5 +61,4 @@
     <!-- extensions -->
     <pr2_wheel_gazebo parent="${parent}" suffix="${suffix}" />
-    <pr2_wheel_rviz parent="${parent}" suffix="${suffix}" />
     <pr2_wheel_transmission parent="${parent}" suffix="${suffix}" reflect="${reflect}" />
   </macro>
@@ -88,4 +86,5 @@
           <mesh filename="$(find pr2_defs)/meshes/caster.stl" />
         </geometry>
+        <material name="Green" />
       </visual>
       <collision name="${suffix}_caster_rotation_collision">
@@ -98,5 +97,4 @@
     <!-- extensions -->
     <pr2_caster_transmission suffix="${suffix}" />
-    <pr2_caster_rviz suffix="${suffix}" />
     <!-- wheel macros -->
     <pr2_wheel parent="${suffix}_caster" suffix="l" reflect="1" />
@@ -124,4 +122,5 @@
           <mesh filename="$(find pr2_defs)/meshes/base.stl" />
         </geometry>
+        <material name="Green" />
       </visual>
       <collision name="${name}_collision">
@@ -150,4 +149,5 @@
           <box size="${base_laser_size_x} ${base_laser_size_y} ${base_laser_size_z}"/>
         </geometry>
+        <material name="Red" />
       </visual>
       <collision name="base_lcollision">
@@ -199,5 +199,4 @@
     <!-- gazebo extensions -->
     <pr2_base_gazebo name="${name}" />
-    <pr2_base_rviz name="${name}" />
   </macro>
 </robot>

File: stacks/pr2/pr2_defs/defs/body/body_defs.urdf.xacro (robot description, xacro)
@@ -4,5 +4,4 @@
        xmlns:interface="http://playerstage.sourceforge.net/gazebo/xmlschema/#interface">
   <include filename="$(find pr2_defs)/defs/body/body_gazebo.xacro" />
-  <include filename="$(find pr2_defs)/defs/body/body_rviz.xacro" />
   <include filename="$(find pr2_defs)/defs/body/body_transmission.xacro" />
   <macro name="pr2_torso" params="name parent *origin">
@@ -31,4 +30,5 @@
           <mesh filename="$(find pr2_defs)/meshes/torso.stl" />
         </geometry>
+        <material name="Grey2" />
       </visual>
       <collision name="${name}_collision">
@@ -42,5 +42,4 @@
     <pr2_torso_gazebo name="${name}" />
     <pr2_torso_transmission name="${name}" />
-    <pr2_torso_rviz name="${name}" />
   </macro>
 </robot>

File: stacks/pr2/pr2_defs/defs/gripper/gripper_defs.urdf.xacro (robot description, xacro)
@@ -5,5 +5,4 @@
        xmlns:interface="http://playerstage.sourceforge.net/gazebo/xmlschema/#interface">
   <include filename="$(find pr2_defs)/defs/gripper/gripper_gazebo.xacro" />
-  <include filename="$(find pr2_defs)/defs/gripper/gripper_rviz.xacro" />
   <include filename="$(find pr2_defs)/defs/gripper/gripper_transmission.xacro" />
   <property name="M_PI" value="3.1415926535897931" />
@@ -45,4 +44,5 @@
           <mesh filename="$(find pr2_defs)/meshes/upper_finger_l.stl" />
         </geometry>
+        <material name="Grey" />
       </visual>
       <collision name="${prefix}_l_finger_collision">
@@ -81,4 +81,5 @@
           <mesh filename="$(find pr2_defs)/meshes/upper_finger_r.stl" />
         </geometry>
+        <material name="Grey" />
       </visual>
       <collision name="${prefix}_r_finger_collision">
@@ -114,4 +115,5 @@
           <mesh filename="$(find pr2_defs)/meshes/finger_tip_l.stl" />
         </geometry>
+        <material name="Green" />
       </visual>
       <collision name="${prefix}_l_finger_tip_collision">
@@ -147,4 +149,5 @@
           <mesh filename="$(find pr2_defs)/meshes/finger_tip_r.stl" />
         </geometry>
+        <material name="Green" />
       </visual>
       <collision name="${prefix}_r_finger_tip_collision">
@@ -158,5 +161,4 @@
     <!-- extensions -->
     <pr2_finger_gazebo prefix="${prefix}" />
-    <pr2_finger_rviz prefix="${prefix}" />
   </macro>
   <macro name="pr2_gripper" params="side parent *origin gear_ratio screw_reduction">
@@ -179,4 +181,5 @@
           <mesh filename="$(find pr2_defs)/meshes/gripper_palm.stl" />
         </geometry>
+        <material name="Red" />
       </visual>
       <collision name="${side}_gripper_palm_collision">
@@ -211,4 +214,5 @@
           <box size="0.001 0.001 0.001" />
         </geometry>
+        <material name="White" />
       </visual>
       <collision name="${side}_gripper_float_collision">
@@ -237,4 +241,5 @@
           <box size="0.001 0.001 0.001" />
         </geometry>
+        <material name="Grey" />
       </visual>
       <collision name="${side}_gripper_tool_collision">
@@ -259,5 +264,4 @@
     <!-- extensions -->
     <pr2_gripper_gazebo side="${side}" />
-    <pr2_gripper_rviz side="${side}" />
     <pr2_gripper_transmission side="${side}" />
   </macro>

File: stacks/pr2/pr2_defs/defs/head/alpha2_head_defs.urdf.xacro (robot description, xacro)
@@ -3,5 +3,4 @@
        xmlns:controller="http://playerstage.sourceforge.net/gazebo/xmlschema/#controller"
        xmlns:interface="http://playerstage.sourceforge.net/gazebo/xmlschema/#interface">
-  <include filename="$(find pr2_defs)/defs/head/alpha2_head_rviz.xacro" />
   <include filename="$(find pr2_defs)/defs/head/alpha2_head_gazebo.xacro" />
   <include filename="$(find pr2_defs)/defs/head/alpha2_head_transmission.xacro" />
@@ -33,4 +32,5 @@
           <mesh filename="$(find pr2_defs)/meshes/head_pan.stl" />
         </geometry>
+        <material name="Blue" />
       </visual>
       <collision name="${name}_collision">
@@ -43,5 +43,4 @@
     <!-- extensions -->
     <pr2_head_pan_alpha2_gazebo name="${name}" />
-    <pr2_head_pan_alpha2_rviz name="${name}" />
     <pr2_head_pan_alpha2_transmission name="${name}" />
   </macro>
@@ -69,4 +68,5 @@
           <mesh filename="$(find pr2_defs)/meshes/head_tilt.stl" />
         </geometry>
+        <material name="Green" />
       </visual>
       <collision name="${name}_collision">
@@ -79,5 +79,4 @@
     <!-- extensions -->
     <pr2_head_tilt_alpha2_gazebo name="${name}" />
-    <pr2_head_tilt_alpha2_rviz name="${name}" />
     <pr2_head_tilt_alpha2_transmission name="${name}" />
   </macro>
@@ -105,4 +104,5 @@
           <mesh filename="$(find pr2_defs)/meshes/head_tilt.stl" />
         </geometry>
+        <material name="Green" />
       </visual>
       <collision name="${name}_collision">
@@ -115,5 +115,4 @@
     <!-- extensions -->
     <pr2_head_tilt_alpha2a_gazebo name="${name}"/>
-    <pr2_head_tilt_alpha2a_rviz name="${name}"/>
     <pr2_head_tilt_alpha2a_transmission name="${name}"/>
   </macro>
@@ -142,4 +141,5 @@
           <mesh filename="$(find pr2_defs)/meshes/head_tilt.stl" />
         </geometry>
+        <material name="Green" />
       </visual>
       <collision name="${name}_collision">
@@ -152,5 +152,4 @@
     <!-- extensions -->
     <pr2_head_tilt_alpha2b_gazebo name="${name}"/>
-    <pr2_head_tilt_alpha2b_rviz name="${name}"/>
     <pr2_head_tilt_alpha2b_transmission name="${name}"/>
   </macro>
@@ -182,4 +181,5 @@
           <box size="0.01 0.01 0.01" />
         </geometry>
+        <material name="Green" />
       </visual>
       <collision name="${name}_plate_frame_collision">
@@ -192,5 +192,4 @@
     <!-- extensions -->
     <pr2_head_alpha2_gazebo name="${name}"/>
-    <pr2_head_alpha2_rviz name="${name}"/>
   </macro>
   <!-- Difference between two heads is motors and gearheads -->
@@ -222,4 +221,5 @@
           <box size="0.01 0.01 0.01" />
         </geometry>
+        <material name="Blue" />
       </visual>
       <collision name="${name}_plate_frame_collision">
@@ -232,5 +232,4 @@
     <!-- extensions -->
     <pr2_head_alpha2a_gazebo name="${name}"/>
-    <pr2_head_alpha2a_rviz name="${name}"/>
     <pr2_head_alpha2a_transmission name="${name}"/>
   </macro>
@@ -262,4 +261,5 @@
           <box size="0.01 0.01 0.01" />
         </geometry>
+        <material name="Blue" />
       </visual>
       <collision name="${name}_plate_frame_collision">
@@ -272,5 +272,4 @@
     <!-- extensions -->
     <pr2_head_alpha2b_gazebo name="${name}"/>
-    <pr2_head_alpha2b_rviz name="${name}"/>
     <pr2_head_alpha2b_transmission name="${name}"/>
   </macro>

File: stacks/pr2/pr2_defs/defs/head/alpha2_head_sensor_package_defs.urdf.xacro (robot description, xacro)
@@ -4,5 +4,4 @@
        xmlns:interface="http://playerstage.sourceforge.net/gazebo/xmlschema/#interface">
   <include filename="$(find pr2_defs)/defs/head/alpha2_head_sensor_package_gazebo.xacro" />
-  <include filename="$(find pr2_defs)/defs/head/alpha2_head_sensor_package_rviz.xacro" />
   <include filename="$(find pr2_defs)/defs/head/alpha2_head_sensor_package_transmission.xacro" />
   <!-- in alpha2 head sensor package, only tilting laser is different, stereo's are the same as alpha1, not repeated -->
@@ -31,4 +30,5 @@
           <mesh filename="$(find pr2_defs)/meshes/hok_tilt.stl" />
         </geometry>
+        <material name="Red" />
       </visual>
       <collision name="${name}_mount_collision">
@@ -56,4 +56,5 @@
           <box size="0.001 0.001 0.001" />
         </geometry>
+        <material name="Red" />
       </visual>
       <collision name="${name}_collision">
@@ -66,5 +67,4 @@
     <!-- extensions -->
     <pr2_tilting_laser_alpha2_gazebo name="${name}"/>
-    <pr2_tilting_laser_alpha2_rviz name="${name}"/>
     <pr2_tilting_laser_alpha2_transmission name="${name}"/>
   </macro>

File: stacks/pr2/pr2_defs/defs/head/head_defs.urdf.xacro (robot description, xacro)
@@ -4,5 +4,4 @@
        xmlns:interface="http://playerstage.sourceforge.net/gazebo/xmlschema/#interface">
   <include filename="$(find pr2_defs)/defs/head/head_gazebo.xacro" />
-  <include filename="$(find pr2_defs)/defs/head/head_rviz.xacro" />
   <include filename="$(find pr2_defs)/defs/head/head_transmission.xacro" />
   <property name="M_PI" value="3.1415926535897931" />
@@ -30,4 +29,5 @@
           <mesh filename="$(find pr2_defs)/meshes/head_pan.stl" />
         </geometry>
+        <material name="Blue" />
       </visual>
       <collision name="${name}_collision">
@@ -41,5 +41,4 @@
     <pr2_head_pan_gazebo name="${name}" />
     <pr2_head_pan_transmission name="${name}" />
-    <pr2_head_pan_rviz name="${name}" />
   </macro>
   <macro name="pr2_head_tilt" params="name parent *origin">
@@ -67,4 +66,5 @@
           <mesh filename="$(find pr2_defs)/meshes/head_tilt.stl" />
         </geometry>
+        <material name="Green" />
       </visual>
       <collision name="${name}_collision">
@@ -77,5 +77,4 @@
     <!-- extensions -->
     <pr2_head_tilt_gazebo name="${name}" />
-    <pr2_head_tilt_rviz name="${name}" />
     <pr2_head_tilt_transmission name="${name}" />
   </macro>
@@ -106,4 +105,5 @@
           <box size="0.01 0.01 0.01" />
         </geometry>
+        <material name="Blue" />
       </visual>
       <collision name="${name}_plate_frame_collision">
@@ -116,5 +116,4 @@
     <!-- extensions -->
     <pr2_head_gazebo name="${name}" />
-    <pr2_head_rviz name="${name}" />
   </macro>
 </robot>

File: stacks/pr2/pr2_defs/defs/head/head_sensor_package_defs.urdf.xacro (robot description, xacro)
@@ -4,5 +4,4 @@
        xmlns:interface="http://playerstage.sourceforge.net/gazebo/xmlschema/#interface">
   <include filename="$(find pr2_defs)/defs/head/head_sensor_package_gazebo.xacro" />
-  <include filename="$(find pr2_defs)/defs/head/head_sensor_package_rviz.xacro" />
   <include filename="$(find pr2_defs)/defs/head/head_sensor_package_transmission.xacro" />
   <property name="stereo_size_x" value="0.005" />
@@ -41,4 +40,5 @@
           <mesh filename="$(find pr2_defs)/meshes/hok_tilt.stl" />
         </geometry>
+        <material name="Red" />
       </visual>
       <collision name="${name}_mount_collision">
@@ -66,4 +66,5 @@
           <box size="0.001 0.001 0.001" />
         </geometry>
+        <material name="Red" />
       </visual>
       <collision name="${name}_collision">
@@ -76,5 +77,4 @@
     <!-- extensions -->
     <pr2_tilting_laser_gazebo name="${name}"/>
-    <pr2_tilting_laser_rviz name="${name}"/>
     <pr2_tilting_laser_transmission name="${name}"/>
   </macro>
@@ -102,4 +102,5 @@
           <box size="0.01 0.01 0.01" />
         </geometry>
+        <material name="Blue" />
       </visual>
       <collision name="${name}_sensor_collision">
@@ -122,5 +123,4 @@
     <!-- extensions -->
     <pr2_head_sensor_package_gazebo name="${name}" />
-    <pr2_head_sensor_package_rviz name="${name}" />
   </macro>
   <!-- Made by Kevin for double stereo camera for PR-2 Beta. -->
@@ -147,4 +147,5 @@
           <box size="0.01 0.01 0.01" />
         </geometry>
+        <material name="Blue" />
       </visual>
       <collision name="${name}_double_stereo_collision">
@@ -165,5 +166,4 @@
     <!-- extensions -->
     <double_stereo_camera_gazebo name="${name}" />
-    <double_stereo_camera_rviz name="${name}" />
   </macro>
   <macro name="stereo_camera" params="name parent *origin">
@@ -185,4 +185,5 @@
           <box size="${stereo_size_x} ${stereo_size_y} ${stereo_size_z}" />
         </geometry>
+        <material name="Blue" />
       </visual>
       <collision name="${name}_collision">
@@ -211,4 +212,5 @@
           <box size="0.01 0.01 0.01" />
         </geometry>
+        <material name="Blue" />
       </visual>
       <collision name="${name}_optical_frame_collision">
@@ -237,4 +239,5 @@
           <box size="0.01 0.01 0.01" />
         </geometry>
+        <material name="Blue" />
       </visual>
       <collision name="${name}_l_stereo_camera_collision">
@@ -263,4 +266,5 @@
           <box size="0.01 0.01 0.01" />
         </geometry>
+        <material name="Blue" />
       </visual>
       <collision name="${name}_r_stereo_camera_collision">
@@ -273,5 +277,4 @@
     <!-- extensions -->
     <stereo_camera_gazebo name="${name}" />
-    <stereo_camera_rviz name="${name}" />
   </macro>
 </robot>

File: stacks/pr2/pr2_defs/defs/head/prosilica_defs.urdf.xacro (robot description, xacro)
@@ -4,5 +4,4 @@
       xmlns:interface="http://playerstage.sourceforge.net/gazebo/xmlschema/#interface">
   <include filename="$(find pr2_defs)/defs/head/prosilica_gazebo.xacro" />
-  <include filename="$(find pr2_defs)/defs/head/prosilica_rviz.xacro" />
   <macro name="prosilica_cam" params="name parent *origin">
     <joint name="${name}_frame_joint" type="fixed">
@@ -24,4 +23,5 @@
           <box size="0.01 0.01 0.01" />
         </geometry>
+        <material name="Blue" />
       </visual>
       <collision name="${name}_collision">
@@ -51,4 +51,5 @@
           <box size="0.01 0.01 0.01" />
         </geometry>
+        <material name="Blue" />
       </visual>
       <collision name="${name}_optical_collision">
@@ -61,5 +62,4 @@
     <!-- extensions -->
     <prosilica_cam_gazebo name="${name}"/>
-    <prosilica_cam_rviz name="${name}"/>
   </macro>
 </root>

File: stacks/pr2/pr2_defs/robots/pr2.urdf.xacro (robot description, xacro)
@@ -13,4 +13,5 @@
   <include filename="$(find pr2_defs)/defs/head/prosilica_defs.urdf.xacro" />
   <include filename="$(find pr2_defs)/defs/gazebo/gazebo_defs.urdf.xacro" />
+  <include filename="$(find pr2_defs)/defs/materials.urdf.xacro" />
   <pr2_base name="base" >
     <origin xyz="0 0 0.051" rpy="0 0 0" /> <!-- 5.1cm is the height of the base when wheels contact ground -->
