Commit message: Convert filepaths to url-style convention -- for now package://
git-svn-id: https://svn.code.sf.net/p/personalrobots/code/pkg/trunk@22359 f5854215-dd47-0410-b2c4-cdd35faa7885

Former-commit-id: 301e074cc94514b07f3b2411fb7d56b296bba222

File: stacks/pr2/pr2_defs/defs/arm/arm_defs.urdf.xacro (robot description, xacro)
@@ -55,5 +55,5 @@
         <origin xyz="0 0 0" rpy="0 0 0" />
         <geometry name="${side}_shoulder_pan_visual_geom">
-          <mesh filename="$(find pr2_defs)/meshes/shoulder_yaw.stl" />
+          <mesh filename="package://pr2_defs/meshes/shoulder_yaw.stl" />
         </geometry>
         <material name="Blue" />
@@ -62,5 +62,5 @@
         <origin xyz="0.0 0 0.0" rpy="0 0 0" />
         <geometry name="${side}_shoulder_pan_collision_geom">
-          <mesh filename="$(find pr2_defs)/meshes/convex/shoulder_yaw_convex.stlb" />
+          <mesh filename="package://pr2_defs/meshes/convex/shoulder_yaw_convex.stlb" />
         </geometry>
       </collision>
@@ -91,5 +91,5 @@
         <origin xyz="0 0 0" rpy="0 0 0" />
         <geometry name="${side}_shoulder_lift_visual_geom">
-          <mesh filename="$(find pr2_defs)/meshes/shoulder_lift.stl" />
+          <mesh filename="package://pr2_defs/meshes/shoulder_lift.stl" />
         </geometry>
         <material name="Grey" />
@@ -98,5 +98,5 @@
         <origin xyz="0 0 0" rpy="0 0 0" />
         <geometry name="${side}_shoulder_lift_collision_geom">
-          <mesh filename="$(find pr2_defs)/meshes/convex/shoulder_lift_convex.stlb" />
+          <mesh filename="package://pr2_defs/meshes/convex/shoulder_lift_convex.stlb" />
         </geometry>
       </collision>
@@ -126,5 +126,5 @@
         <origin xyz="0 0 0" rpy="0 0 0" />
         <geometry name="${side}_upper_arm_roll_visual_geom">
-          <mesh filename="$(find pr2_defs)/meshes/upper_arm_roll.stl" />
+          <mesh filename="package://pr2_defs/meshes/upper_arm_roll.stl" />
         </geometry>
         <material name="RollLinks" />
@@ -161,5 +161,5 @@
         <origin xyz="0 0 0" rpy="0 0 0" />
         <geometry name="${side}_upper_arm_visual_geom">
-          <mesh filename="$(find pr2_defs)/meshes/upper_arm.stl" />
+          <mesh filename="package://pr2_defs/meshes/upper_arm.stl" />
         </geometry>
         <material name="Green" />
@@ -168,5 +168,5 @@
         <origin xyz="0 0 0" rpy="0 0 0" />
         <geometry name="${side}_upper_arm_collision_geom">
-          <mesh filename="$(find pr2_defs)/meshes/convex/upper_arm_convex.stlb" />
+          <mesh filename="package://pr2_defs/meshes/convex/upper_arm_convex.stlb" />
         </geometry>
       </collision>
@@ -194,5 +194,5 @@
         <origin xyz="0 0 0" rpy="0 0 0" />
         <geometry name="${side}_elbow_flex_visual_geom">
-          <mesh filename="$(find pr2_defs)/meshes/elbow_flex.stl" />
+          <mesh filename="package://pr2_defs/meshes/elbow_flex.stl" />
         </geometry>
         <material name="Grey" />
@@ -201,5 +201,5 @@
         <origin xyz="0 0 0" rpy="0 0 0" />
         <geometry name="${side}_elbow_flex_collision_geom">
-          <mesh filename="$(find pr2_defs)/meshes/convex/elbow_flex_convex.stlb" />
+          <mesh filename="package://pr2_defs/meshes/convex/elbow_flex_convex.stlb" />
         </geometry>
       </collision>
@@ -228,5 +228,5 @@
         <origin xyz="0 0 0" rpy="0 0 0" />
         <geometry name="${side}_forearm_roll_visual_geom">
-          <mesh filename="$(find pr2_defs)/meshes/forearm_roll.stl" />
+          <mesh filename="package://pr2_defs/meshes/forearm_roll.stl" />
         </geometry>
         <material name="RollLinks" />
@@ -258,5 +258,5 @@
         <origin xyz="0 0 0" rpy="0 0 0" />
         <geometry name="${side}_forearm_visual_geom">
-          <mesh filename="$(find pr2_defs)/meshes/forearm.stl" />
+          <mesh filename="package://pr2_defs/meshes/forearm.stl" />
         </geometry>
         <material name="Blue" />
@@ -265,5 +265,5 @@
         <origin xyz="0 0 0" rpy="0 0 0" />
         <geometry name="${side}_forearm_collision_geom">
-          <mesh filename="$(find pr2_defs)/meshes/convex/forearm_convex.stlb" />
+          <mesh filename="package://pr2_defs/meshes/convex/forearm_convex.stlb" />
         </geometry>
       </collision>
@@ -291,5 +291,5 @@
         <origin xyz="0 0 0" rpy="0 0 0" />
         <geometry name="${side}_wrist_flex_visual_geom">
-          <mesh filename="$(find pr2_defs)/meshes/wrist_flex.stl" />
+          <mesh filename="package://pr2_defs/meshes/wrist_flex.stl" />
         </geometry>
         <material name="Grey" />
@@ -298,5 +298,5 @@
         <origin xyz="0 0 0" rpy="0 0 0" />
         <geometry name="${side}_wrist_flex_collision_geom">
-          <mesh filename="$(find pr2_defs)/meshes/convex/wrist_flex_convex.stlb" />
+          <mesh filename="package://pr2_defs/meshes/convex/wrist_flex_convex.stlb" />
         </geometry>
       </collision>
@@ -324,5 +324,5 @@
         <origin xyz="0 0 0" rpy="0 0 0" />
         <geometry name="${side}_wrist_roll_visual_geom">
-          <mesh filename="$(find pr2_defs)/meshes/wrist_roll.stl" />
+          <mesh filename="package://pr2_defs/meshes/wrist_roll.stl" />
         </geometry>
         <material name="RollLinks" />

File: stacks/pr2/pr2_defs/defs/base/alpha2_base_defs.urdf.xacro (robot description, xacro)
@@ -54,5 +54,5 @@
         <origin xyz="0 0 0" rpy="0 0 0" />
         <geometry name="${parent}_${suffix}_wheel_visual_geom">
-          <mesh filename="$(find pr2_defs)/meshes/pr2_wheel.stl" />
+          <mesh filename="package://pr2_defs/meshes/pr2_wheel.stl" />
         </geometry>
         <material name="Caster_${suffix}" />
@@ -90,5 +90,5 @@
         <origin xyz="0 0 0" rpy="0 0 0" />
         <geometry name="${suffix}_caster_rotation_visual_geom">
-          <mesh filename="$(find pr2_defs)/meshes/caster.stl" />
+          <mesh filename="package://pr2_defs/meshes/caster.stl" />
         </geometry>
         <material name="Green" />
@@ -123,5 +123,5 @@
         <origin xyz="0 0 ${base_height_offset}" rpy="0 0 0" />
         <geometry name="${name}_visual_geom">
-          <mesh filename="$(find pr2_defs)/meshes/base.stl" />
+          <mesh filename="package://pr2_defs/meshes/base.stl" />
         </geometry>
         <material name="Green" />

File: stacks/pr2/pr2_defs/defs/base/base_defs.urdf.xacro (robot description, xacro)
@@ -48,5 +48,5 @@
         <origin xyz="0 0 0" rpy="0 0 0" />
         <geometry name="${parent}_${suffix}_wheel_visual_geom">
-          <mesh filename="$(find pr2_defs)/meshes/pr2_wheel.stl" />
+          <mesh filename="package://pr2_defs/meshes/pr2_wheel.stl" />
         </geometry>
         <material name="Caster_${suffix}" />
@@ -84,5 +84,5 @@
         <origin xyz="0 0 0" rpy="0 0 0" />
         <geometry name="${suffix}_caster_rotation_visual_geom">
-          <mesh filename="$(find pr2_defs)/meshes/caster.stl" />
+          <mesh filename="package://pr2_defs/meshes/caster.stl" />
         </geometry>
         <material name="Green" />
@@ -120,5 +120,5 @@
         <origin xyz="0 0 ${base_height_offset}" rpy="0 0 0" />
         <geometry name="${name}_visual_geom">
-          <mesh filename="$(find pr2_defs)/meshes/base.stl" />
+          <mesh filename="package://pr2_defs/meshes/base.stl" />
         </geometry>
         <material name="Green" />

File: stacks/pr2/pr2_defs/defs/body/body_defs.urdf.xacro (robot description, xacro)
@@ -28,5 +28,5 @@
         <origin xyz="0 0 0" rpy="0 0 0" />
         <geometry name="${name}_visual_geom">
-          <mesh filename="$(find pr2_defs)/meshes/torso.stl" />
+          <mesh filename="package://pr2_defs/meshes/torso.stl" />
         </geometry>
         <material name="Grey2" />

File: stacks/pr2/pr2_defs/defs/gripper/gripper_defs.urdf.xacro (robot description, xacro)
@@ -42,5 +42,5 @@
         <origin xyz="0 0 0" rpy="0 0 0" />
         <geometry name="${prefix}_l_finger_visual_geom">
-          <mesh filename="$(find pr2_defs)/meshes/upper_finger_l.stl" />
+          <mesh filename="package://pr2_defs/meshes/upper_finger_l.stl" />
         </geometry>
         <material name="Grey" />
@@ -49,5 +49,5 @@
         <origin xyz="0 0 0" rpy="0 0 0" />
         <geometry name="${prefix}_l_finger_collision_geom">
-          <mesh filename="$(find pr2_defs)/meshes/convex/upper_finger_l_convex.stlb" />
+          <mesh filename="package://pr2_defs/meshes/convex/upper_finger_l_convex.stlb" />
         </geometry>
         <verbose value="Yes" />
@@ -79,5 +79,5 @@
         <origin xyz="0 0 0" rpy="0 0 0" />
         <geometry name="${prefix}_r_finger_visual_geom">
-          <mesh filename="$(find pr2_defs)/meshes/upper_finger_r.stl" />
+          <mesh filename="package://pr2_defs/meshes/upper_finger_r.stl" />
         </geometry>
         <material name="Grey" />
@@ -86,5 +86,5 @@
         <origin xyz="0 0 0" rpy="0 0 0" />
         <geometry name="${prefix}_r_finger_collision_geom">
-          <mesh filename="$(find pr2_defs)/meshes/convex/upper_finger_r_convex.stlb" />
+          <mesh filename="package://pr2_defs/meshes/convex/upper_finger_r_convex.stlb" />
         </geometry>
         <verbose value="Yes" />
@@ -113,5 +113,5 @@
         <origin xyz="0 0 0" rpy="0 0 0" />
         <geometry name="${prefix}_l_finger_tip_visual_geom">
-          <mesh filename="$(find pr2_defs)/meshes/finger_tip_l.stl" />
+          <mesh filename="package://pr2_defs/meshes/finger_tip_l.stl" />
         </geometry>
         <material name="Green" />
@@ -120,5 +120,5 @@
         <origin xyz="0 0 0" rpy="0 0 0" />
         <geometry name="${prefix}_l_finger_tip_collision_geom">
-          <mesh filename="$(find pr2_defs)/meshes/convex/finger_tip_l_convex.stlb" />
+          <mesh filename="package://pr2_defs/meshes/convex/finger_tip_l_convex.stlb" />
         </geometry>
         <verbose value="Yes" />
@@ -147,5 +147,5 @@
         <origin xyz="0 0 0" rpy="0 0 0" />
         <geometry name="${prefix}_r_finger_tip_visual_geom">
-          <mesh filename="$(find pr2_defs)/meshes/finger_tip_r.stl" />
+          <mesh filename="package://pr2_defs/meshes/finger_tip_r.stl" />
         </geometry>
         <material name="Green" />
@@ -154,5 +154,5 @@
         <origin xyz="0 0 0" rpy="0 0 0" />
         <geometry name="${prefix}_r_finger_tip_collision_geom">
-          <mesh filename="$(find pr2_defs)/meshes/convex/finger_tip_r_convex.stlb" />
+          <mesh filename="package://pr2_defs/meshes/convex/finger_tip_r_convex.stlb" />
         </geometry>
         <verbose value="Yes" />
@@ -179,5 +179,5 @@
         <origin xyz="0 0 0" rpy="0 0 0" />
         <geometry name="${side}_gripper_palm_visual_geom">
-          <mesh filename="$(find pr2_defs)/meshes/gripper_palm.stl" />
+          <mesh filename="package://pr2_defs/meshes/gripper_palm.stl" />
         </geometry>
         <material name="Red" />
@@ -186,5 +186,5 @@
         <origin xyz="0 0 0" rpy="0 0 0" />
         <geometry name="${side}_gripper_palm_collision_geom">
-          <mesh filename="$(find pr2_defs)/meshes/convex/gripper_palm_convex.stlb" />
+          <mesh filename="package://pr2_defs/meshes/convex/gripper_palm_convex.stlb" />
         </geometry>
         <verbose value="Yes" />

File: stacks/pr2/pr2_defs/defs/head/alpha2_head_defs.urdf.xacro (robot description, xacro)
@@ -30,5 +30,5 @@
         <origin xyz="0 0 0.0" rpy="0 0 0 " />
         <geometry name="${name}_visual_geom">
-          <mesh filename="$(find pr2_defs)/meshes/head_pan.stl" />
+          <mesh filename="package://pr2_defs/meshes/head_pan.stl" />
         </geometry>
         <material name="Blue" />
@@ -66,5 +66,5 @@
         <origin xyz="0 0 0" rpy="0.0 0.0 0.0 " />
         <geometry name="${name}_visual_geom">
-          <mesh filename="$(find pr2_defs)/meshes/head_tilt.stl" />
+          <mesh filename="package://pr2_defs/meshes/head_tilt.stl" />
         </geometry>
         <material name="Green" />
@@ -102,5 +102,5 @@
         <origin xyz="0 0 0" rpy="0.0 0.0 0.0" />
         <geometry name="${name}_visual_geom">
-          <mesh filename="$(find pr2_defs)/meshes/head_tilt.stl" />
+          <mesh filename="package://pr2_defs/meshes/head_tilt.stl" />
         </geometry>
         <material name="Green" />
@@ -139,5 +139,5 @@
         <origin xyz="0 0 0" rpy="0.0 0.0 0.0 " />
         <geometry name="${name}_visual_geom">
-          <mesh filename="$(find pr2_defs)/meshes/head_tilt.stl" />
+          <mesh filename="package://pr2_defs/meshes/head_tilt.stl" />
         </geometry>
         <material name="Green" />

File: stacks/pr2/pr2_defs/defs/head/alpha2_head_sensor_package_defs.urdf.xacro (robot description, xacro)
@@ -28,5 +28,5 @@
         <origin xyz="0 0 0" rpy="0 0 0" />
         <geometry name="${name}_mount_visual_geom">
-          <mesh filename="$(find pr2_defs)/meshes/hok_tilt.stl" />
+          <mesh filename="package://pr2_defs/meshes/hok_tilt.stl" />
         </geometry>
         <material name="Red" />

File: stacks/pr2/pr2_defs/defs/head/head_defs.urdf.xacro (robot description, xacro)
@@ -27,5 +27,5 @@
         <origin xyz="0 0 0.0" rpy="0 0 0 " />
         <geometry name="${name}_visual_geom">
-          <mesh filename="$(find pr2_defs)/meshes/head_pan.stl" />
+          <mesh filename="package://pr2_defs/meshes/head_pan.stl" />
         </geometry>
         <material name="Blue" />
@@ -64,5 +64,5 @@
         <origin xyz="0 0 0" rpy="0.0 0.0 0.0 " />
         <geometry name="${name}_visual_geom">
-          <mesh filename="$(find pr2_defs)/meshes/head_tilt.stl" />
+          <mesh filename="package://pr2_defs/meshes/head_tilt.stl" />
         </geometry>
         <material name="Green" />

File: stacks/pr2/pr2_defs/defs/head/head_sensor_package_defs.urdf.xacro (robot description, xacro)
@@ -38,5 +38,5 @@
         <origin xyz="0 0 0" rpy="0 0 0" />
         <geometry name="${name}_mount_visual_geom">
-          <mesh filename="$(find pr2_defs)/meshes/hok_tilt.stl" />
+          <mesh filename="package://pr2_defs/meshes/hok_tilt.stl" />
         </geometry>
         <material name="Red" />

File: stacks/pr2/pr2_defs/defs/materials.urdf.xacro (robot description, xacro)
@@ -20,11 +20,11 @@
   </material>
   <material name="Caster_l">
-    <texture filename="$(find pr2_ogre)/Media/materials/textures/pr2_wheel_left.png" />
+    <texture filename="package://pr2_ogre/Media/materials/textures/pr2_wheel_left.png" />
   </material>
   <material name="Caster_r">
-    <texture filename="$(find pr2_ogre)/Media/materials/textures/pr2_wheel_right.png" />
+    <texture filename="package://pr2_ogre/Media/materials/textures/pr2_wheel_right.png" />
   </material>
   <material name="RollLinks">
-    <texture filename="$(find pr2_ogre)/Media/materials/textures/pr2_wheel_left.png" />
+    <texture filename="package://pr2_ogre/Media/materials/textures/pr2_wheel_left.png" />
   </material>
 </robot>
