Commit message: update URDF that I missed in robots/
git-svn-id: https://svn.code.sf.net/p/personalrobots/code/pkg/trunk@22400 f5854215-dd47-0410-b2c4-cdd35faa7885

Former-commit-id: 96e8d35e7978476eb2980171794e8e8dd62655e6

File: stacks/pr2/pr2_defs/robots/hca.urdf.xacro (robot description, xacro)
@@ -11,9 +11,10 @@
   <include filename="$(find pr2_defs)/defs/materials.urdf.xacro" />
   <!-- Make base joint for visualization -->
-  <joint name="base_joint" type="fixed" />
+  <joint name="base_joint" type="fixed">
+    <origin xyz=" 0 0 0.53 " rpy=" 0 0 0" />
+    <parent link="world" />
+    <child link="base_link" />
+  </joint>
   <link name="base_link">
-    <parent name="world" />
-    <origin xyz=" 0 0 0.53 " rpy=" 0 0 0" />
-    <joint name="base_joint" />
     <inertial>
       <mass value="100" />

File: stacks/pr2/pr2_defs/robots/hcb.urdf.xacro (robot description, xacro)
@@ -11,9 +11,10 @@
   <include filename="$(find pr2_defs)/defs/materials.urdf.xacro" />
   <!-- Make base joint for visualization -->
-  <joint name="base_joint" type="fixed" />
+  <joint name="base_joint" type="fixed">
+    <origin xyz="0 0 0.53" rpy="0 0 0" />
+    <parent link="world" />
+    <child link="base_link" />
+  </joint>
   <link name="base_link">
-    <parent name="world" />
-    <origin xyz=" 0 0 0.53 " rpy=" 0 0 0" />
-    <joint name="base_joint" />
     <inertial>
       <mass value="100" />

File: stacks/pr2/pr2_defs/robots/hcc.urdf.xacro (robot description, xacro)
@@ -12,9 +12,10 @@
   <include filename="$(find pr2_defs)/defs/materials.urdf.xacro" />
   <!-- Make base joint for visualization -->
-  <joint name="base_joint" type="fixed" />
+  <joint name="base_joint" type="fixed">
+    <origin xyz="0 0 0.53" rpy="0 0 0" />
+    <parent link="world" />
+    <child link="base_link" />
+  </joint>
   <link name="base_link">
-    <parent name="world" />
-    <origin xyz=" 0 0 0.53 " rpy=" 0 0 0" />
-    <joint name="base_joint" />
     <inertial>
       <mass value="100" />

File: stacks/pr2/pr2_defs/robots/l_arm.urdf.xacro (robot description, xacro)
@@ -29,9 +29,10 @@
   </pr2_gripper>
   <!-- Solid Base -->
-  <joint name="base_joint" type="fixed" />
+  <joint name="base_joint" type="fixed">
+    <origin xyz="0 0 0" rpy="0 0 0" />
+    <parent link="world" />
+    <child link="base_link" />
+  </joint>
   <link name="torso_lift_link">
-    <parent name="world" />
-    <origin xyz="0 0 0" rpy=" 0 0 0" />
-    <joint name="base_joint" />
     <inertial>
       <mass value="1000" />

File: stacks/pr2/pr2_defs/robots/l_gripper.urdf.xacro (robot description, xacro)
@@ -24,9 +24,10 @@
   </pr2_gripper>
   <!-- Solid Base -->
-  <joint name="base_joint" type="fixed"/>
+  <joint name="base_joint" type="fixed">
+    <origin xyz="0 0 0" rpy="0 0 0" />
+    <parent link="world" />
+    <child link="base_link" />
+  </joint>
   <link name="base_link">
-    <parent name=" world" />
-    <origin xyz="0 0 0" rpy="0 0 0" />
-    <joint name="base_joint" />
     <inertial>
       <mass value="1000" />

File: stacks/pr2/pr2_defs/robots/r_arm.urdf.xacro (robot description, xacro)
@@ -29,9 +29,10 @@
   </pr2_gripper>
   <!-- Solid Base -->
-  <joint name="base_joint" type="fixed" />
+  <joint name="base_joint" type="fixed">
+    <origin xyz="0 0 0" rpy="0 0 0" />
+    <parent link="world" />
+    <child link="torso_lift_link" />
+  </joint>
   <link name="torso_lift_link">
-    <parent name="world" />
-    <origin xyz="0 0 0" rpy=" 0 0 0" />
-    <joint name="base_joint" />
     <inertial>
       <mass value="1000" />

File: stacks/pr2/pr2_defs/robots/r_forearm_gripper.urdf.xacro (robot description, xacro)
@@ -28,10 +28,11 @@
   <!-- Solid Base -->
   <joint name="base_joint" type="planar">
+    <origin xyz="0 0 1.002" rpy=" 0 0 0" />
+    <parent link=" world" />
+    <!-- rotation of a local coordinate frame attached to the link with respect to a global coordinate frame -->
+    <!-- position of a local coordinate frame attached to the link with respect to the parent link's coordinate frame -->
+    <child link="base_link" />
   </joint>
   <link name="base_link"><!-- link specifying the base of the robot -->
-    <parent name=" world" />
-    <!-- rotation of a local coordinate frame attached to the link with respect to a global coordinate frame -->
-    <origin xyz=" 0 0 1.002 " rpy=" 0 0 0" /> <!-- position of a local coordinate frame attached to the link with respect to the parent link's coordinate frame -->
-    <joint name="base_joint" />
     <inertial>
       <mass value="1000" />

File: stacks/pr2/pr2_defs/robots/r_gripper.urdf.xacro (robot description, xacro)
@@ -24,9 +24,10 @@
   </pr2_gripper>
   <!-- Solid Base -->
-  <joint name="base_joint" type="fixed"/>
+  <joint name="base_joint" type="fixed">
+    <parent link=" world" />
+    <origin xyz="0 0 0" rpy="0 0 0" />
+    <child link="base_link" />
+  </joint>
   <link name="base_link">
-    <parent name=" world" />
-    <origin xyz="0 0 0" rpy="0 0 0" />
-    <joint name="base_joint" />
     <inertial>
       <mass value="1000" />
