Commit message: fix urdf for texas
git-svn-id: https://svn.code.sf.net/p/personalrobots/code/pkg/trunk@23598 f5854215-dd47-0410-b2c4-cdd35faa7885

Former-commit-id: 7543ad6b839220ecb73c883cc3f97781673d4117

File: sandbox/texas/texas.urdf.xacro (robot description, xacro)
@@ -2,4 +2,5 @@
   <include filename="$(find pr2_defs)/calibration/default_cal.xml" />
   <include filename="$(find pr2_defs)/defs/base/base_defs.urdf.xacro" />
+  <include filename="$(find pr2_defs)/defs/materials.urdf.xacro" />
 <pr2_caster suffix="bl" parent="base_link">
       <origin xyz="0 0 0" rpy="0 0 0" />
@@ -14,5 +15,5 @@
     <inertial>
       <mass value="100" />
-      <com xyz=" 0 0 0 " />
+      <origin xyz=" 0 0 0 " />
       <inertia ixx="100"  ixy="0"  ixz="0" iyy="100" iyz="0" izz="100" />
     </inertial>

Commit message: Fixed dallas bot launch file to calibrate
git-svn-id: https://svn.code.sf.net/p/personalrobots/code/pkg/trunk@23601 f5854215-dd47-0410-b2c4-cdd35faa7885

Former-commit-id: e1f4a74f73e8fb2a5ef314c32200171abd64a5f1

File: sandbox/texas/texas.urdf.xacro (robot description, xacro)
@@ -3,7 +3,7 @@
   <include filename="$(find pr2_defs)/defs/base/base_defs.urdf.xacro" />
   <include filename="$(find pr2_defs)/defs/materials.urdf.xacro" />
-<pr2_caster suffix="bl" parent="base_link">
-      <origin xyz="0 0 0" rpy="0 0 0" />
-</pr2_caster>
+  <pr2_caster suffix="bl" parent="base_link" ref_position="-0.785">
+    <origin xyz="0 0 0" rpy="0 0 0" />
+  </pr2_caster>
   <!-- Solid Base for visualizer -->
   <joint name="base_joint" type="planar">

Commit message: fixed caster offset
git-svn-id: https://svn.code.sf.net/p/personalrobots/code/pkg/trunk@23670 f5854215-dd47-0410-b2c4-cdd35faa7885

Former-commit-id: b6c22fcd0276df70b4c286e194bb4fd6f7d1fed1

File: sandbox/texas/texas.urdf.xacro (robot description, xacro)
@@ -4,5 +4,5 @@
   <include filename="$(find pr2_defs)/defs/materials.urdf.xacro" />
   <pr2_caster_alpha2 suffix="bl" parent="base_link" ref_position="-0.785">
-    <origin xyz="0 0 0" rpy="0 0 0" />
+    <origin xyz="-0.43 0 0" rpy="0 0 0" />
   </pr2_caster_alpha2>
   <!-- Solid Base for visualizer -->
